File: clamp/clamps.sch (KiCad schematic (older format))
At the start: 36 parts

Commit message: annotate
Parts:
- gave numbers to parts that had none: 36
Changed lines of the file:
@@
 $EndDescr
 $Comp
-L C C?
+L C C1
 U 1 1 586230E1
 P 7100 1550
-F 0 "C?" H 7125 1650 50  0000 L CNN
+F 0 "C1" H 7125 1650 50  0000 L CNN
 F 1 "C" H 7125 1450 50  0000 L CNN
 F 2 "Capacitors_SMD:C_1206" H 7138 1400 50  0001 C CNN
@@
 +VE
 $Comp
-L LM741 U?
+L LM741 U3
 U 1 1 586230E9
 P 4900 1500
-F 0 "U?" H 4900 1750 50  0000 L CNN
+F 0 "U3" H 4900 1750 50  0000 L CNN
 F 1 "LM741" H 4900 1650 50  0000 L CNN
 F 2 "Housings_SOIC:SOIC-8_3.9x4.9mm_Pitch1.27mm" H 4950 1550 50  0001 C CNN
@@
 -VE
 $Comp
-L 1N4148 D?
+L 1N4148 D1
 U 1 1 586230F4
 P 5500 1500
-F 0 "D?" V 5425 1575 40  0000 L BNN
+F 0 "D1" V 5425 1575 40  0000 L BNN
 F 1 "1N4148" H 5375 1425 40  0000 L CNN
 F 2 "Diodes_SMD:MiniMELF_Standard" H 5500 1650 30  0001 C CNN
@@
 	5650 1500 6050 1500
 $Comp
-L R R?
+L R R13
 U 1 1 58623100
 P 5500 850
-F 0 "R?" V 5580 850 50  0000 C CNN
+F 0 "R13" V 5580 850 50  0000 C CNN
 F 1 "R" V 5500 850 50  0000 C CNN
 F 2 "Resistors_SMD:R_1206" V 5430 850 50  0001 C CNN
@@
 Connection ~ 6050 1500
 $Comp
-L C C?
+L C C5
 U 1 1 5862310D
 P 7600 1550
-F 0 "C?" H 7625 1650 50  0000 L CNN
+F 0 "C5" H 7625 1650 50  0000 L CNN
 F 1 "C" H 7625 1450 50  0000 L CNN
 F 2 "Capacitors_SMD:C_1206" H 7638 1400 50  0001 C CNN
@@
 $EndComp
 $Comp
-L LM741 U?
+L LM741 U4
 U 1 1 58623114
 P 4900 2800
-F 0 "U?" H 4900 3050 50  0000 L CNN
+F 0 "U4" H 4900 3050 50  0000 L CNN
 F 1 "LM741" H 4900 2950 50  0000 L CNN
 F 2 "Housings_SOIC:SOIC-8_3.9x4.9mm_Pitch1.27mm" H 4950 2850 50  0001 C CNN
@@
 NoConn ~ 5000 3100
 $Comp
-L 1N4148 D?
+L 1N4148 D4
 U 1 1 58623121
 P 5550 2800
-F 0 "D?" V 5475 2875 40  0000 L BNN
+F 0 "D4" V 5475 2875 40  0000 L BNN
 F 1 "1N4148" H 5425 2725 40  0000 L CNN
 F 2 "Diodes_SMD:MiniMELF_Standard" H 5550 2950 30  0001 C CNN
@@
 I-SET
 $Comp
-L R R?
+L R R5
 U 1 1 58623130
 P 3600 1200
-F 0 "R?" V 3680 1200 50  0000 C CNN
+F 0 "R5" V 3680 1200 50  0000 C CNN
 F 1 "R" V 3600 1200 50  0000 C CNN
 F 2 "Resistors_SMD:R_1206" V 3530 1200 50  0001 C CNN
@@
 $EndComp
 $Comp
-L R R?
+L R R6
 U 1 1 58623137
 P 3600 1400
-F 0 "R?" V 3680 1400 50  0000 C CNN
+F 0 "R6" V 3680 1400 50  0000 C CNN
 F 1 "R" V 3600 1400 50  0000 C CNN
 F 2 "Resistors_SMD:R_1206" V 3530 1400 50  0001 C CNN
@@
 	1650 1400 1650 2800
 $Comp
-L R R?
+L R R9
 U 1 1 58623142
 P 3650 2700
-F 0 "R?" V 3730 2700 50  0000 C CNN
+F 0 "R9" V 3730 2700 50  0000 C CNN
 F 1 "R" V 3650 2700 50  0000 C CNN
 F 2 "Resistors_SMD:R_1206" V 3580 2700 50  0001 C CNN
@@
 $EndComp
 $Comp
-L R R?
+L R R10
 U 1 1 58623149
 P 3650 2900
-F 0 "R?" V 3730 2900 50  0000 C CNN
+F 0 "R10" V 3730 2900 50  0000 C CNN
 F 1 "R" V 3650 2900 50  0000 C CNN
 F 2 "Resistors_SMD:R_1206" V 3580 2900 50  0001 C CNN
@@
 GND
 $Comp
-L C C?
+L C C3
 U 1 1 5862315A
 P 7350 1550
-F 0 "C?" H 7375 1650 50  0000 L CNN
+F 0 "C3" H 7375 1650 50  0000 L CNN
 F 1 "C" H 7375 1450 50  0000 L CNN
 F 2 "Capacitors_SMD:C_1206" H 7388 1400 50  0001 C CNN
@@
 GND
 $Comp
-L C C?
+L C C2
 U 1 1 58623165
 P 7100 2550
-F 0 "C?" H 7125 2650 50  0000 L CNN
+F 0 "C2" H 7125 2650 50  0000 L CNN
 F 1 "C" H 7125 2450 50  0000 L CNN
 F 2 "Capacitors_SMD:C_1206" H 7138 2400 50  0001 C CNN
@@
 $EndComp
 $Comp
-L C C?
+L C C6
 U 1 1 5862316C
 P 7600 2550
-F 0 "C?" H 7625 2650 50  0000 L CNN
+F 0 "C6" H 7625 2650 50  0000 L CNN
 F 1 "C" H 7625 2450 50  0000 L CNN
 F 2 "Capacitors_SMD:C_1206" H 7638 2400 50  0001 C CNN
@@
 GND
 $Comp
-L C C?
+L C C4
 U 1 1 58623177
 P 7350 2550
-F 0 "C?" H 7375 2650 50  0000 L CNN
+F 0 "C4" H 7375 2650 50  0000 L CNN
 F 1 "C" H 7375 2450 50  0000 L CNN
 F 2 "Capacitors_SMD:C_1206" H 7388 2400 50  0001 C CNN
@@
 NoConn ~ 7550 4750
 $Comp
-L LM741 U?
+L LM741 U5
 U 1 1 58623192
 P 4900 4100
-F 0 "U?" H 4900 4350 50  0000 L CNN
+F 0 "U5" H 4900 4350 50  0000 L CNN
 F 1 "LM741" H 4900 4250 50  0000 L CNN
 F 2 "Housings_SOIC:SOIC-8_3.9x4.9mm_Pitch1.27mm" H 4950 4150 50  0001 C CNN
@@
 -VE
 $Comp
-L 1N4148 D?
+L 1N4148 D2
 U 1 1 5862319C
 P 5500 4100
-F 0 "D?" V 5425 4175 40  0000 L BNN
+F 0 "D2" V 5425 4175 40  0000 L BNN
 F 1 "1N4148" H 5375 4025 40  0000 L CNN
 F 2 "Diodes_SMD:MiniMELF_Standard" H 5500 4250 30  0001 C CNN
@@
 Connection ~ 6050 4100
 $Comp
-L LM741 U?
+L LM741 U6
 U 1 1 586231AA
 P 4900 5400
-F 0 "U?" H 4900 5650 50  0000 L CNN
+F 0 "U6" H 4900 5650 50  0000 L CNN
 F 1 "LM741" H 4900 5550 50  0000 L CNN
 F 2 "Housings_SOIC:SOIC-8_3.9x4.9mm_Pitch1.27mm" H 4950 5450 50  0001 C CNN
@@
 NoConn ~ 5000 5700
 $Comp
-L 1N4148 D?
+L 1N4148 D3
 U 1 1 586231B8
 P 5500 5400
-F 0 "D?" V 5425 5475 40  0000 L BNN
+F 0 "D3" V 5425 5475 40  0000 L BNN
 F 1 "1N4148" H 5375 5325 40  0000 L CNN
 F 2 "Diodes_SMD:MiniMELF_Standard" H 5500 5550 30  0001 C CNN
@@
 Connection ~ 6050 4750
 $Comp
-L LM741 U?
+L LM741 U2
 U 1 1 586231C1
 P 2600 5300
-F 0 "U?" H 2600 5550 50  0000 L CNN
+F 0 "U2" H 2600 5550 50  0000 L CNN
 F 1 "LM741" H 2600 5450 50  0000 L CNN
 F 2 "Housings_SOIC:SOIC-8_3.9x4.9mm_Pitch1.27mm" H 2650 5350 50  0001 C CNN
@@
 	3000 5950 2700 5950
 $Comp
-L R R?
+L R R4
 U 1 1 586231CB
 P 2550 5950
-F 0 "R?" V 2630 5950 50  0000 C CNN
+F 0 "R4" V 2630 5950 50  0000 C CNN
 F 1 "R" V 2550 5950 50  0000 C CNN
 F 2 "Resistors_SMD:R_1206" V 2480 5950 50  0001 C CNN
@@
 $EndComp
 $Comp
-L R R?
+L R R2
 U 1 1 586231D2
 P 2000 5400
-F 0 "R?" V 2080 5400 50  0000 C CNN
+F 0 "R2" V 2080 5400 50  0000 C CNN
 F 1 "R" V 2000 5400 50  0000 C CNN
 F 2 "Resistors_SMD:R_1206" V 1930 5400 50  0001 C CNN
@@
 	3150 4700 1850 4700
 $Comp
-L R R?
+L R R7
 U 1 1 586231E6
 P 3600 4000
-F 0 "R?" V 3680 4000 50  0000 C CNN
+F 0 "R7" V 3680 4000 50  0000 C CNN
 F 1 "R" V 3600 4000 50  0000 C CNN
 F 2 "Resistors_SMD:R_1206" V 3530 4000 50  0001 C CNN
@@
 $EndComp
 $Comp
-L R R?
+L R R8
 U 1 1 586231ED
 P 3600 4200
-F 0 "R?" V 3680 4200 50  0000 C CNN
+F 0 "R8" V 3680 4200 50  0000 C CNN
 F 1 "R" V 3600 4200 50  0000 C CNN
 F 2 "Resistors_SMD:R_1206" V 3530 4200 50  0001 C CNN
@@
 	1650 4200 1650 5400
 $Comp
-L R R?
+L R R12
 U 1 1 586231FB
 P 3650 5300
-F 0 "R?" V 3730 5300 50  0000 C CNN
+F 0 "R12" V 3730 5300 50  0000 C CNN
 F 1 "R" V 3650 5300 50  0000 C CNN
 F 2 "Resistors_SMD:R_1206" V 3580 5300 50  0001 C CNN
@@
 $EndComp
 $Comp
-L R R?
+L R R11
 U 1 1 58623202
 P 3650 5050
-F 0 "R?" V 3730 5050 50  0000 C CNN
+F 0 "R11" V 3730 5050 50  0000 C CNN
 F 1 "R" V 3650 5050 50  0000 C CNN
 F 2 "Resistors_SMD:R_1206" V 3580 5050 50  0001 C CNN
@@
 V-SET
 $Comp
-L CONN_01X12 P?
+L CONN_01X12 P1
 U 1 1 58623218
 P 7750 4300
-F 0 "P?" H 7750 4950 50  0000 C CNN
+F 0 "P1" H 7750 4950 50  0000 C CNN
 F 1 "CONN_01X12" V 7850 4300 50  0000 C CNN
 F 2 "Pin_Headers:Pin_Header_Straight_1x12" H 7750 4300 50  0001 C CNN
@@
 	6050 5400 5650 5400
 $Comp
-L C C?
+L C C7
 U 1 1 58623221
 P 7850 1550
-F 0 "C?" H 7875 1650 50  0000 L CNN
+F 0 "C7" H 7875 1650 50  0000 L CNN
 F 1 "C" H 7875 1450 50  0000 L CNN
 F 2 "Capacitors_SMD:C_1206" H 7888 1400 50  0001 C CNN
@@
 $EndComp
 $Comp
-L C C?
+L C C11
 U 1 1 58623228
 P 8350 1550
-F 0 "C?" H 8375 1650 50  0000 L CNN
+F 0 "C11" H 8375 1650 50  0000 L CNN
 F 1 "C" H 8375 1450 50  0000 L CNN
 F 2 "Capacitors_SMD:C_1206" H 8388 1400 50  0001 C CNN
@@
 GND
 $Comp
-L C C?
+L C C9
 U 1 1 58623231
 P 8100 1550
-F 0 "C?" H 8125 1650 50  0000 L CNN
+F 0 "C9" H 8125 1650 50  0000 L CNN
 F 1 "C" H 8125 1450 50  0000 L CNN
 F 2 "Capacitors_SMD:C_1206" H 8138 1400 50  0001 C CNN
@@
 GND
 $Comp
-L C C?
+L C C8
 U 1 1 5862323C
 P 7850 2550
-F 0 "C?" H 7875 2650 50  0000 L CNN
+F 0 "C8" H 7875 2650 50  0000 L CNN
 F 1 "C" H 7875 2450 50  0000 L CNN
 F 2 "Capacitors_SMD:C_1206" H 7888 2400 50  0001 C CNN
@@
 $EndComp
 $Comp
-L C C?
+L C C12
 U 1 1 58623243
 P 8350 2550
-F 0 "C?" H 8375 2650 50  0000 L CNN
+F 0 "C12" H 8375 2650 50  0000 L CNN
 F 1 "C" H 8375 2450 50  0000 L CNN
 F 2 "Capacitors_SMD:C_1206" H 8388 2400 50  0001 C CNN
@@
 GND
 $Comp
-L C C?
+L C C10
 U 1 1 5862324C
 P 8100 2550
-F 0 "C?" H 8125 2650 50  0000 L CNN
+F 0 "C10" H 8125 2650 50  0000 L CNN
 F 1 "C" H 8125 2450 50  0000 L CNN
 F 2 "Capacitors_SMD:C_1206" H 8138 2400 50  0001 C CNN
@@
 	2900 2700 3500 2700
 $Comp
-L LM741 U?
+L LM741 U1
 U 1 1 58623261
 P 2600 2700
-F 0 "U?" H 2600 2950 50  0000 L CNN
+F 0 "U1" H 2600 2950 50  0000 L CNN
 F 1 "LM741" H 2600 2850 50  0000 L CNN
 F 2 "Housings_SOIC:SOIC-8_3.9x4.9mm_Pitch1.27mm" H 2650 2750 50  0001 C CNN
@@
 	3000 3350 2700 3350
 $Comp
-L R R?
+L R R3
 U 1 1 5862326B
 P 2550 3350
-F 0 "R?" V 2630 3350 50  0000 C CNN
+F 0 "R3" V 2630 3350 50  0000 C CNN
 F 1 "R" V 2550 3350 50  0000 C CNN
 F 2 "Resistors_SMD:R_1206" V 2480 3350 50  0001 C CNN
@@
 $EndComp
 $Comp
-L R R?
+L R R1
 U 1 1 58623272
 P 2000 2800
-F 0 "R?" V 2080 2800 50  0000 C CNN
+F 0 "R1" V 2080 2800 50  0000 C CNN
 F 1 "R" V 2000 2800 50  0000 C CNN
 F 2 "Resistors_SMD:R_1206" V 1930 2800 50  0001 C CNN
