File: clamp/adc.sch (KiCad schematic (older format))
At the start: 27 parts, among them P2 CONN_01X15, U10 LM741, U11 LM311N, U7 LM741, U8 DG444, U9 LM741

Commit message: add trigger pullup
Parts:
- added R?: 5k, symbol R
- R17: value 47 -> 1k
- R18: value 47k -> 10k
Connections:
- net +VE: now also R?.1
- net TRIGGER: now also R?.2
Changed lines of the file:
@@
 P 7850 2950
 F 0 "R18" V 7930 2950 50  0000 C CNN
-F 1 "47k" V 7850 2950 50  0000 C CNN
+F 1 "10k" V 7850 2950 50  0000 C CNN
 F 2 "" V 7780 2950 50  0000 C CNN
 F 3 "" H 7850 2950 50  0000 C CNN
@@
 P 7350 3950
 F 0 "R17" V 7430 3950 50  0000 C CNN
-F 1 "47" V 7350 3950 50  0000 C CNN
+F 1 "1k" V 7350 3950 50  0000 C CNN
 F 2 "" V 7280 3950 50  0000 C CNN
 F 3 "" H 7350 3950 50  0000 C CNN
@@
 Connection ~ 4200 2100
 Wire Wire Line
-	1650 2700 2900 2700
+	1650 2700 1950 2700
+Wire Wire Line
+	1950 2700 2900 2700
 Wire Wire Line
 	4100 3200 4450 3200
@@
 	4450 2900 4100 2900
 Wire Wire Line
-	2750 2100 4800 2100
-Wire Wire Line
-	5100 2100 5900 2100
+	2750 2100 4200 2100
+Wire Wire Line
+	4200 2100 4800 2100
+Wire Wire Line
+	5100 2100 5550 2100
+Wire Wire Line
+	5550 2100 5900 2100
 Wire Wire Line
 	2900 3200 2450 3200
@@
 	6100 2300 6100 2400
 Wire Wire Line
-	3750 4200 4200 4200
+	3750 4200 3850 4200
+Wire Wire Line
+	3850 4200 4200 4200
 Wire Wire Line
 	2900 4100 3150 4100
@@
 	3850 4200 3850 4850
 Wire Wire Line
-	2850 4300 3150 4300
+	2850 4300 3050 4300
+Wire Wire Line
+	3050 4300 3150 4300
 Wire Wire Line
 	3050 4300 3050 4850
@@
 	4200 2700 4200 4200
 Wire Wire Line
-	2750 2100 2750 3100
+	2750 2100 2750 2600
+Wire Wire Line
+	2750 2600 2750 3100
 Connection ~ 2750 2600
 Wire Wire Line
@@
 	1950 4300 2550 4300
 Wire Wire Line
-	6500 2000 7550 2000
-Wire Wire Line
-	6750 1650 6750 3100
+	6500 2000 6750 2000
+Wire Wire Line
+	6750 2000 7550 2000
+Wire Wire Line
+	6750 1650 6750 2000
+Wire Wire Line
+	6750 2000 6750 2800
+Wire Wire Line
+	6750 2800 6750 3100
 Wire Wire Line
 	5750 1900 5900 1900
@@
 	5550 2800 6000 2800
 Wire Wire Line
-	5550 2100 5550 3000
+	5550 2100 5550 2800
+Wire Wire Line
+	5550 2800 5550 3000
 Connection ~ 5550 2100
 Connection ~ 5550 2800
@@
 	7750 2400 7750 2500
 Wire Wire Line
-	8150 2100 8900 2100
-Wire Wire Line
-	8300 2100 8300 3550
+	8150 2100 8300 2100
+Wire Wire Line
+	8300 2100 8900 2100
+Wire Wire Line
+	8300 2100 8300 2950
+Wire Wire Line
+	8300 2950 8300 3250
+Wire Wire Line
+	8300 3250 8300 3550
 Connection ~ 8300 2100
 Wire Wire Line
-	7350 2200 7350 3800
+	7350 2200 7350 2950
+Wire Wire Line
+	7350 2950 7350 3250
+Wire Wire Line
+	7350 3250 7350 3550
+Wire Wire Line
+	7350 3550 7350 3800
 Connection ~ 7350 2950
 Wire Wire Line
@@
 	9100 2500 9100 2750
 Wire Wire Line
-	9500 2200 9900 2200
+	9500 2200 9750 2200
+Wire Wire Line
+	9750 2200 9900 2200
 Wire Wire Line
 	9200 2500 9200 2750
@@
 	4900 4450 4900 4550
 Wire Wire Line
-	4900 4550 6600 4550
+	4900 4550 5100 4550
+Wire Wire Line
+	5100 4550 5350 4550
+Wire Wire Line
+	5350 4550 5600 4550
+Wire Wire Line
+	5600 4550 5850 4550
+Wire Wire Line
+	5850 4550 6100 4550
+Wire Wire Line
+	6100 4550 6350 4550
+Wire Wire Line
+	6350 4550 6600 4550
 Connection ~ 5100 4550
 Text GLabel 5100 4850 3    60   Input ~ 0
@@
 	4900 5450 4900 5550
 Wire Wire Line
-	4900 5550 6600 5550
+	4900 5550 5100 5550
+Wire Wire Line
+	5100 5550 5350 5550
+Wire Wire Line
+	5350 5550 5600 5550
+Wire Wire Line
+	5600 5550 5850 5550
+Wire Wire Line
+	5850 5550 6100 5550
+Wire Wire Line
+	6100 5550 6350 5550
+Wire Wire Line
+	6350 5550 6600 5550
 Connection ~ 5100 5550
 Text GLabel 5100 5850 3    60   Input ~ 0
@@
 Text GLabel 6350 5850 3    60   Input ~ 0
 GND
+$Comp
+L R R?
+U 1 1 58620487
+P 9750 1850
+F 0 "R?" V 9830 1850 50  0000 C CNN
+F 1 "5k" V 9750 1850 50  0000 C CNN
+F 2 "" V 9680 1850 50  0000 C CNN
+F 3 "" H 9750 1850 50  0000 C CNN
+	1    9750 1850
+	1    0    0    -1
+$EndComp
+Wire Wire Line
+	9750 2000 9750 2200
+Connection ~ 9750 2200
+Text GLabel 9750 1550 1    60   Input ~ 0
++VE
+Wire Wire Line
+	9750 1550 9750 1700
 $EndSCHEMATC

Commit message: update
Parts:
- added P?: CONN_01X03, symbol CONN_01X03
Connections:
- net at C13.1, U10.3 (+), U8.15 (D3)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: now also P?.1 (P1)
- net at D5.2 (C), D6.1 (A), R18.1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: now also P?.3 (P3); no longer U11.2 (+)
- new net: P?.2 (P2), U11.2 (+)
Changed lines of the file:
@@
 	6500 2000 6750 2000
 Wire Wire Line
-	6750 2000 7550 2000
+	6750 2000 7100 2000
+Wire Wire Line
+	7100 2000 7550 2000
 Wire Wire Line
 	6750 1650 6750 2000
@@
 	8150 2100 8300 2100
 Wire Wire Line
-	8300 2100 8900 2100
+	8300 2100 8500 2100
+Wire Wire Line
+	8750 2100 8900 2100
 Wire Wire Line
 	8300 2100 8300 2950
@@
 Wire Wire Line
 	9750 1550 9750 1700
+$Comp
+L CONN_01X03 P?
+U 1 1 58621C5B
+P 9100 950
+F 0 "P?" H 9100 1150 50  0000 C CNN
+F 1 "CONN_01X03" V 9200 950 50  0000 C CNN
+F 2 "" H 9100 950 50  0000 C CNN
+F 3 "" H 9100 950 50  0000 C CNN
+	1    9100 950
+	1    0    0    -1
+$EndComp
+Wire Wire Line
+	7100 2000 7100 850
+Wire Wire Line
+	7100 850  8900 850
+Connection ~ 7100 2000
+Wire Wire Line
+	8900 950  8750 950
+Wire Wire Line
+	8750 950  8750 1300
+Wire Wire Line
+	8750 1300 8750 2100
+Wire Wire Line
+	8900 1050 8500 1050
+Wire Wire Line
+	8500 1050 8500 2100
 $EndSCHEMATC
