File: src/main2.kicad_pcb (KiCad board)
At the start: 2 copper layers, 102 parts, among them P1 CONN_01X12, P2 CONN_01X15, P3 CONN_01X03, P4 CONN_01X08, P501 CONN_01X07, Q1 2N3904, Q501 2N3904, Q502 2N3904, U1 LM741, U12 LTZ1000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

Commit message: 4 layer
Parts:
- Q501, Q502: value 2N3904 -> MMBT3904
- moved C502 13.7 mm to (112.5, 51.3)
- moved R506 13.7 mm to (101.3, 34.0)
- moved R507 13.7 mm to (101.3, 39.6)
- moved R508 13.7 mm to (101.3, 51.3)
- moved R509 13.7 mm to (101.3, 46.7)
- moved C505 13.7 mm to (117.3, 44.7)
- moved Q502 13.7 mm to (111.5, 36.8), turned to 90 degrees
- moved U502 13.7 mm to (112.3, 44.5)
- moved R501 13.5 mm to (85.6, 43.9)
- moved D501 11.9 mm to (88.6, 39.4)
- moved D502 11.1 mm to (91.7, 51.1)
- moved Q501 6.28 mm to (54.9, 35.3), turned to 90 degrees
- moved C503 6.18 mm to (49.0, 35.8)
- moved C501 4.44 mm to (54.4, 42.2)
- moved R502 4.44 mm to (54.4, 38.9)
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Connections:
- Q501 pad 1: Net-(Q501-Pad1) -> Net-(C501-Pad2)
- Q501 pad 2: Net-(C501-Pad2) -> Net-(Q501-Pad2)
- R501 pad 1: Net-(Q501-Pad1) -> Net-(Q501-Pad2)
- R506 pad 1: Net-(Q502-Pad1) -> Net-(Q502-Pad2)
- R507 pad 1: Net-(Q502-Pad1) -> Net-(Q502-Pad2)
- U502 pad 6: Net-(Q502-Pad2) -> Net-(Q502-Pad1)
Routing:
- net REF: track 76.6 -> 169.6 mm
- net 0V: track 110.5 -> 32.0 mm, vias 0 -> 5
- net (no net): track 46.0 -> 0.00 mm
- net +VE: track 444.0 -> 414.3 mm, vias 9 -> 13
- net Net-(Q502-Pad2): track 4.10 -> 21.1 mm
- net Net-(R502-Pad1): track 5.34 -> 19.9 mm
- net Net-(R505-Pad1): track 9.64 -> 23.5 mm
- net Net-(Q502-Pad1): track 14.3 -> 4.13 mm
- net Net-(R504-Pad2): track 0.00 -> 7.83 mm
- net Net-(C501-Pad2): track 10.6 -> 12.7 mm
- added copper zone on In2.Cu, net +VE
- added copper zone on In1.Cu, net 0V
Other:
- copper layers 2 -> 4
- net class Default: via_drill 0.75 -> 0.5

Commit message: update
Parts:
- added R510: R, Resistors_SMD:R_1206, F.Cu at (48.8, 41.1)
- moved D501 10.1 mm to (82.3, 47.2), turned to 90 degrees
- moved D502 5.95 mm to (87.1, 47.2)
- moved R501 5.57 mm to (80.5, 41.7), turned to 0 degrees
- moved C504 0.76 mm to (50.0, 49.5)
Connections:
- P501 pad 3: REF -> -VE
- P501 pad 4: 0V -> H-0V
- P501 pad 5: 0V -> REF
- R501 pad 2: 0V -> H-0V
- U501 pad 4: 0V -> -VE
- U502 pad 4: 0V -> -VE
Routing:
- net Net-(D501-Pad1): track 0.00 -> 41.5 mm
- net Net-(Q501-Pad2): track 0.00 -> 33.9 mm
- net Net-(C502-Pad1): track 11.5 -> 30.5 mm
- net REF: track 169.6 -> 178.6 mm
- net H-0V: track 0.00 -> 4.66 mm
- net -VE: track 370.4 -> 373.2 mm, vias 10 -> 11
- net 0V: track 32.0 -> 33.9 mm
- net +VE: track 414.3 -> 414.8 mm

Commit message: update
Parts:
- moved C502 2.55 mm to (110.0, 51.1), turned to 180 degrees
- moved R510 0.72 mm to (49.3, 41.7)
Routing:
- net H-0V: track 4.66 -> 80.5 mm
- net -VE: track 373.2 -> 377.0 mm, vias 11 -> 12
- net 0V: track 33.9 -> 35.2 mm, vias 5 -> 6
- net REF: track 178.6 -> 179.5 mm
- added copper zone on B.Cu, net -VE

Commit message: update
Routing:
- net REF: track 179.5 -> 215.4 mm
- net Net-(Q502-Pad2): track 20.6 -> 15.0 mm
- net Net-(C501-Pad2): track 12.7 -> 11.3 mm
- net Net-(R505-Pad1): track 23.5 -> 22.3 mm
- net H-0V: track 80.5 -> 80.0 mm
- net Net-(D501-Pad1): track 41.5 -> 41.0 mm
- net Net-(R502-Pad1): track 19.9 -> 19.4 mm

Commit message: looks good
Parts:
- moved D502 1.27 mm to (88.4, 47.2)
- moved R501 0.92 mm to (81.3, 42.2)
- moved P501 0.51 mm to (43.9, 35.8)
- moved RV501 0.25 mm to (64.5, 43.7)
- moved R504 0.25 mm to (66.5, 36.1)
- moved R505 0.25 mm to (66.5, 49.0)
Routing:
- net H-0V: track 80.0 -> 69.4 mm
- net REF: track 215.4 -> 210.7 mm
- net +VE: track 414.8 -> 418.5 mm, vias 13 -> 14
- net Net-(D501-Pad1): track 41.0 -> 37.5 mm
- net Net-(Q501-Pad2): track 33.7 -> 30.6 mm
- net 0V: track 35.4 -> 36.5 mm, vias 6 -> 8
