File: src/2dw232-ref.sch (KiCad schematic (older format))
At the start: 22 parts, among them Q501 2N3904, Q502 2N3904, U501 LM741, U502 LM741

Commit message: update
Parts:
- C501, C502: footprint (none) -> Capacitors_SMD:C_1206
- C503: value C -> 10uF; footprint (none) -> Capacitors_SMD:C_1206
- C504, C505: value C -> 0.1uF; footprint (none) -> Capacitors_SMD:C_1206
- D501, D502: footprint (none) -> Diodes_ThroughHole:Diode_DO-35_SOD27_Horizontal_RM10
- P501: renamed from P?; footprint (none) -> Pin_Headers:Pin_Header_Straight_1x07
- Q501, Q502: footprint (none) -> TO_SOT_Packages_SMD:SOT-23
- R501, R504, R505, R506, R507, R508, R509: footprint (none) -> Resistors_ThroughHole:Resistor_Horizontal_RM7mm
- R502, R503: footprint (none) -> Resistors_SMD:R_1206
- RV501: footprint (none) -> Potentiometers:Potentiometer_Bourns_3296Y_3-8Zoll_Angular_ScrewUp
- U501, U502: footprint (none) -> Housings_SOIC:SOIC-8_3.9x4.9mm_Pitch1.27mm
Changed lines of the file:
@@
 F 0 "U502" H 6450 2800 50  0000 L CNN
 F 1 "LM741" H 6450 2700 50  0000 L CNN
-F 2 "" H 6500 2600 50  0000 C CNN
+F 2 "Housings_SOIC:SOIC-8_3.9x4.9mm_Pitch1.27mm" H 6500 2600 50  0001 C CNN
 F 3 "" H 6600 2700 50  0000 C CNN
 	1    6450 2550
@@
 F 0 "R508" V 5430 3650 50  0000 C CNN
 F 1 "10k" V 5350 3650 50  0000 C CNN
-F 2 "" V 5280 3650 50  0000 C CNN
+F 2 "Resistors_ThroughHole:Resistor_Horizontal_RM7mm" V 5280 3650 50  0001 C CNN
 F 3 "" H 5350 3650 50  0000 C CNN
 	1    5350 3650
@@
 F 0 "R507" V 5430 2100 50  0000 C CNN
 F 1 "5.1k" V 5350 2100 50  0000 C CNN
-F 2 "" V 5280 2100 50  0000 C CNN
+F 2 "Resistors_ThroughHole:Resistor_Horizontal_RM7mm" V 5280 2100 50  0001 C CNN
 F 3 "" H 5350 2100 50  0000 C CNN
 	1    5350 2100
@@
 	7050 2550 6750 2550
 Wire Wire Line
-	4750 1750 5350 1750
-Wire Wire Line
-	5350 1750 7600 1750
+	4750 1750 7600 1750
 Wire Wire Line
 	5350 1750 5350 1950
 Wire Wire Line
-	5350 2250 5350 2650
-Wire Wire Line
-	5350 2650 5350 3000
+	5350 2250 5350 3000
 Text GLabel 6350 2200 1    60   Input ~ 0
 +VE
@@
 0V
 Wire Wire Line
-	6350 2850 6350 4150
-Wire Wire Line
-	6350 4150 6350 4350
-Wire Wire Line
-	5350 2650 5750 2650
-Wire Wire Line
-	5750 2650 6150 2650
+	6350 2850 6350 4350
+Wire Wire Line
+	5350 2650 6150 2650
 Connection ~ 5350 2650
 $Comp
@@
 F 0 "D501" H 4750 2800 50  0000 C CNN
 F 1 "ZENER" H 4750 2600 50  0000 C CNN
-F 2 "" H 4750 2700 50  0000 C CNN
+F 2 "Diodes_ThroughHole:Diode_DO-35_SOD27_Horizontal_RM10" H 4750 2700 50  0001 C CNN
 F 3 "" H 4750 2700 50  0000 C CNN
 	1    4750 2700
@@
 $EndComp
 Wire Wire Line
-	3850 2450 4750 2450
-Wire Wire Line
-	4750 2450 6150 2450
-Wire Wire Line
-	4750 2250 4750 2450
-Wire Wire Line
-	4750 2450 4750 2500
-Wire Wire Line
-	1400 4150 2600 4150
-Wire Wire Line
-	2600 4150 3850 4150
-Wire Wire Line
-	3850 4150 4750 4150
-Wire Wire Line
-	4750 4150 5350 4150
-Wire Wire Line
-	5350 4150 5750 4150
-Wire Wire Line
-	5750 4150 6350 4150
+	3850 2450 6150 2450
+Wire Wire Line
+	4750 2250 4750 2500
+Wire Wire Line
+	1400 4150 6350 4150
 Connection ~ 6350 4150
 Connection ~ 5350 4150
@@
 F 0 "R506" V 4830 2100 50  0000 C CNN
 F 1 "120" V 4750 2100 50  0000 C CNN
-F 2 "" V 4680 2100 50  0000 C CNN
+F 2 "Resistors_ThroughHole:Resistor_Horizontal_RM7mm" V 4680 2100 50  0001 C CNN
 F 3 "" H 4750 2100 50  0000 C CNN
 	1    4750 2100
@@
 F 0 "Q502" H 7350 2625 40  0000 C CNN
 F 1 "2N3904" H 7325 2550 40  0000 L CNN
-F 2 "" H 7200 2550 60  0001 C CNN
+F 2 "TO_SOT_Packages_SMD:SOT-23" H 7200 2550 60  0001 C CNN
 F 3 "" H 7200 2550 60  0001 C CNN
 	1    7200 2550
@@
 F 0 "C502" H 5775 3500 50  0000 L CNN
 F 1 "10p" H 5775 3300 50  0000 L CNN
-F 2 "" H 5788 3250 50  0000 C CNN
+F 2 "Capacitors_SMD:C_1206" H 5788 3250 50  0001 C CNN
 F 3 "" H 5750 3400 50  0000 C CNN
 	1    5750 3400
@@
 F 0 "D502" H 4750 3450 50  0000 C CNN
 F 1 "ZENER" H 4750 3250 50  0000 C CNN
-F 2 "" H 4750 3350 50  0000 C CNN
+F 2 "Diodes_ThroughHole:Diode_DO-35_SOD27_Horizontal_RM10" H 4750 3350 50  0001 C CNN
 F 3 "" H 4750 3350 50  0000 C CNN
 	1    4750 3350
@@
 $EndComp
 Wire Wire Line
-	4750 2900 4750 3000
-Wire Wire Line
-	4750 3000 4750 3150
+	4750 2900 4750 3150
 $Comp
 L R R504
@@
 F 0 "R504" V 3930 2700 50  0000 C CNN
 F 1 "1k" V 3850 2700 50  0000 C CNN
-F 2 "" V 3780 2700 50  0000 C CNN
+F 2 "Resistors_ThroughHole:Resistor_Horizontal_RM7mm" V 3780 2700 50  0001 C CNN
 F 3 "" H 3850 2700 50  0000 C CNN
 	1    3850 2700
@@
 $EndComp
 Wire Wire Line
-	3850 2200 3850 2450
-Wire Wire Line
-	3850 2450 3850 2550
+	3850 2200 3850 2550
 $Comp
 L POT RV501
@@
 F 0 "RV501" H 3850 3120 50  0000 C CNN
 F 1 "1k" H 3850 3200 50  0000 C CNN
-F 2 "" H 3850 3200 50  0000 C CNN
+F 2 "Potentiometers:Potentiometer_Bourns_3296Y_3-8Zoll_Angular_ScrewUp" H 3850 3200 50  0001 C CNN
 F 3 "" H 3850 3200 50  0000 C CNN
 	1    3850 3200
@@
 F 0 "R505" V 3930 3800 50  0000 C CNN
 F 1 "10k" V 3850 3800 50  0000 C CNN
-F 2 "" V 3780 3800 50  0000 C CNN
+F 2 "Resistors_ThroughHole:Resistor_Horizontal_RM7mm" V 3780 3800 50  0001 C CNN
 F 3 "" H 3850 3800 50  0000 C CNN
 	1    3850 3800
@@
 	3850 2850 3850 3050
 Wire Wire Line
-	3850 3350 3850 3400
-Wire Wire Line
-	3850 3400 3850 3650
+	3850 3350 3850 3650
 Connection ~ 4750 4150
 Wire Wire Line
-	2800 3400 3850 3400
-Wire Wire Line
-	3850 3400 4000 3400
+	2800 3400 4000 3400
 Connection ~ 3850 3400
 Wire Wire Line
@@
 F 0 "U501" H 2500 3750 50  0000 L CNN
 F 1 "LM741" H 2500 3650 50  0000 L CNN
-F 2 "" H 2550 3550 50  0000 C CNN
+F 2 "Housings_SOIC:SOIC-8_3.9x4.9mm_Pitch1.27mm" H 2550 3550 50  0001 C CNN
 F 3 "" H 2650 3650 50  0000 C CNN
 	1    2500 3500
@@
 F 0 "R503" V 3380 3000 50  0000 C CNN
 F 1 "10k" V 3300 3000 50  0000 C CNN
-F 2 "" V 3230 3000 50  0000 C CNN
+F 2 "Resistors_SMD:R_1206" V 3230 3000 50  0001 C CNN
 F 3 "" H 3300 3000 50  0000 C CNN
 	1    3300 3000
@@
 $EndComp
 Wire Wire Line
-	2500 3000 3000 3000
-Wire Wire Line
-	3000 3000 3150 3000
+	2500 3000 3150 3000
 Wire Wire Line
 	3000 3000 3000 3600
@@
 F 0 "R502" V 2430 3000 50  0000 C CNN
 F 1 "1M" V 2350 3000 50  0000 C CNN
-F 2 "" V 2280 3000 50  0000 C CNN
+F 2 "Resistors_SMD:R_1206" V 2280 3000 50  0001 C CNN
 F 3 "" H 2350 3000 50  0000 C CNN
 	1    2350 3000
@@
 F 0 "C501" H 1925 3350 50  0000 L CNN
 F 1 "10uF" H 1925 3150 50  0000 L CNN
-F 2 "" H 1938 3100 50  0000 C CNN
+F 2 "Capacitors_SMD:C_1206" H 1938 3100 50  0001 C CNN
 F 3 "" H 1900 3250 50  0000 C CNN
 	1    1900 3250
@@
 	1900 3400 1900 3500
 Wire Wire Line
-	1650 3500 1900 3500
-Wire Wire Line
-	1900 3500 2200 3500
+	1650 3500 2200 3500
 Text GLabel 2600 2700 1    60   Input ~ 0
 +VE
@@
 F 0 "Q501" H 1650 3575 40  0000 C CNN
 F 1 "2N3904" H 1625 3500 40  0000 L CNN
-F 2 "" H 1500 3500 60  0001 C CNN
+F 2 "TO_SOT_Packages_SMD:SOT-23" H 1500 3500 60  0001 C CNN
 F 3 "" H 1500 3500 60  0001 C CNN
 	1    1500 3500
@@
 F 0 "R501" V 1480 3850 50  0000 C CNN
 F 1 "200R" V 1400 3850 50  0000 C CNN
-F 2 "" V 1330 3850 50  0000 C CNN
+F 2 "Resistors_ThroughHole:Resistor_Horizontal_RM7mm" V 1330 3850 50  0001 C CNN
 F 3 "" H 1400 3850 50  0000 C CNN
 	1    1400 3850
@@
 F 0 "R509" V 5430 3150 50  0000 C CNN
 F 1 "0" V 5350 3150 50  0000 C CNN
-F 2 "" V 5280 3150 50  0000 C CNN
+F 2 "Resistors_ThroughHole:Resistor_Horizontal_RM7mm" V 5280 3150 50  0001 C CNN
 F 3 "" H 5350 3150 50  0000 C CNN
 	1    5350 3150
@@
 P 1850 1250
 F 0 "C503" H 1875 1350 50  0000 L CNN
-F 1 "C" H 1875 1150 50  0000 L CNN
-F 2 "" H 1888 1100 50  0000 C CNN
+F 1 "10uF" H 1875 1150 50  0000 L CNN
+F 2 "Capacitors_SMD:C_1206" H 1888 1100 50  0001 C CNN
 F 3 "" H 1850 1250 50  0000 C CNN
 	1    1850 1250
@@
 P 2150 1250
 F 0 "C504" H 2175 1350 50  0000 L CNN
-F 1 "C" H 2175 1150 50  0000 L CNN
-F 2 "" H 2188 1100 50  0000 C CNN
+F 1 "0.1uF" H 2175 1150 50  0000 L CNN
+F 2 "Capacitors_SMD:C_1206" H 2188 1100 50  0001 C CNN
 F 3 "" H 2150 1250 50  0000 C CNN
 	1    2150 1250
@@
 P 2450 1250
 F 0 "C505" H 2475 1350 50  0000 L CNN
-F 1 "C" H 2475 1150 50  0000 L CNN
-F 2 "" H 2488 1100 50  0000 C CNN
+F 1 "0.1uF" H 2475 1150 50  0000 L CNN
+F 2 "Capacitors_SMD:C_1206" H 2488 1100 50  0001 C CNN
 F 3 "" H 2450 1250 50  0000 C CNN
 	1    2450 1250
@@
 	1850 950  1850 1100
 Wire Wire Line
-	1850 1100 2150 1100
-Wire Wire Line
-	2150 1100 2450 1100
-Wire Wire Line
-	1850 1400 2150 1400
-Wire Wire Line
-	2150 1400 2450 1400
+	1850 1100 2450 1100
+Wire Wire Line
+	1850 1400 2450 1400
 Connection ~ 2150 1100
 Connection ~ 2150 1400
@@
 	1850 1400 1850 1600
 $Comp
-L CONN_01X07 P?
+L CONN_01X07 P501
 U 1 1 5883052B
 P 3500 1200
-F 0 "P?" H 3500 1600 50  0000 C CNN
+F 0 "P501" H 3500 1600 50  0000 C CNN
 F 1 "CONN_01X07" V 3600 1200 50  0000 C CNN
-F 2 "" H 3500 1200 50  0000 C CNN
+F 2 "Pin_Headers:Pin_Header_Straight_1x07" H 3500 1200 50  0001 C CNN
 F 3 "" H 3500 1200 50  0000 C CNN
 	1    3500 1200

Commit message: 4 layer
Parts:
- removed Q501, Q502: 2N3904, TO_SOT_Packages_SMD:SOT-23, symbol 2N3904
- added Q501, Q502: MMBT3904, TO_SOT_Packages_SMD:SOT-23, symbol MMBT3904
- R504, R505, R506, R507, R508, R509: footprint Resistors_ThroughHole:Resistor_Horizontal_RM7mm -> Resistors_ThroughHole:Resistor_TO-220_Vertical
Connections:
- net +VE: now also Q501.3 (C), Q502.3 (C)
- net at U502.6: now also Q502.1 (B)
- net at R506.1, R507.1: now also Q502.2 (E)
- net at C501.2, U501.6: now also Q501.1 (B)
- net at R501.1: now also Q501.2 (E)
Changed lines of the file:
@@
 F 0 "R508" V 5430 3650 50  0000 C CNN
 F 1 "10k" V 5350 3650 50  0000 C CNN
-F 2 "Resistors_ThroughHole:Resistor_Horizontal_RM7mm" V 5280 3650 50  0001 C CNN
+F 2 "Resistors_ThroughHole:Resistor_TO-220_Vertical" V 5280 3650 50  0001 C CNN
 F 3 "" H 5350 3650 50  0000 C CNN
 	1    5350 3650
@@
 F 0 "R507" V 5430 2100 50  0000 C CNN
 F 1 "5.1k" V 5350 2100 50  0000 C CNN
-F 2 "Resistors_ThroughHole:Resistor_Horizontal_RM7mm" V 5280 2100 50  0001 C CNN
+F 2 "Resistors_ThroughHole:Resistor_TO-220_Vertical" V 5280 2100 50  0001 C CNN
 F 3 "" H 5350 2100 50  0000 C CNN
 	1    5350 2100
@@
 $EndComp
 Wire Wire Line
-	7050 2550 6750 2550
-Wire Wire Line
-	4750 1750 7600 1750
+	4750 1750 7800 1750
 Wire Wire Line
 	5350 1750 5350 1950
@@
 F 0 "R506" V 4830 2100 50  0000 C CNN
 F 1 "120" V 4750 2100 50  0000 C CNN
-F 2 "Resistors_ThroughHole:Resistor_Horizontal_RM7mm" V 4680 2100 50  0001 C CNN
+F 2 "Resistors_ThroughHole:Resistor_TO-220_Vertical" V 4680 2100 50  0001 C CNN
 F 3 "" H 4750 2100 50  0000 C CNN
 	1    4750 2100
@@
 Connection ~ 5350 1750
 Connection ~ 4750 2450
-$Comp
-L 2N3904 Q502
-U 1 1 588188E4
-P 7200 2550
-F 0 "Q502" H 7350 2625 40  0000 C CNN
-F 1 "2N3904" H 7325 2550 40  0000 L CNN
-F 2 "TO_SOT_Packages_SMD:SOT-23" H 7200 2550 60  0001 C CNN
-F 3 "" H 7200 2550 60  0001 C CNN
-	1    7200 2550
-	1    0    0    -1
-$EndComp
 Text GLabel 7300 2200 1    60   Input ~ 0
 +VE
@@
 F 0 "R504" V 3930 2700 50  0000 C CNN
 F 1 "1k" V 3850 2700 50  0000 C CNN
-F 2 "Resistors_ThroughHole:Resistor_Horizontal_RM7mm" V 3780 2700 50  0001 C CNN
+F 2 "Resistors_ThroughHole:Resistor_TO-220_Vertical" V 3780 2700 50  0001 C CNN
 F 3 "" H 3850 2700 50  0000 C CNN
 	1    3850 2700
@@
 F 0 "R505" V 3930 3800 50  0000 C CNN
 F 1 "10k" V 3850 3800 50  0000 C CNN
-F 2 "Resistors_ThroughHole:Resistor_Horizontal_RM7mm" V 3780 3800 50  0001 C CNN
+F 2 "Resistors_ThroughHole:Resistor_TO-220_Vertical" V 3780 3800 50  0001 C CNN
 F 3 "" H 3850 3800 50  0000 C CNN
 	1    3850 3800
@@
 	1900 3400 1900 3500
 Wire Wire Line
-	1650 3500 2200 3500
+	1700 3500 2200 3500
 Text GLabel 2600 2700 1    60   Input ~ 0
 +VE
@@
 	2600 2700 2600 3200
 Connection ~ 3850 4150
-$Comp
-L 2N3904 Q501
-U 1 1 5881F2EF
-P 1500 3500
-F 0 "Q501" H 1650 3575 40  0000 C CNN
-F 1 "2N3904" H 1625 3500 40  0000 L CNN
-F 2 "TO_SOT_Packages_SMD:SOT-23" H 1500 3500 60  0001 C CNN
-F 3 "" H 1500 3500 60  0001 C CNN
-	1    1500 3500
-	-1   0    0    -1
-$EndComp
 Connection ~ 1900 3500
 Text GLabel 1400 2700 1    60   Input ~ 0
@@
 $EndComp
 Wire Wire Line
-	7600 1750 7600 3000
-Wire Wire Line
-	7600 3000 7300 3000
+	7800 1750 7800 3000
+Wire Wire Line
+	7800 3000 7300 3000
 Wire Wire Line
 	7300 3000 7300 2750
@@
 F 0 "R509" V 5430 3150 50  0000 C CNN
 F 1 "0" V 5350 3150 50  0000 C CNN
-F 2 "Resistors_ThroughHole:Resistor_Horizontal_RM7mm" V 5280 3150 50  0001 C CNN
+F 2 "Resistors_ThroughHole:Resistor_TO-220_Vertical" V 5280 3150 50  0001 C CNN
 F 3 "" H 5350 3150 50  0000 C CNN
 	1    5350 3150
@@
 Wire Wire Line
 	3700 1500 3950 1500
+$Comp
+L MMBT3904 Q502
+U 1 1 58835E41
+P 7200 2550
+F 0 "Q502" H 7400 2625 50  0000 L CNN
+F 1 "MMBT3904" H 7400 2550 50  0000 L CNN
+F 2 "TO_SOT_Packages_SMD:SOT-23" H 7400 2475 50  0000 L CIN
+F 3 "" H 7200 2550 50  0000 L CNN
+	1    7200 2550
+	1    0    0    -1
+$EndComp
+Wire Wire Line
+	7000 2550 6750 2550
+$Comp
+L MMBT3904 Q501
+U 1 1 58836CA2
+P 1500 3500
+F 0 "Q501" H 1700 3575 50  0000 L CNN
+F 1 "MMBT3904" H 1700 3500 50  0000 L CNN
+F 2 "TO_SOT_Packages_SMD:SOT-23" H 1700 3425 50  0000 L CIN
+F 3 "" H 1500 3500 50  0000 L CNN
+	1    1500 3500
+	-1   0    0    -1
+$EndComp
 $EndSCHEMATC

Commit message: update
Parts:
- added R510: R, Resistors_SMD:R_1206, symbol R
Connections:
- net 0V: now also R510.2; no longer P501.4 (P4), P501.5 (P5), R501.2, U501.4 (V-), U502.4 (V-)
- net REF: now also P501.5 (P5); no longer P501.3 (P3)
- new net -VE: P501.3 (P3), U501.4 (V-), U502.4 (V-)
- new net H-0V: P501.4 (P4), R501.2, R510.1
Other:
- moved on the sheet: R501
Changed lines of the file:
@@
 Wire Wire Line
 	6350 2200 6350 2250
-Text GLabel 6350 4350 3    60   Input ~ 0
-0V
-Wire Wire Line
-	6350 2850 6350 4350
+Text GLabel 5750 4400 3    60   Input ~ 0
+0V
 Wire Wire Line
 	5350 2650 6150 2650
@@
 	4750 2250 4750 2500
 Wire Wire Line
-	1400 4150 6350 4150
-Connection ~ 6350 4150
+	3850 4150 5750 4150
 Connection ~ 5350 4150
 $Comp
@@
 L R R501
 U 1 1 58821BA0
-P 1400 3850
-F 0 "R501" V 1480 3850 50  0000 C CNN
-F 1 "200R" V 1400 3850 50  0000 C CNN
-F 2 "Resistors_ThroughHole:Resistor_Horizontal_RM7mm" V 1330 3850 50  0001 C CNN
-F 3 "" H 1400 3850 50  0000 C CNN
-	1    1400 3850
+P 1400 4000
+F 0 "R501" V 1480 4000 50  0000 C CNN
+F 1 "200R" V 1400 4000 50  0000 C CNN
+F 2 "Resistors_ThroughHole:Resistor_Horizontal_RM7mm" V 1330 4000 50  0001 C CNN
+F 3 "" H 1400 4000 50  0000 C CNN
+	1    1400 4000
 	1    0    0    -1
 $EndComp
@@
 Wire Wire Line
 	7300 2200 7300 2350
-Connection ~ 2600 4150
 NoConn ~ 6450 2850
 NoConn ~ 6550 2850
@@
 NoConn ~ 2500 3800
 Wire Wire Line
-	1400 4000 1400 4150
-Wire Wire Line
 	4750 3550 4750 4150
 Wire Wire Line
@@
 Wire Wire Line
 	3850 3950 3850 4150
-Wire Wire Line
-	2600 3800 2600 4150
 Connection ~ 8050 6800
 Wire Wire Line
-	5750 3550 5750 4150
+	5750 3550 5750 4400
 Connection ~ 5750 4150
 $Comp
@@
 REF
 Connection ~ 3850 2450
-Text GLabel 3950 1100 2    60   Input ~ 0
+Text GLabel 3950 1300 2    60   Input ~ 0
 REF
-Wire Wire Line
-	3700 1100 3950 1100
-Text GLabel 3950 1200 2    60   Input ~ 0
-0V
-Text GLabel 3950 1300 2    60   Input ~ 0
-0V
 Text GLabel 3950 1400 2    60   Input ~ 0
 0V
 Text GLabel 3950 1500 2    60   Input ~ 0
 0V
-Wire Wire Line
-	3700 1200 3950 1200
-Wire Wire Line
-	3700 1300 3950 1300
 Wire Wire Line
 	3700 1400 3950 1400
@@
 	-1   0    0    -1
 $EndComp
+Wire Wire Line
+	1400 3850 1400 3700
+Wire Wire Line
+	1400 4150 1400 4300
+Text GLabel 1400 4300 3    60   Input ~ 0
+H-0V
+Text GLabel 3950 1100 2    60   Input ~ 0
+-VE
+Wire Wire Line
+	3700 1100 3950 1100
+Text GLabel 3950 1200 2    60   Input ~ 0
+H-0V
+Wire Wire Line
+	3700 1200 3950 1200
+Wire Wire Line
+	3700 1300 3950 1300
+Text GLabel 2600 4050 3    60   Input ~ 0
+-VE
+Wire Wire Line
+	2600 3800 2600 4050
+Text GLabel 6350 3050 3    60   Input ~ 0
+-VE
+Wire Wire Line
+	6350 2850 6350 3050
+Text GLabel 5900 1050 2    60   Input ~ 0
+H-0V
+Text GLabel 5100 1050 0    60   Input ~ 0
+0V
+$Comp
+L R R510
+U 1 1 5883C0FE
+P 5500 1050
+F 0 "R510" V 5580 1050 50  0000 C CNN
+F 1 "R" V 5500 1050 50  0000 C CNN
+F 2 "Resistors_SMD:R_1206" V 5430 1050 50  0001 C CNN
+F 3 "" H 5500 1050 50  0000 C CNN
+	1    5500 1050
+	0    1    1    0
+$EndComp
+Wire Wire Line
+	5100 1050 5350 1050
+Wire Wire Line
+	5650 1050 5900 1050
 $EndSCHEMATC

Commit message: update
Other:
- moved on the sheet: R501
Changed lines of the file:
@@
 $EndComp
 Wire Wire Line
-	4750 1750 7800 1750
+	4750 1750 5350 1750
+Wire Wire Line
+	5350 1750 7800 1750
 Wire Wire Line
 	5350 1750 5350 1950
 Wire Wire Line
-	5350 2250 5350 3000
+	5350 2250 5350 2650
+Wire Wire Line
+	5350 2650 5350 3000
 Text GLabel 6350 2200 1    60   Input ~ 0
 +VE
@@
 0V
 Wire Wire Line
-	5350 2650 6150 2650
+	5350 2650 5750 2650
+Wire Wire Line
+	5750 2650 6150 2650
 Connection ~ 5350 2650
 $Comp
@@
 $EndComp
 Wire Wire Line
-	3850 2450 6150 2450
-Wire Wire Line
-	4750 2250 4750 2500
-Wire Wire Line
-	3850 4150 5750 4150
+	3850 2450 4750 2450
+Wire Wire Line
+	4750 2450 6150 2450
+Wire Wire Line
+	4750 2250 4750 2450
+Wire Wire Line
+	4750 2450 4750 2500
+Wire Wire Line
+	3850 4150 4750 4150
+Wire Wire Line
+	4750 4150 5350 4150
+Wire Wire Line
+	5350 4150 5750 4150
 Connection ~ 5350 4150
 $Comp
@@
 $EndComp
 Wire Wire Line
-	4750 2900 4750 3150
+	4750 2900 4750 3000
+Wire Wire Line
+	4750 3000 4750 3150
 $Comp
 L R R504
@@
 $EndComp
 Wire Wire Line
-	3850 2200 3850 2550
+	3850 2200 3850 2450
+Wire Wire Line
+	3850 2450 3850 2550
 $Comp
 L POT RV501
@@
 	3850 2850 3850 3050
 Wire Wire Line
-	3850 3350 3850 3650
+	3850 3350 3850 3400
+Wire Wire Line
+	3850 3400 3850 3650
 Connection ~ 4750 4150
 Wire Wire Line
-	2800 3400 4000 3400
+	2800 3400 3850 3400
+Wire Wire Line
+	3850 3400 4000 3400
 Connection ~ 3850 3400
 Wire Wire Line
@@
 $EndComp
 Wire Wire Line
-	2500 3000 3150 3000
+	2500 3000 3000 3000
+Wire Wire Line
+	3000 3000 3150 3000
 Wire Wire Line
 	3000 3000 3000 3600
@@
 	1900 3400 1900 3500
 Wire Wire Line
-	1700 3500 2200 3500
+	1700 3500 1900 3500
+Wire Wire Line
+	1900 3500 2200 3500
 Text GLabel 2600 2700 1    60   Input ~ 0
 +VE
 Wire Wire Line
 	2600 2700 2600 3200
-Connection ~ 3850 4150
 Connection ~ 1900 3500
 Text GLabel 1400 2700 1    60   Input ~ 0
@@
 L R R501
 U 1 1 58821BA0
-P 1400 4000
-F 0 "R501" V 1480 4000 50  0000 C CNN
-F 1 "200R" V 1400 4000 50  0000 C CNN
-F 2 "Resistors_ThroughHole:Resistor_Horizontal_RM7mm" V 1330 4000 50  0001 C CNN
-F 3 "" H 1400 4000 50  0000 C CNN
-	1    1400 4000
+P 1400 3950
+F 0 "R501" V 1480 3950 50  0000 C CNN
+F 1 "200R" V 1400 3950 50  0000 C CNN
+F 2 "Resistors_ThroughHole:Resistor_Horizontal_RM7mm" V 1330 3950 50  0001 C CNN
+F 3 "" H 1400 3950 50  0000 C CNN
+	1    1400 3950
 	1    0    0    -1
 $EndComp
@@
 Connection ~ 8050 6800
 Wire Wire Line
-	5750 3550 5750 4400
+	5750 3550 5750 4150
+Wire Wire Line
+	5750 4150 5750 4400
 Connection ~ 5750 4150
 $Comp
@@
 	1850 950  1850 1100
 Wire Wire Line
-	1850 1100 2450 1100
-Wire Wire Line
-	1850 1400 2450 1400
+	1850 1100 2150 1100
+Wire Wire Line
+	2150 1100 2450 1100
+Wire Wire Line
+	1850 1400 2150 1400
+Wire Wire Line
+	2150 1400 2450 1400
 Connection ~ 2150 1100
 Connection ~ 2150 1400
@@
 $EndComp
 Wire Wire Line
-	1400 3850 1400 3700
-Wire Wire Line
-	1400 4150 1400 4300
-Text GLabel 1400 4300 3    60   Input ~ 0
+	1400 3800 1400 3700
+Wire Wire Line
+	1400 4100 1400 4250
+Text GLabel 1400 4250 3    60   Input ~ 0
 H-0V
 Text GLabel 3950 1100 2    60   Input ~ 0

Commit message: just the dw232
Changed lines of the file:
@@
 $EndComp
 Wire Wire Line
-	4750 1750 5350 1750
-Wire Wire Line
-	5350 1750 7800 1750
+	4750 1750 7800 1750
 Wire Wire Line
 	5350 1750 5350 1950
 Wire Wire Line
-	5350 2250 5350 2650
-Wire Wire Line
-	5350 2650 5350 3000
+	5350 2250 5350 3000
 Text GLabel 6350 2200 1    60   Input ~ 0
 +VE
@@
 0V
 Wire Wire Line
-	5350 2650 5750 2650
-Wire Wire Line
-	5750 2650 6150 2650
+	5350 2650 6150 2650
 Connection ~ 5350 2650
 $Comp
@@
 $EndComp
 Wire Wire Line
-	3850 2450 4750 2450
-Wire Wire Line
-	4750 2450 6150 2450
-Wire Wire Line
-	4750 2250 4750 2450
-Wire Wire Line
-	4750 2450 4750 2500
-Wire Wire Line
-	3850 4150 4750 4150
-Wire Wire Line
-	4750 4150 5350 4150
-Wire Wire Line
-	5350 4150 5750 4150
+	3850 2450 6150 2450
+Wire Wire Line
+	4750 2250 4750 2500
+Wire Wire Line
+	3850 4150 5750 4150
 Connection ~ 5350 4150
 $Comp
@@
 $EndComp
 Wire Wire Line
-	4750 2900 4750 3000
-Wire Wire Line
-	4750 3000 4750 3150
+	4750 2900 4750 3150
 $Comp
 L R R504
@@
 $EndComp
 Wire Wire Line
-	3850 2200 3850 2450
-Wire Wire Line
-	3850 2450 3850 2550
+	3850 2200 3850 2550
 $Comp
 L POT RV501
@@
 	3850 2850 3850 3050
 Wire Wire Line
-	3850 3350 3850 3400
-Wire Wire Line
-	3850 3400 3850 3650
+	3850 3350 3850 3650
 Connection ~ 4750 4150
 Wire Wire Line
-	2800 3400 3850 3400
-Wire Wire Line
-	3850 3400 4000 3400
+	2800 3400 4000 3400
 Connection ~ 3850 3400
 Wire Wire Line
@@
 $EndComp
 Wire Wire Line
-	2500 3000 3000 3000
-Wire Wire Line
-	3000 3000 3150 3000
+	2500 3000 3150 3000
 Wire Wire Line
 	3000 3000 3000 3600
@@
 	1900 3400 1900 3500
 Wire Wire Line
-	1700 3500 1900 3500
-Wire Wire Line
-	1900 3500 2200 3500
+	1700 3500 2200 3500
 Text GLabel 2600 2700 1    60   Input ~ 0
 +VE
@@
 Connection ~ 8050 6800
 Wire Wire Line
-	5750 3550 5750 4150
-Wire Wire Line
-	5750 4150 5750 4400
+	5750 3550 5750 4400
 Connection ~ 5750 4150
 $Comp
@@
 	1850 950  1850 1100
 Wire Wire Line
-	1850 1100 2150 1100
-Wire Wire Line
-	2150 1100 2450 1100
-Wire Wire Line
-	1850 1400 2150 1400
-Wire Wire Line
-	2150 1400 2450 1400
+	1850 1100 2450 1100
+Wire Wire Line
+	1850 1400 2450 1400
 Connection ~ 2150 1100
 Connection ~ 2150 1400

Commit message: update
Parts:
- removed D501, D502: ZENER, Diodes_ThroughHole:Diode_DO-35_SOD27_Horizontal_RM10, symbol ZENER
- removed R501: 200R, Resistors_ThroughHole:Resistor_Horizontal_RM7mm, symbol R
- removed R509: 0, Resistors_ThroughHole:Resistor_TO-220_Vertical, symbol R
- added RV502: 1k, Potentiometers:Potentiometer_Bourns_3296Y_3-8Zoll_Angular_ScrewUp, symbol POT
- added U503: 2DW232, symbol 2DW232
Connections:
- net 0V: now also U503.2 (A2)
- net H-0V: now also U503.5 (R2)
- net REF: now also Q502.2 (E), R506.1, R507.1; no longer R506.2, U502.3 (+)
- net at C502.1, R507.2, U502.2 (-): now also RV502.1
- net at R508.1: now also RV502.2, RV502.3
- net at R503.2: now also U503.3 (K)
- net at Q501.2 (E): now also U503.4 (R1)
- new net: R506.2, U502.3 (+), U503.1 (A1)
Other:
- moved on the sheet: C502, Q502, R504, R505, R506, R507, R508, U502
