File: src/2dw232-ref.sch (KiCad schematic (older format))
At the start: 21 parts, among them P501 CONN_01X07, Q501 MMBT3904, Q502 MMBT3904, U501 LM741, U502 LM741, U503 2DW232

Commit message: update
Parts:
- added C506: 10uF, Capacitors_SMD:C_1206, symbol C
- added C507, C508: 0.1uF, Capacitors_SMD:C_1206, symbol C
- U503: footprint (none) -> footprint:TO-5_Housing_2DW232_5Pin
Connections:
- net +VE: now also C506.1, C507.1, C508.1; no longer C503.1, C504.1, C505.1
- net -VE: now also C503.1, C504.1, C505.1
- net 0V: now also C506.2, C507.2, C508.2
- net REF: now also R506.2, U502.3 (+), U503.1 (A1); no longer Q502.2 (E), R504.1, R506.1, R507.1
- new net: Q502.2 (E), R504.1, R506.1, R507.1
Changed lines of the file:
@@
 $EndComp
 Wire Wire Line
-	3850 1750 9100 1750
+	3850 1750 8750 1750
 Wire Wire Line
 	6300 1750 6300 1950
@@
 $EndComp
 Text GLabel 1850 950  1    60   Input ~ 0
-+VE
+-VE
 Wire Wire Line
 	1850 950  1850 1100
@@
 Wire Wire Line
 	3700 1000 3950 1000
-Text GLabel 9100 1750 2    60   Input ~ 0
-REF
 Text GLabel 3950 1300 2    60   Input ~ 0
 REF
@@
 F 0 "U503" H 5150 3800 50  0000 L CNN
 F 1 "2DW232" H 5150 3200 50  0000 L CNN
-F 2 "" V 5000 3550 50  0000 C CNN
+F 2 "footprint:TO-5_Housing_2DW232_5Pin" V 5000 3550 50  0001 C CNN
 F 3 "" V 5000 3550 50  0000 C CNN
 	1    5200 3150
@@
 Wire Wire Line
 	5700 2700 5700 4500
-Connection ~ 8750 1750
 Wire Wire Line
 	5600 2900 5850 2900
@@
 	6450 3400 6300 3400
 Connection ~ 6300 3400
+$Comp
+L C C506
+U 1 1 5883AA71
+P 850 1250
+F 0 "C506" H 875 1350 50  0000 L CNN
+F 1 "10uF" H 875 1150 50  0000 L CNN
+F 2 "Capacitors_SMD:C_1206" H 888 1100 50  0001 C CNN
+F 3 "" H 850 1250 50  0000 C CNN
+	1    850  1250
+	1    0    0    -1
+$EndComp
+$Comp
+L C C507
+U 1 1 5883AA77
+P 1150 1250
+F 0 "C507" H 1175 1350 50  0000 L CNN
+F 1 "0.1uF" H 1175 1150 50  0000 L CNN
+F 2 "Capacitors_SMD:C_1206" H 1188 1100 50  0001 C CNN
+F 3 "" H 1150 1250 50  0000 C CNN
+	1    1150 1250
+	1    0    0    -1
+$EndComp
+$Comp
+L C C508
+U 1 1 5883AA7D
+P 1450 1250
+F 0 "C508" H 1475 1350 50  0000 L CNN
+F 1 "0.1uF" H 1475 1150 50  0000 L CNN
+F 2 "Capacitors_SMD:C_1206" H 1488 1100 50  0001 C CNN
+F 3 "" H 1450 1250 50  0000 C CNN
+	1    1450 1250
+	1    0    0    -1
+$EndComp
+Text GLabel 850  950  1    60   Input ~ 0
++VE
+Wire Wire Line
+	850  950  850  1100
+Wire Wire Line
+	850  1100 1450 1100
+Wire Wire Line
+	850  1400 1450 1400
+Connection ~ 1150 1100
+Connection ~ 1150 1400
+Text GLabel 850  1600 3    60   Input ~ 0
+0V
+Wire Wire Line
+	850  1400 850  1600
+Text GLabel 5200 1550 1    60   Input ~ 0
+REF
+Wire Wire Line
+	5200 1550 5200 2450
+Connection ~ 5200 2450
 $EndSCHEMATC

Commit message: update
Other:
- moved on the sheet: P501, R506, R507
Changed lines of the file:
@@
 L R R507
 U 1 1 588184DE
-P 6300 2100
-F 0 "R507" V 6380 2100 50  0000 C CNN
-F 1 "5.1k" V 6300 2100 50  0000 C CNN
-F 2 "Resistors_ThroughHole:Resistor_TO-220_Vertical" V 6230 2100 50  0001 C CNN
-F 3 "" H 6300 2100 50  0000 C CNN
-	1    6300 2100
-	1    0    0    -1
-$EndComp
-Wire Wire Line
-	3850 1750 8750 1750
-Wire Wire Line
-	6300 1750 6300 1950
-Wire Wire Line
-	6300 2250 6300 3050
+P 6300 2150
+F 0 "R507" V 6380 2150 50  0000 C CNN
+F 1 "5.1k" V 6300 2150 50  0000 C CNN
+F 2 "Resistors_ThroughHole:Resistor_TO-220_Vertical" V 6230 2150 50  0001 C CNN
+F 3 "" H 6300 2150 50  0000 C CNN
+	1    6300 2150
+	1    0    0    -1
+$EndComp
+Wire Wire Line
+	3850 1750 4450 1750
+Wire Wire Line
+	4450 1750 6300 1750
+Wire Wire Line
+	6300 1750 8750 1750
+Wire Wire Line
+	6300 1750 6300 2000
+Wire Wire Line
+	6300 2300 6300 2650
+Wire Wire Line
+	6300 2650 6300 3050
 Text GLabel 7300 2200 1    60   Input ~ 0
 +VE
@@
 0V
 Wire Wire Line
-	6300 2650 7100 2650
+	6300 2650 6700 2650
+Wire Wire Line
+	6700 2650 7100 2650
 Connection ~ 6300 2650
 Wire Wire Line
-	4450 2450 7100 2450
-Wire Wire Line
-	3850 4150 6700 4150
+	4450 2450 4150 2450
+Wire Wire Line
+	4150 2450 7100 2450
+Wire Wire Line
+	3850 4150 4450 4150
+Wire Wire Line
+	4450 4150 6300 4150
+Wire Wire Line
+	6300 4150 6700 4150
 Connection ~ 6300 4150
 $Comp
 L R R506
 U 1 1 5881872C
-P 4450 2100
-F 0 "R506" V 4530 2100 50  0000 C CNN
-F 1 "120" V 4450 2100 50  0000 C CNN
-F 2 "Resistors_ThroughHole:Resistor_TO-220_Vertical" V 4380 2100 50  0001 C CNN
-F 3 "" H 4450 2100 50  0000 C CNN
-	1    4450 2100
+P 4450 2150
+F 0 "R506" V 4530 2150 50  0000 C CNN
+F 1 "120" V 4450 2150 50  0000 C CNN
+F 2 "Resistors_ThroughHole:Resistor_TO-220_Vertical" V 4380 2150 50  0001 C CNN
+F 3 "" H 4450 2150 50  0000 C CNN
+	1    4450 2150
 	1    0    0    -1
 $EndComp
@@
 	3850 2700 3850 3050
 Wire Wire Line
-	3850 3350 3850 3600
-Wire Wire Line
-	2800 3400 4000 3400
+	3850 3350 3850 3400
+Wire Wire Line
+	3850 3400 3850 3600
+Wire Wire Line
+	2800 3400 3850 3400
+Wire Wire Line
+	3850 3400 4000 3400
 Connection ~ 3850 3400
 Wire Wire Line
@@
 $EndComp
 Wire Wire Line
-	2500 3000 3150 3000
+	2500 3000 3000 3000
+Wire Wire Line
+	3000 3000 3150 3000
 Wire Wire Line
 	3000 3000 3000 3600
@@
 	1900 3400 1900 3500
 Wire Wire Line
-	1700 3500 2200 3500
+	1700 3500 1900 3500
+Wire Wire Line
+	1900 3500 2200 3500
 Text GLabel 2600 2700 1    60   Input ~ 0
 +VE
@@
 	3850 3900 3850 4150
 Wire Wire Line
-	6700 3550 6700 4400
+	6700 3550 6700 4150
+Wire Wire Line
+	6700 4150 6700 4400
 Connection ~ 6700 4150
 Wire Wire Line
-	6300 3350 6300 3600
+	6300 3350 6300 3400
+Wire Wire Line
+	6300 3400 6300 3600
 $Comp
 L C C503
@@
 	1850 950  1850 1100
 Wire Wire Line
-	1850 1100 2450 1100
-Wire Wire Line
-	1850 1400 2450 1400
+	1850 1100 2150 1100
+Wire Wire Line
+	2150 1100 2450 1100
+Wire Wire Line
+	1850 1400 2150 1400
+Wire Wire Line
+	2150 1400 2450 1400
 Connection ~ 2150 1100
 Connection ~ 2150 1400
@@
 L CONN_01X07 P501
 U 1 1 5883052B
-P 3500 1200
-F 0 "P501" H 3500 1600 50  0000 C CNN
-F 1 "CONN_01X07" V 3600 1200 50  0000 C CNN
-F 2 "Pin_Headers:Pin_Header_Straight_1x07" H 3500 1200 50  0001 C CNN
-F 3 "" H 3500 1200 50  0000 C CNN
-	1    3500 1200
+P 6800 1150
+F 0 "P501" H 6800 1550 50  0000 C CNN
+F 1 "CONN_01X07" V 6900 1150 50  0000 C CNN
+F 2 "Pin_Headers:Pin_Header_Straight_1x07" H 6800 1150 50  0001 C CNN
+F 3 "" H 6800 1150 50  0000 C CNN
+	1    6800 1150
 	-1   0    0    -1
 $EndComp
-Text GLabel 3950 900  2    60   Input ~ 0
-+VE
-Wire Wire Line
-	3700 900  3950 900
-Text GLabel 3950 1000 2    60   Input ~ 0
-0V
-Wire Wire Line
-	3700 1000 3950 1000
-Text GLabel 3950 1300 2    60   Input ~ 0
+Text GLabel 7250 850  2    60   Input ~ 0
++VE
+Wire Wire Line
+	7000 850  7250 850
+Text GLabel 7250 950  2    60   Input ~ 0
+0V
+Wire Wire Line
+	7000 950  7250 950
+Text GLabel 7250 1250 2    60   Input ~ 0
 REF
-Text GLabel 3950 1400 2    60   Input ~ 0
-0V
-Text GLabel 3950 1500 2    60   Input ~ 0
-0V
-Wire Wire Line
-	3700 1400 3950 1400
-Wire Wire Line
-	3700 1500 3950 1500
+Text GLabel 7250 1350 2    60   Input ~ 0
+0V
+Text GLabel 7250 1450 2    60   Input ~ 0
+0V
+Wire Wire Line
+	7000 1350 7250 1350
+Wire Wire Line
+	7000 1450 7250 1450
 $Comp
 L MMBT3904 Q502
@@
 Text GLabel 5850 2900 2    60   Input ~ 0
 H-0V
-Text GLabel 3950 1100 2    60   Input ~ 0
+Text GLabel 7250 1050 2    60   Input ~ 0
 -VE
 Wire Wire Line
-	3700 1100 3950 1100
-Text GLabel 3950 1200 2    60   Input ~ 0
+	7000 1050 7250 1050
+Text GLabel 7250 1150 2    60   Input ~ 0
 H-0V
 Wire Wire Line
-	3700 1200 3950 1200
-Wire Wire Line
-	3700 1300 3950 1300
+	7000 1150 7250 1150
+Wire Wire Line
+	7000 1250 7250 1250
 Text GLabel 2600 4050 3    60   Input ~ 0
 -VE
@@
 	4450 2600 4600 2600
 Wire Wire Line
-	4450 2250 4450 2600
-Wire Wire Line
-	4450 1750 4450 1950
+	4450 2300 4450 2450
+Wire Wire Line
+	4450 2450 4450 2600
+Wire Wire Line
+	4450 1750 4450 2000
 Connection ~ 4450 1750
 Connection ~ 4450 2450
@@
 	850  950  850  1100
 Wire Wire Line
-	850  1100 1450 1100
-Wire Wire Line
-	850  1400 1450 1400
+	850  1100 1150 1100
+Wire Wire Line
+	1150 1100 1450 1100
+Wire Wire Line
+	850  1400 1150 1400
+Wire Wire Line
+	1150 1400 1450 1400
 Connection ~ 1150 1100
 Connection ~ 1150 1400
@@
 Wire Wire Line
 	850  1400 850  1600
-Text GLabel 5200 1550 1    60   Input ~ 0
+Text GLabel 4150 1550 1    60   Input ~ 0
 REF
 Wire Wire Line
-	5200 1550 5200 2450
-Connection ~ 5200 2450
+	4150 1550 4150 2450
 $EndSCHEMATC
