File: src/2dw232-ref.sch (KiCad schematic (older format))
At the start: 24 parts, among them P501 CONN_01X07, Q501 MMBT3904, Q502 MMBT3904, U501 LM741, U502 LM741, U503 2DW232

Commit message: update
Changed lines of the file:
@@
 $Descr A4 11693 8268
 encoding utf-8
-Sheet 2 2
+Sheet 2 3
 Title ""
 Date ""
@@
 $EndComp
 Wire Wire Line
-	3850 1750 4450 1750
-Wire Wire Line
-	4450 1750 6300 1750
-Wire Wire Line
-	6300 1750 8750 1750
+	3850 1750 8750 1750
 Wire Wire Line
 	6300 1750 6300 2000
 Wire Wire Line
-	6300 2300 6300 2650
-Wire Wire Line
-	6300 2650 6300 3050
+	6300 2300 6300 3050
 Text GLabel 7300 2200 1    60   Input ~ 0
 +VE
@@
 0V
 Wire Wire Line
-	6300 2650 6700 2650
-Wire Wire Line
-	6700 2650 7100 2650
+	6300 2650 7100 2650
 Connection ~ 6300 2650
 Wire Wire Line
-	4450 2450 4150 2450
-Wire Wire Line
 	4150 2450 7100 2450
 Wire Wire Line
-	3850 4150 4450 4150
-Wire Wire Line
-	4450 4150 6300 4150
-Wire Wire Line
-	6300 4150 6700 4150
+	3850 4150 6700 4150
 Connection ~ 6300 4150
 $Comp
@@
 	3850 2700 3850 3050
 Wire Wire Line
-	3850 3350 3850 3400
-Wire Wire Line
-	3850 3400 3850 3600
-Wire Wire Line
-	2800 3400 3850 3400
-Wire Wire Line
-	3850 3400 4000 3400
+	3850 3350 3850 3600
+Wire Wire Line
+	2800 3400 4000 3400
 Connection ~ 3850 3400
 Wire Wire Line
@@
 $EndComp
 Wire Wire Line
-	2500 3000 3000 3000
-Wire Wire Line
-	3000 3000 3150 3000
+	2500 3000 3150 3000
 Wire Wire Line
 	3000 3000 3000 3600
@@
 	1900 3400 1900 3500
 Wire Wire Line
-	1700 3500 1900 3500
-Wire Wire Line
-	1900 3500 2200 3500
+	1700 3500 2200 3500
 Text GLabel 2600 2700 1    60   Input ~ 0
 +VE
@@
 	3850 3900 3850 4150
 Wire Wire Line
-	6700 3550 6700 4150
-Wire Wire Line
-	6700 4150 6700 4400
+	6700 3550 6700 4400
 Connection ~ 6700 4150
 Wire Wire Line
-	6300 3350 6300 3400
-Wire Wire Line
-	6300 3400 6300 3600
+	6300 3350 6300 3600
 $Comp
 L C C503
@@
 	1850 950  1850 1100
 Wire Wire Line
-	1850 1100 2150 1100
-Wire Wire Line
-	2150 1100 2450 1100
-Wire Wire Line
-	1850 1400 2150 1400
-Wire Wire Line
-	2150 1400 2450 1400
+	1850 1100 2450 1100
+Wire Wire Line
+	1850 1400 2450 1400
 Connection ~ 2150 1100
 Connection ~ 2150 1400
@@
 Wire Wire Line
 	2600 3800 2600 4050
-Text GLabel 7300 3050 3    60   Input ~ 0
+Text GLabel 7300 3000 3    60   Input ~ 0
 -VE
 Wire Wire Line
-	7300 2850 7300 3050
+	7300 2850 7300 3000
 Text GLabel 5800 1050 2    60   Input ~ 0
 H-0V
@@
 	4450 2600 4600 2600
 Wire Wire Line
-	4450 2300 4450 2450
-Wire Wire Line
-	4450 2450 4450 2600
+	4450 2300 4450 2600
 Wire Wire Line
 	4450 1750 4450 2000
@@
 	850  950  850  1100
 Wire Wire Line
-	850  1100 1150 1100
-Wire Wire Line
-	1150 1100 1450 1100
-Wire Wire Line
-	850  1400 1150 1400
-Wire Wire Line
-	1150 1400 1450 1400
+	850  1100 1450 1100
+Wire Wire Line
+	850  1400 1450 1400
 Connection ~ 1150 1100
 Connection ~ 1150 1400

Commit message: change schematic from 0V to AGND
Connections:
- net 0V renamed AGND
- net H-0V renamed H-GND
Changed lines of the file:
@@
 	7300 2200 7300 2250
 Text GLabel 6700 4400 3    60   Input ~ 0
-0V
+AGND
 Wire Wire Line
 	6300 2650 7100 2650
@@
 Connection ~ 2150 1400
 Text GLabel 1850 1600 3    60   Input ~ 0
-0V
+AGND
 Wire Wire Line
 	1850 1400 1850 1600
@@
 	7000 850  7250 850
 Text GLabel 7250 950  2    60   Input ~ 0
-0V
+AGND
 Wire Wire Line
 	7000 950  7250 950
@@
 REF
 Text GLabel 7250 1350 2    60   Input ~ 0
-0V
+AGND
 Text GLabel 7250 1450 2    60   Input ~ 0
-0V
+AGND
 Wire Wire Line
 	7000 1350 7250 1350
@@
 	1400 3700 1400 4500
 Text GLabel 5850 2900 2    60   Input ~ 0
-H-0V
+H-GND
 Text GLabel 7250 1050 2    60   Input ~ 0
 -VE
@@
 	7000 1050 7250 1050
 Text GLabel 7250 1150 2    60   Input ~ 0
-H-0V
+H-GND
 Wire Wire Line
 	7000 1150 7250 1150
@@
 	7300 2850 7300 3000
 Text GLabel 5800 1050 2    60   Input ~ 0
-H-0V
+H-GND
 Text GLabel 5150 1050 0    60   Input ~ 0
-0V
+AGND
 $Comp
 L R R510
@@
 Connection ~ 1150 1400
 Text GLabel 850  1600 3    60   Input ~ 0
-0V
+AGND
 Wire Wire Line
 	850  1400 850  1600
