File: src/main.kicad_pcb (KiCad board)
At the start: 2 copper layers, 80 parts, among them P1 CONN_01X12, P2 CONN_01X15, P3 CONN_01X03, P4 CONN_01X08, Q1 2N3904, U1 LM741, U12 LTZ1000, U13 LM741, U14 LM741, U2 LM741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

Commit message: update
Routing:
- net REF: track 48.2 -> 71.2 mm
- net Net-(C30-Pad1): track 75.6 -> 59.4 mm
- net +VE: track 397.5 -> 382.3 mm
- net Net-(D8-Pad1): track 22.2 -> 12.3 mm
- net Net-(R1-Pad1): track 9.75 -> 0.00 mm
- net Net-(D2-Pad2): track 8.79 -> 2.92 mm
- net Net-(R10-Pad1): track 5.44 -> 0.00 mm, vias 1 -> 0
- net OUT: track 183.7 -> 179.9 mm
- net I-FB: track 12.5 -> 9.45 mm
- net Net-(R11-Pad1): track 7.11 -> 4.06 mm
- net Net-(R12-Pad2): track 2.67 -> 0.00 mm
- net GND: track 103.9 -> 101.6 mm
- net Net-(R24-Pad2): track 29.8 -> 27.8 mm
- net -VE: track 372.0 -> 370.4 mm
- net Net-(C26-Pad1): track 56.5 -> 55.2 mm
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
Commit message: update
Parts:
- removed C1, C10, C11, C12, C14, C15, C16, C17, C18, C19, C2, C20, C21, C22, C23, C24, C25, C3, C4, C5, C6, C7, C8, C9: C, Capacitors_SMD:C_1206
- removed C26: 22nF, Capacitors_SMD:C_1206
- removed C27, C33: 10uF, Capacitors_SMD:C_1206
- removed C28, C29, C30, C31, C32, C34: 0.1uF, Capacitors_SMD:C_1206
- removed D1, D2, D3, D4, D7, D8: 1N4148, Diodes_SMD:MiniMELF_Standard
- removed D5, D6: 1N4148, Diodes_ThroughHole:Diode_DO-35_SOD27_Horizontal_RM10
- removed P1: CONN_01X12, Pin_Headers:Pin_Header_Straight_1x12
- removed P2: CONN_01X15, Pin_Headers:Pin_Header_Straight_1x15
- removed P3: CONN_01X03, Pin_Headers:Pin_Header_Straight_1x03
- removed P4: CONN_01X08, Pin_Headers:Pin_Header_Straight_1x08
- removed Q1: 2N3904, TO_SOT_Packages_SMD:SOT-23
- removed R1, R10, R11, R12, R13, R14, R15, R2, R3, R4, R5, R6, R7, R8, R9: R, Resistors_SMD:R_1206
- removed R20: 120, Resistors_ThroughHole:Resistor_TO-220_Vertical
- removed R21, r1: 70k, Resistors_ThroughHole:Resistor_TO-220_Vertical
- removed R22: 1k, Resistors_SMD:R_1206
- removed R23: 1M, Resistors_SMD:R_1206
- removed R24: 10k, Resistors_SMD:R_1206
- removed R25: 12k, Resistors_ThroughHole:Resistor_TO-220_Vertical
- removed R26: 1k, Resistors_ThroughHole:Resistor_TO-220_Vertical
- removed R28: 0, Resistors_SMD:R_1206
- removed U1, U2, U3, U4, U5, U6, U7: LM741, Housings_SOIC:SOIC-8_3.9x4.9mm_Pitch1.27mm
- removed U12: LTZ1000, footprint:TO-5_Housing_8Pin
- removed U13, U14: LM741, SMD_Packages:SOIC-8-N
- added C501: 10uF, Capacitors_SMD:C_1206, F.Cu at (54.4, 42.2)
- added C502: 10p, Capacitors_SMD:C_1206, F.Cu at (110.0, 51.1)
- added C503: 10uF, Capacitors_SMD:C_1206, F.Cu at (49.0, 35.8)
- added C504: 0.1uF, Capacitors_SMD:C_1206, F.Cu at (50.0, 49.5)
- added C505: 0.1uF, Capacitors_SMD:C_1206, F.Cu at (117.3, 44.7)
- added D501: ZENER, Diodes_ThroughHole:Diode_DO-35_SOD27_Horizontal_RM10, F.Cu at (82.3, 47.2)
- added D502: ZENER, Diodes_ThroughHole:Diode_DO-35_SOD27_Horizontal_RM10, F.Cu at (88.4, 47.2)
- added P501: CONN_01X07, Pin_Headers:Pin_Header_Straight_1x07, F.Cu at (43.9, 35.8)
- added Q501: MMBT3904, TO_SOT_Packages_SMD:SOT-23, F.Cu at (54.9, 35.3)
- added Q502: MMBT3904, TO_SOT_Packages_SMD:SOT-23, F.Cu at (111.5, 36.8)
- added R501: 200R, Resistors_ThroughHole:Resistor_Horizontal_RM7mm, F.Cu at (81.3, 42.2)
- added R502: 1M, Resistors_SMD:R_1206, F.Cu at (54.4, 38.9)
- added R503: 10k, Resistors_SMD:R_1206, F.Cu at (58.7, 35.8)
- added R504: 1k, Resistors_ThroughHole:Resistor_TO-220_Vertical, F.Cu at (66.5, 36.1)
- added R505: 10k, Resistors_ThroughHole:Resistor_TO-220_Vertical, F.Cu at (66.5, 49.0)
- added R506: 120, Resistors_ThroughHole:Resistor_TO-220_Vertical, F.Cu at (101.3, 34.0)
- added R507: 5.1k, Resistors_ThroughHole:Resistor_TO-220_Vertical, F.Cu at (101.3, 39.6)
- added R508: 10k, Resistors_ThroughHole:Resistor_TO-220_Vertical, F.Cu at (101.3, 51.3)
- added R509: 0, Resistors_ThroughHole:Resistor_TO-220_Vertical, F.Cu at (101.3, 46.7)
- added R510: R, Resistors_SMD:R_1206, F.Cu at (49.3, 41.7)
- added RV501: 1k, Potentiometers:Potentiometer_Bourns_3296Y_3-8Zoll_Angular_ScrewUp, F.Cu at (64.5, 43.7)
- added U501: LM741, Housings_SOIC:SOIC-8_3.9x4.9mm_Pitch1.27mm, F.Cu at (55.1, 48.3)
- added U502: LM741, Housings_SOIC:SOIC-8_3.9x4.9mm_Pitch1.27mm, F.Cu at (112.3, 44.5)
Routing:
- net -VE: track 370.4 -> 6.64 mm, vias 10 -> 2
- net +VE: track 382.3 -> 36.2 mm, vias 9 -> 5
- net OUT: track 179.9 -> 0.00 mm
- net GND: track 101.6 -> 0.00 mm, vias 19 -> 0
- net Net-(C29-Pad2): track 71.0 -> 0.00 mm, vias 2 -> 0
- net H-0V: track 0.00 -> 69.4 mm
- net REF: track 71.2 -> 139.6 mm, vias 2 -> 0
- net Net-(C30-Pad1): track 59.4 -> 0.00 mm
- net GND-H: track 57.2 -> 0.00 mm
- net Net-(C26-Pad1): track 55.2 -> 0.00 mm
- net Net-(D501-Pad1): track 0.00 -> 37.5 mm
- net 0V: track 0.00 -> 36.5 mm, vias 0 -> 8
- net Net-(R20-Pad1): track 34.4 -> 0.00 mm, vias 2 -> 0
- net Net-(Q501-Pad2): track 0.00 -> 30.6 mm
- net Net-(C502-Pad1): track 0.00 -> 30.2 mm
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- added copper zone on In2.Cu, net +VE
- added copper zone on B.Cu, net -VE
- added copper zone on In1.Cu, net 0V
- removed copper zone on F.Cu, net (none)
Other:
- copper layers 2 -> 4
- net class Default: via_dia 1.75 -> 1; via_drill 0.75 -> 0.5
- board text removed: "+I"
- board text removed: "+V"
- board text removed: "+VE"
- board text removed: "-I"
- board text removed: "-V"
- board text removed: "-VE"
- board text removed: "GND"
- board text removed: "I-FB"
- board text removed: "I-SET"
- board text removed: "OUT"
- board text removed: "REF"
- board text removed: "V-SET"
- board text removed: "V_FB"

Commit message: remove pin header vias
Routing:
- net +VE: track 36.2 -> 32.3 mm, vias 5 -> 4
- net 0V: track 36.5 -> 32.8 mm, vias 8 -> 7
- net REF: track 139.6 -> 141.1 mm
Changed lines of the file:
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@@
     (thickness 1.6)
     (drawings 0)
-    (tracks 206)
+    (tracks 201)
     (zones 0)
     (modules 23)
@@
   (segment (start 235.458 80.518) (end 235.204 80.518) (width 0.75) (layer B.Cu) (net 0))
   (segment (start 235.204 80.518) (end 235.458 80.518) (width 0.75) (layer B.Cu) (net 0))
-  (segment (start 43.942 35.814) (end 43.942 32.258) (width 0.75) (layer F.Cu) (net 1) (status 10))
-  (via (at 44.196 32.004) (size 1) (drill 0.5) (layers F.Cu B.Cu) (net 1))
-  (segment (start 43.942 32.258) (end 44.196 32.004) (width 0.75) (layer F.Cu) (net 1))
   (segment (start 117.348 43.204) (end 117.348 40.132) (width 0.75) (layer F.Cu) (net 1) (status 10))
   (via (at 117.348 40.132) (size 1) (drill 0.5) (layers F.Cu B.Cu) (net 1))
@@
   (via (at 57.15 53.594) (size 1) (drill 0.5) (layers F.Cu B.Cu) (net 2))
   (segment (start 57.023 53.467) (end 57.15 53.594) (width 0.75) (layer F.Cu) (net 2))
-  (segment (start 46.863 47.879) (end 46.863 53.975) (width 0.75) (layer F.Cu) (net 4))
-  (segment (start 46.863 53.975) (end 48.275998 55.387998) (width 0.75) (layer F.Cu) (net 4))
-  (segment (start 79.502 55.387998) (end 48.275998 55.387998) (width 0.75) (layer F.Cu) (net 4))
-  (segment (start 44.958 45.974) (end 46.863 47.879) (width 0.75) (layer F.Cu) (net 4) (status 10))
+  (segment (start 46.99 46.99) (end 46.99 53.848) (width 0.75) (layer F.Cu) (net 4))
+  (segment (start 48.783998 55.387998) (end 46.99 53.594) (width 0.75) (layer F.Cu) (net 4))
+  (segment (start 79.502 55.387998) (end 48.783998 55.387998) (width 0.75) (layer F.Cu) (net 4))
+  (segment (start 45.974 45.974) (end 43.942 45.974) (width 0.75) (layer F.Cu) (net 4) (status 10))
+  (segment (start 45.974 45.974) (end 46.99 46.99) (width 0.75) (layer F.Cu) (net 4))
   (segment (start 69.088 36.068) (end 69.088 36.576) (width 0.75) (layer F.Cu) (net 4) (status 30))
   (segment (start 69.088 36.576) (end 79.502 46.99) (width 0.75) (layer F.Cu) (net 4) (status 10))
@@
   (segment (start 98.806 46.736) (end 98.806 47.752) (width 0.75) (layer F.Cu) (net 7) (status 30))
   (segment (start 98.806 46.736) (end 98.806 39.624) (width 0.75) (layer F.Cu) (net 7) (status 30))
-  (segment (start 43.942 51.054) (end 43.942 54.356) (width 0.75) (layer F.Cu) (net 8) (status 10))
-  (via (at 44.196 54.61) (size 1) (drill 0.5) (layers F.Cu B.Cu) (net 8))
-  (segment (start 43.942 54.356) (end 44.196 54.61) (width 0.75) (layer F.Cu) (net 8))
   (segment (start 49.022 37.314) (end 50.062 37.314) (width 0.75) (layer F.Cu) (net 8) (status 10))
   (via (at 52.07 35.306) (size 1) (drill 0.5) (layers F.Cu B.Cu) (net 8))

Commit message: update
Parts:
- removed D501, D502: ZENER, Diodes_ThroughHole:Diode_DO-35_SOD27_Horizontal_RM10
- removed R501: 200R, Resistors_ThroughHole:Resistor_Horizontal_RM7mm
- removed R509: 0, Resistors_ThroughHole:Resistor_TO-220_Vertical
- added RV502: 1k, Potentiometers:Potentiometer_Bourns_3296Y_3-8Zoll_Angular_ScrewUp, F.Cu at (0.00, 0.00)
- added U503: 2DW232, footprint:TO-5_Housing_2DW232_5Pin, F.Cu at (0.00, 0.00)
Connections:
- Q502 pad 2: Net-(Q502-Pad2) -> REF
- R506 pad 1: Net-(Q502-Pad2) -> REF
- R506 pad 2: REF -> Net-(R506-Pad2)
- R507 pad 1: Net-(Q502-Pad2) -> REF
- U502 pad 3: REF -> Net-(R506-Pad2)
Routing:
- net Net-(R506-Pad2): track 0.00 -> 33.1 mm
- net REF: track 141.1 -> 123.1 mm
- net Net-(Q502-Pad2): track 15.0 -> 0.00 mm
- net 0V: track 32.8 -> 29.5 mm, vias 7 -> 6
- net (no net): track 17.3 -> 20.6 mm, vias 0 -> 1

Commit message: update
Parts:
- moved RV502 109.1 mm to (98.3, 47.2), turned to 270 degrees
- moved U503 94.9 mm to (85.1, 41.9)
- moved Q502 0.51 mm to (111.5, 36.3)
Routing:
- net Net-(Q501-Pad2): track 30.6 -> 41.5 mm
- net Net-(R503-Pad2): track 37.5 -> 27.6 mm
- net REF: track 123.1 -> 131.1 mm, vias 0 -> 2
- net Net-(R506-Pad2): track 33.1 -> 38.1 mm
- net Net-(R508-Pad1): track 4.57 -> 8.16 mm
- net (no net): track 20.6 -> 17.3 mm, vias 1 -> 0
- net Net-(C502-Pad1): track 30.2 -> 30.9 mm
- net Net-(Q502-Pad1): track 4.13 -> 4.64 mm
- net +VE: track 32.3 -> 32.8 mm
- net H-0V: track 69.4 -> 69.6 mm, vias 0 -> 4

Commit message: update
Parts:
- moved Q502 15.2 mm to (126.7, 36.3)
- moved C505 14.7 mm to (132.1, 44.7)
- moved C502 14.7 mm to (124.7, 51.1)
- moved R506 14.7 mm to (116.1, 34.0)
- moved R507 14.7 mm to (116.1, 39.6)
- moved R508 14.7 mm to (116.1, 51.3)
- moved RV502 14.7 mm to (113.0, 47.2)
- moved U502 14.7 mm to (127.0, 44.5)
- moved U503 5.59 mm to (90.7, 41.9)
Routing:
- net REF: track 131.1 -> 155.4 mm
- net (no net): track 17.3 -> 0.38 mm
- net Net-(R506-Pad2): track 38.1 -> 28.2 mm
- net Net-(R503-Pad2): track 27.6 -> 35.8 mm
- net Net-(C502-Pad1): track 30.9 -> 23.8 mm
- net Net-(Q501-Pad2): track 41.5 -> 47.1 mm
- net Net-(Q502-Pad1): track 4.64 -> 9.05 mm
- net H-0V: track 69.6 -> 71.9 mm, vias 4 -> 2
- net 0V: track 29.3 -> 28.2 mm
- removed copper zone on B.Cu, net GND

Commit message: update
Parts:
- moved R510 0.25 mm to (49.0, 41.7)
Routing:
- net Net-(R506-Pad2): track 28.2 -> 49.6 mm, vias 0 -> 1
- net REF: track 155.4 -> 139.6 mm, vias 2 -> 0
- net 0V: track 28.2 -> 14.6 mm, vias 6 -> 4
- net Net-(C502-Pad1): track 23.8 -> 32.1 mm
- net Net-(R503-Pad2): track 35.8 -> 36.8 mm
- net Net-(Q501-Pad2): track 47.1 -> 47.8 mm

Commit message: update
Parts:
- added C506: 10uF, Capacitors_SMD:C_1206, F.Cu at (51.1, 35.3)
- added C507: 0.1uF, Capacitors_SMD:C_1206, F.Cu at (50.3, 48.5)
- added C508: 0.1uF, Capacitors_SMD:C_1206, F.Cu at (122.4, 45.0)
- moved C504 10.7 mm to (60.7, 48.5), turned to 90 degrees
- moved C502 3.30 mm to (128.0, 51.1), turned to 0 degrees
- moved C503 0.92 mm to (48.3, 35.3)
- moved C505 0.36 mm to (131.8, 45.0), turned to 90 degrees
Connections:
- C503 pad 1: +VE -> -VE
- C504 pad 1: +VE -> -VE
- C505 pad 1: +VE -> -VE
- Q502 pad 2: REF -> Net-(Q502-Pad2)
- R504 pad 1: REF -> Net-(Q502-Pad2)
- R506 pad 1: REF -> Net-(Q502-Pad2)
- R506 pad 2: Net-(R506-Pad2) -> REF
- R507 pad 1: REF -> Net-(Q502-Pad2)
- U502 pad 3: Net-(R506-Pad2) -> REF
- U503 pad 1: Net-(R506-Pad2) -> REF
Routing:
- net Net-(R506-Pad2): track 49.6 -> 0.00 mm, vias 1 -> 0
- net Net-(Q502-Pad2): track 0.00 -> 36.8 mm
- net REF: track 139.6 -> 126.9 mm, vias 0 -> 1
- net -VE: track 6.64 -> 16.5 mm, vias 2 -> 3
- net 0V: track 14.6 -> 23.8 mm, vias 4 -> 6
- net +VE: track 32.6 -> 25.4 mm, vias 4 -> 5
- net H-0V: track 71.6 -> 74.2 mm, vias 2 -> 0
- net Net-(R505-Pad1): track 22.7 -> 23.7 mm
- net Net-(C502-Pad1): track 32.1 -> 33.1 mm
- net Net-(R503-Pad2): track 36.8 -> 36.0 mm
