File: src/main.kicad_pcb (KiCad board)
At the start: 4 copper layers, 24 parts, among them P501 CONN_01X07, Q501 MMBT3904, Q502 MMBT3904, U501 LM741, U502 LM741, U503 2DW232

Commit message: update
Routing:
- net Net-(Q502-Pad2): track 36.8 -> 88.6 mm, vias 0 -> 2
- net H-0V: track 74.2 -> 72.8 mm
- net Net-(Q501-Pad2): track 47.8 -> 48.4 mm, vias 0 -> 2
- net REF: track 126.9 -> 126.5 mm, vias 1 -> 0

Commit message: update
Routing:
- net REF: track 126.5 -> 122.5 mm
- net Net-(R503-Pad2): track 36.5 -> 35.3 mm
- net Net-(Q501-Pad2): track 48.4 -> 47.5 mm
- net Net-(Q502-Pad2): vias 2 -> 0
Changed lines of the file:
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@@
     (links 50)
     (no_connects 0)
-    (area 0 0 0 0)
+    (area 41.402 29.718 209.413002 133.975002)
     (thickness 1.6)
     (drawings 0)
-    (tracks 208)
+    (tracks 207)
     (zones 0)
     (modules 24)
@@
   (via (at 57.15 53.594) (size 1) (drill 0.5) (layers F.Cu B.Cu) (net 2))
   (segment (start 57.023 53.467) (end 57.15 53.594) (width 0.75) (layer F.Cu) (net 2))
-  (segment (start 96.012 42.672) (end 96.012 55.626) (width 0.75) (layer F.Cu) (net 3))
-  (segment (start 93.218 41.91) (end 93.98 42.672) (width 0.75) (layer F.Cu) (net 3) (status 400000))
+  (segment (start 90.932 56.896) (end 91.694 56.896) (width 0.75) (layer F.Cu) (net 3))
+  (segment (start 93.218 55.372) (end 93.218 41.91) (width 0.75) (layer F.Cu) (net 3))
+  (segment (start 93.218 55.372) (end 91.694 56.896) (width 0.75) (layer F.Cu) (net 3))
+  (segment (start 90.932 56.896) (end 48.514 56.896) (width 0.75) (layer F.Cu) (net 3))
+  (segment (start 48.514 56.896) (end 45.974 54.356) (width 0.75) (layer F.Cu) (net 3))
+  (segment (start 45.974 54.356) (end 45.974 46.482) (width 0.75) (layer F.Cu) (net 3))
+  (segment (start 45.974 46.482) (end 45.466 45.974) (width 0.75) (layer F.Cu) (net 3))
+  (segment (start 43.942 45.974) (end 45.466 45.974) (width 0.75) (layer F.Cu) (net 3) (status 20))
+  (segment (start 93.218 41.91) (end 93.98 42.672) (width 0.75) (layer F.Cu) (net 3))
   (segment (start 93.98 42.672) (end 94.742 42.672) (width 0.75) (layer F.Cu) (net 3))
   (segment (start 116.332 42.672) (end 96.012 42.672) (width 0.75) (layer F.Cu) (net 3))
@@
   (segment (start 118.618 42.672) (end 118.872 42.672) (width 0.75) (layer F.Cu) (net 3))
   (segment (start 118.872 42.672) (end 121.158 44.958) (width 0.75) (layer F.Cu) (net 3))
-  (segment (start 96.012 55.626) (end 94.742 56.896) (width 0.75) (layer F.Cu) (net 3))
-  (segment (start 94.742 56.896) (end 48.514 56.896) (width 0.75) (layer F.Cu) (net 3))
-  (segment (start 48.514 56.896) (end 45.974 54.356) (width 0.75) (layer F.Cu) (net 3))
-  (segment (start 45.974 54.356) (end 45.974 46.482) (width 0.75) (layer F.Cu) (net 3))
-  (segment (start 45.974 46.482) (end 45.466 45.974) (width 0.75) (layer F.Cu) (net 3))
-  (segment (start 43.942 45.974) (end 45.466 45.974) (width 0.75) (layer F.Cu) (net 3) (status 20))
-  (segment (start 95.885 55.753) (end 94.742 56.896) (width 0.75) (layer F.Cu) (net 3))
-  (segment (start 96.012 55.626) (end 95.885 55.753) (width 0.75) (layer F.Cu) (net 3))
   (segment (start 113.538 34.036) (end 113.538 35.052) (width 0.75) (layer F.Cu) (net 3))
   (segment (start 113.538 35.052) (end 116.332 37.846) (width 0.75) (layer F.Cu) (net 3))
@@
   (segment (start 115.57 44.704) (end 118.11 47.244) (width 0.75) (layer F.Cu) (net 12) (status 30))
   (segment (start 118.618 51.308) (end 118.618 46.736) (width 0.75) (layer F.Cu) (net 12) (status 30))
-  (segment (start 81.788 31.75) (end 80.264 31.75) (width 0.75) (layer F.Cu) (net 13))
-  (segment (start 76.2 35.814) (end 76.2 36.068) (width 0.75) (layer F.Cu) (net 13))
-  (segment (start 80.264 31.75) (end 76.2 35.814) (width 0.75) (layer F.Cu) (net 13))
+  (segment (start 80.518 31.75) (end 80.264 31.75) (width 0.75) (layer F.Cu) (net 13))
+  (segment (start 80.264 31.75) (end 78.232 33.782) (width 0.75) (layer F.Cu) (net 13))
+  (segment (start 71.12 33.782) (end 69.088 35.814) (width 0.75) (layer F.Cu) (net 13))
+  (segment (start 78.232 33.782) (end 71.12 33.782) (width 0.75) (layer F.Cu) (net 13))
+  (segment (start 69.088 35.814) (end 69.088 36.068) (width 0.75) (layer F.Cu) (net 13))
+  (segment (start 81.788 31.75) (end 80.518 31.75) (width 0.75) (layer F.Cu) (net 13))
   (segment (start 116.078 31.75) (end 81.788 31.75) (width 0.75) (layer F.Cu) (net 13))
   (segment (start 81.788 31.75) (end 81.28 31.75) (width 0.75) (layer F.Cu) (net 13))
-  (segment (start 69.088 36.068) (end 72.136 36.068) (width 0.75) (layer F.Cu) (net 13) (status 10))
-  (via (at 76.2 36.068) (size 1) (drill 0.5) (layers F.Cu B.Cu) (net 13))
-  (segment (start 72.136 36.068) (end 76.2 36.068) (width 0.75) (layer B.Cu) (net 13))
-  (via (at 72.136 36.068) (size 1) (drill 0.5) (layers F.Cu B.Cu) (net 13))
   (segment (start 116.078 31.75) (end 118.618 34.036) (width 0.75) (layer F.Cu) (net 13) (status 20))
   (segment (start 98.298 31.496) (end 99.314 31.75) (width 0.75) (layer F.Cu) (net 13))
@@
   (segment (start 69.088 36.068) (end 69.088 36.322) (width 0.75) (layer F.Cu) (net 13) (status 30))
   (segment (start 127.74676 35.372) (end 127.74676 35.29076) (width 0.75) (layer F.Cu) (net 13) (status 30))
-  (segment (start 93.726 34.544) (end 93.726 38.608) (width 0.75) (layer F.Cu) (net 14))
-  (segment (start 92.456 39.878) (end 93.726 38.608) (width 0.75) (layer F.Cu) (net 14) (status 20))
+  (segment (start 92.456 40.005) (end 92.456 39.624) (width 0.75) (layer F.Cu) (net 14))
+  (segment (start 92.456 39.624) (end 93.218 38.862) (width 0.75) (layer F.Cu) (net 14))
+  (segment (start 93.218 35.052) (end 91.694 33.528) (width 0.75) (layer F.Cu) (net 14))
+  (segment (start 93.218 38.862) (end 93.218 35.052) (width 0.75) (layer F.Cu) (net 14))
   (segment (start 81.788 33.528) (end 81.534 33.274) (width 0.75) (layer F.Cu) (net 14))
   (via (at 81.534 33.274) (size 1) (drill 0.5) (layers F.Cu B.Cu) (net 14))
@@
   (segment (start 77.978 31.75) (end 77.947681 31.719681) (width 0.75) (layer F.Cu) (net 14))
   (segment (start 77.947681 31.719681) (end 69.595754 31.719681) (width 0.75) (layer F.Cu) (net 14))
-  (segment (start 92.71 33.528) (end 81.788 33.528) (width 0.75) (layer F.Cu) (net 14))
-  (segment (start 92.71 33.528) (end 93.726 34.544) (width 0.75) (layer F.Cu) (net 14))
+  (segment (start 91.694 33.528) (end 81.788 33.528) (width 0.75) (layer F.Cu) (net 14))
   (segment (start 55.86476 34.356) (end 55.86476 33.03524) (width 0.75) (layer F.Cu) (net 14) (status 10))
   (segment (start 57.15 31.75) (end 58.42 31.75) (width 0.75) (layer F.Cu) (net 14))
@@
   (segment (start 43.18 43.434) (end 43.942 43.434) (width 0.75) (layer F.Cu) (net 15) (status 30))
   (segment (start 49.022 43.106) (end 48.588 43.106) (width 0.75) (layer F.Cu) (net 15) (status 30))
-  (segment (start 74.168 39.878) (end 74.168 40.64) (width 0.75) (layer F.Cu) (net 16))
-  (segment (start 74.168 39.878) (end 74.168 35.306) (width 0.75) (layer F.Cu) (net 16))
-  (segment (start 88.011 41.91) (end 76.2 41.91) (width 0.75) (layer F.Cu) (net 16) (status 10))
-  (segment (start 72.39 33.528) (end 74.168 35.306) (width 0.75) (layer F.Cu) (net 16))
-  (segment (start 59.182 33.528) (end 58.674 34.036) (width 0.75) (layer F.Cu) (net 16) (status 20))
-  (segment (start 72.39 33.528) (end 59.182 33.528) (width 0.75) (layer F.Cu) (net 16))
-  (segment (start 75.438 41.91) (end 76.2 41.91) (width 0.75) (layer F.Cu) (net 16))
-  (segment (start 74.168 40.64) (end 75.438 41.91) (width 0.75) (layer F.Cu) (net 16))
+  (segment (start 65.278 33.528) (end 67.056 35.306) (width 0.75) (layer F.Cu) (net 16))
+  (segment (start 65.278 33.528) (end 59.182 33.528) (width 0.75) (layer F.Cu) (net 16))
+  (segment (start 58.674 34.036) (end 59.182 33.528) (width 0.75) (layer F.Cu) (net 16) (status 20))
+  (segment (start 67.056 38.608) (end 67.564 39.116) (width 0.75) (layer F.Cu) (net 16))
+  (segment (start 67.564 39.116) (end 72.898 39.116) (width 0.75) (layer F.Cu) (net 16))
+  (segment (start 67.056 35.306) (end 67.056 38.608) (width 0.75) (layer F.Cu) (net 16))
+  (segment (start 85.217 39.116) (end 88.011 41.91) (width 0.75) (layer F.Cu) (net 16))
+  (segment (start 72.898 39.116) (end 85.217 39.116) (width 0.75) (layer F.Cu) (net 16))
   (segment (start 58.674 34.036) (end 58.674 34.364) (width 0.75) (layer F.Cu) (net 16) (status 30))
   (zone (net 7) (net_name 0V) (layer In1.Cu) (hatch edge 0.508)

Commit message: update
Parts:
- moved R503 1.52 mm to (58.7, 37.3)
- moved R504 1.02 mm to (66.5, 35.1)
Routing:
- net Net-(Q502-Pad2): track 88.6 -> 72.4 mm
- net Net-(R503-Pad2): track 35.3 -> 32.3 mm
- net Net-(R504-Pad2): track 7.83 -> 9.56 mm
- net Net-(R502-Pad1): track 19.4 -> 17.9 mm
- net Net-(Q501-Pad2): track 47.5 -> 48.8 mm, vias 2 -> 0
- net REF: track 122.5 -> 123.5 mm
- net H-0V: track 72.8 -> 72.0 mm

Commit message: update
Routing:
- net Net-(R503-Pad2): track 32.3 -> 33.1 mm
Changed lines of the file:
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@@
     (thickness 1.6)
     (drawings 0)
-    (tracks 212)
+    (tracks 220)
     (zones 0)
     (modules 24)
@@
   (via (at 57.15 53.594) (size 1) (drill 0.5) (layers F.Cu B.Cu) (net 2))
   (segment (start 57.023 53.467) (end 57.15 53.594) (width 0.75) (layer F.Cu) (net 2))
+  (segment (start 48.514 56.896) (end 47.752 56.896) (width 0.75) (layer F.Cu) (net 3))
+  (segment (start 43.942 45.974) (end 45.466 45.974) (width 0.75) (layer F.Cu) (net 3) (status 10))
+  (segment (start 45.974 46.482) (end 45.466 45.974) (width 0.75) (layer F.Cu) (net 3))
+  (segment (start 45.974 54.356) (end 45.974 46.482) (width 0.75) (layer F.Cu) (net 3))
+  (segment (start 93.218 55.372) (end 91.694 56.896) (width 0.75) (layer F.Cu) (net 3))
+  (segment (start 93.218 55.372) (end 93.218 41.91) (width 0.75) (layer F.Cu) (net 3) (status 20))
+  (segment (start 48.514 56.896) (end 91.694 56.896) (width 0.75) (layer F.Cu) (net 3))
+  (segment (start 45.974 55.118) (end 45.974 54.356) (width 0.75) (layer F.Cu) (net 3))
+  (segment (start 46.228 55.372) (end 45.974 55.118) (width 0.75) (layer F.Cu) (net 3))
+  (segment (start 47.752 56.896) (end 46.228 55.372) (width 0.75) (layer F.Cu) (net 3))
   (segment (start 121.158 44.958) (end 119.634 44.958) (width 0.75) (layer F.Cu) (net 3))
   (segment (start 119.634 44.958) (end 117.348 42.672) (width 0.75) (layer F.Cu) (net 3))
@@
   (segment (start 113.284 34.036) (end 111.252 36.068) (width 0.75) (layer F.Cu) (net 3))
   (segment (start 111.252 36.068) (end 111.252 42.672) (width 0.75) (layer F.Cu) (net 3))
-  (segment (start 48.514 56.896) (end 91.694 56.896) (width 0.75) (layer F.Cu) (net 3))
-  (segment (start 93.218 55.372) (end 93.218 41.91) (width 0.75) (layer F.Cu) (net 3) (status 20))
-  (segment (start 93.218 55.372) (end 91.694 56.896) (width 0.75) (layer F.Cu) (net 3))
-  (segment (start 48.514 56.896) (end 45.974 54.356) (width 0.75) (layer F.Cu) (net 3))
-  (segment (start 45.974 54.356) (end 45.974 46.482) (width 0.75) (layer F.Cu) (net 3))
-  (segment (start 45.974 46.482) (end 45.466 45.974) (width 0.75) (layer F.Cu) (net 3))
-  (segment (start 43.942 45.974) (end 45.466 45.974) (width 0.75) (layer F.Cu) (net 3) (status 10))
   (segment (start 93.218 41.91) (end 93.98 42.672) (width 0.75) (layer F.Cu) (net 3) (status 10))
   (segment (start 93.98 42.672) (end 94.742 42.672) (width 0.75) (layer F.Cu) (net 3))
@@
   (segment (start 69.088 35.052) (end 69.088 35.306) (width 0.75) (layer F.Cu) (net 13) (status 30))
   (segment (start 127.74676 35.372) (end 127.74676 35.29076) (width 0.75) (layer F.Cu) (net 13) (status 30))
+  (segment (start 63.492001 37.853999) (end 69.080001 37.853999) (width 0.75) (layer F.Cu) (net 14))
+  (segment (start 69.080001 37.853999) (end 69.088 37.861998) (width 0.75) (layer F.Cu) (net 14))
+  (segment (start 63.119 37.465) (end 63.119 37.480998) (width 0.75) (layer F.Cu) (net 14))
+  (segment (start 63.119 37.480998) (end 63.492001 37.853999) (width 0.75) (layer F.Cu) (net 14))
+  (segment (start 63.492001 37.853999) (end 63.5 37.861998) (width 0.75) (layer F.Cu) (net 14))
+  (segment (start 69.088 37.861998) (end 69.834002 37.861998) (width 0.75) (layer F.Cu) (net 14))
+  (segment (start 69.834002 37.861998) (end 70.104 37.592) (width 0.75) (layer F.Cu) (net 14))
   (segment (start 70.104 37.592) (end 71.374 36.322) (width 0.75) (layer F.Cu) (net 14))
   (segment (start 71.374 36.322) (end 71.374 35.814) (width 0.75) (layer F.Cu) (net 14))
-  (segment (start 63.5 37.861998) (end 63.5 37.846) (width 0.75) (layer F.Cu) (net 14))
-  (segment (start 63.5 37.846) (end 60.01 34.356) (width 0.75) (layer F.Cu) (net 14))
   (segment (start 74.422 33.528) (end 72.136 33.528) (width 0.75) (layer F.Cu) (net 14))
   (segment (start 71.374 34.29) (end 71.374 35.814) (width 0.75) (layer F.Cu) (net 14))
   (segment (start 72.136 33.528) (end 71.374 34.29) (width 0.75) (layer F.Cu) (net 14))
+  (segment (start 75.184 33.528) (end 74.422 33.528) (width 0.75) (layer F.Cu) (net 14))
+  (segment (start 75.184 33.528) (end 91.694 33.528) (width 0.75) (layer F.Cu) (net 14))
+  (segment (start 93.218 38.862) (end 92.456 39.624) (width 0.75) (layer F.Cu) (net 14) (status 20))
+  (segment (start 93.218 35.052) (end 91.694 33.528) (width 0.75) (layer F.Cu) (net 14))
+  (segment (start 93.218 38.862) (end 93.218 35.052) (width 0.75) (layer F.Cu) (net 14))
+  (segment (start 63.119 37.465) (end 60.01 34.356) (width 0.75) (layer F.Cu) (net 14))
   (segment (start 60.01 34.356) (end 55.86476 34.356) (width 0.75) (layer F.Cu) (net 14))
   (segment (start 63.515998 37.861998) (end 63.5 37.861998) (width 0.75) (layer F.Cu) (net 14))
-  (segment (start 63.5 37.861998) (end 63.246 37.861998) (width 0.75) (layer F.Cu) (net 14))
-  (segment (start 63.246 37.846) (end 63.246 37.861998) (width 0.75) (layer F.Cu) (net 14))
-  (segment (start 68.58 37.861998) (end 70.104 37.861998) (width 0.75) (layer F.Cu) (net 14))
-  (segment (start 68.58 37.861998) (end 63.246 37.861998) (width 0.75) (layer F.Cu) (net 14))
-  (segment (start 63.246 37.861998) (end 63.246 37.846) (width 0.75) (layer F.Cu) (net 14))
-  (segment (start 75.184 33.528) (end 74.422 33.528) (width 0.75) (layer F.Cu) (net 14))
-  (segment (start 75.184 33.528) (end 91.694 33.528) (width 0.75) (layer F.Cu) (net 14))
-  (segment (start 92.456 39.624) (end 93.218 38.862) (width 0.75) (layer F.Cu) (net 14) (status 20))
-  (segment (start 93.218 35.052) (end 91.694 33.528) (width 0.75) (layer F.Cu) (net 14))
-  (segment (start 93.218 38.862) (end 93.218 35.052) (width 0.75) (layer F.Cu) (net 14))
+  (segment (start 68.58 37.861998) (end 69.088 37.861998) (width 0.75) (layer F.Cu) (net 14))
   (segment (start 92.456 40.005) (end 92.456 39.624) (width 0.75) (layer F.Cu) (net 14) (status 30))
   (segment (start 92.456 40.005) (end 92.456 39.878) (width 0.75) (layer F.Cu) (net 14) (status 30))
@@
   (segment (start 43.18 43.434) (end 43.942 43.434) (width 0.75) (layer F.Cu) (net 15) (status 30))
   (segment (start 49.022 43.106) (end 48.588 43.106) (width 0.75) (layer F.Cu) (net 15) (status 30))
+  (segment (start 88.011 41.91) (end 88.011 41.783) (width 0.75) (layer F.Cu) (net 16) (status C00000))
+  (segment (start 88.011 41.783) (end 85.598 39.37) (width 0.75) (layer F.Cu) (net 16) (status 400000))
+  (segment (start 85.598 39.37) (end 84.582 39.37) (width 0.75) (layer F.Cu) (net 16))
   (segment (start 67.31 39.37) (end 62.156 39.37) (width 0.75) (layer F.Cu) (net 16))
   (segment (start 62.156 39.37) (end 58.674 35.888) (width 0.75) (layer F.Cu) (net 16))
   (segment (start 67.564 39.37) (end 67.31 39.37) (width 0.75) (layer F.Cu) (net 16))
   (segment (start 67.31 39.37) (end 67.056 39.37) (width 0.75) (layer F.Cu) (net 16))
-  (segment (start 88.011 41.91) (end 85.217 39.37) (width 0.75) (layer F.Cu) (net 16) (status 20))
-  (segment (start 67.564 39.37) (end 85.217 39.37) (width 0.75) (layer F.Cu) (net 16))
+  (segment (start 67.564 39.37) (end 84.582 39.37) (width 0.75) (layer F.Cu) (net 16))
+  (segment (start 84.582 39.37) (end 85.217 39.37) (width 0.75) (layer F.Cu) (net 16))
   (segment (start 58.674 35.56) (end 58.674 35.888) (width 0.75) (layer F.Cu) (net 16) (status 30))
   (zone (net 7) (net_name 0V) (layer In1.Cu) (hatch edge 0.508)

Commit message: update
Parts:
- added C301: C, Capacitors_SMD:C_1206, F.Cu at (56.6, 65.6)
- added C302: C, Capacitors_SMD:C_1206, F.Cu at (55.6, 78.0)
- added C303: C, Capacitors_SMD:C_1206, F.Cu at (82.0, 81.8)
- added C304: C, Capacitors_SMD:C_1206, F.Cu at (88.6, 69.1)
- added C305: C, Capacitors_SMD:C_1206, F.Cu at (94.7, 89.2)
- added C306: C, Capacitors_SMD:C_1206, F.Cu at (105.7, 88.9)
- added C307: C, Capacitors_SMD:C_1206, F.Cu at (109.2, 85.6)
- added C308: C, Capacitors_SMD:C_1206, F.Cu at (119.9, 85.6)
- added C309: C, Capacitors_SMD:C_1206, F.Cu at (65.0, 84.6)
- added C310: C, Capacitors_SMD:C_1206, F.Cu at (114.6, 101.1)
- added C311: C, Capacitors_SMD:C_1206, F.Cu at (93.0, 77.5)
- added C312: C, Capacitors_SMD:C_1206, F.Cu at (65.8, 75.2)
- added C313: C, Capacitors_SMD:C_1206, F.Cu at (74.4, 84.6)
- added C314: C, Capacitors_ThroughHole:C_Radial_D7.5_L11.2_P2.5, F.Cu at (91.4, 71.1)
- added D301: 1N4148, Diodes_ThroughHole:Diode_DO-35_SOD27_Horizontal_RM10, F.Cu at (105.9, 108.7)
- added D302: 1N4148, Diodes_ThroughHole:Diode_DO-35_SOD27_Horizontal_RM10, F.Cu at (116.1, 113.8)
- added P301: CONN_01X15, Pin_Headers:Pin_Header_Straight_1x15, F.Cu at (43.9, 63.0)
- added P302: CONN_01X03, Pin_Headers:Pin_Header_Straight_1x03, F.Cu at (94.0, 111.5)
- added R301: R, Resistors_ThroughHole:Resistor_TO-220_Vertical, F.Cu at (68.3, 94.0)
- added R302: R, Resistors_ThroughHole:Resistor_TO-220_Vertical, F.Cu at (68.3, 98.3)
- added R303: R, Resistors_ThroughHole:Resistor_TO-220_Vertical, F.Cu at (84.6, 88.9)
- added R304: 1k, Resistors_SMD:R_1206, F.Cu at (108.0, 100.3)
- added R305: 10k, Resistors_SMD:R_1206, F.Cu at (125.2, 115.3)
- added R306: 5k, Resistors_SMD:R_1206, F.Cu at (113.3, 77.0)
- added U301: LM741, Housings_SOIC:SOIC-8_3.9x4.9mm_Pitch1.27mm, F.Cu at (69.6, 84.8)
- added U302: DG444, Housings_SOIC:SOIC-16_3.9x9.9mm_Pitch1.27mm, F.Cu at (55.1, 85.1)
- added U303: LM741, Housings_SOIC:SOIC-8_3.9x4.9mm_Pitch1.27mm, F.Cu at (87.1, 81.5)
- added U304: LM741, Housings_SOIC:SOIC-8_3.9x4.9mm_Pitch1.27mm, F.Cu at (100.1, 88.9)
- added U305: LM311N, Housings_SOIC:SOIC-8_3.9x4.9mm_Pitch1.27mm, F.Cu at (114.3, 85.6)
- added W301: TEST_1P, Pin_Headers:Pin_Header_Straight_1x01, F.Cu at (68.8, 117.1)
Routing:
- net REF: track 123.9 -> 153.0 mm, vias 0 -> 1
- net REF_PLUS_CTL: track 0.00 -> 19.0 mm, vias 0 -> 2
- net RESET: track 0.00 -> 18.5 mm
- net 3.3V: track 0.00 -> 17.7 mm, vias 0 -> 2
- net 0V: track 23.8 -> 39.1 mm, vias 6 -> 10
- net IN_CTL: track 0.00 -> 14.9 mm, vias 0 -> 1
- net Net-(R303-Pad2): track 0.00 -> 13.5 mm
- net IN: track 0.00 -> 12.5 mm
- net Net-(R301-Pad1): track 0.00 -> 12.4 mm
- net -VE: track 16.5 -> 25.3 mm, vias 3 -> 4
- net REF_SUB_CTL: track 0.00 -> 8.24 mm
- net +VE: track 25.4 -> 33.4 mm, vias 5 -> 6
- net (no net): vias 0 -> 1

Commit message: complete
Parts:
- C314: footprint Capacitors_ThroughHole:C_Radial_D7.5_L11.2_P2.5 -> Capacitors_ThroughHole:C_Rect_L7_W3.5_P5
- D301, D302: footprint Diodes_ThroughHole:Diode_DO-35_SOD27_Horizontal_RM10 -> Diodes_SMD:MiniMELF_Standard
- moved C310 70.3 mm to (53.3, 66.5)
- moved W301 51.3 mm to (84.8, 68.3)
- moved R305 31.2 mm to (101.1, 95.5), turned to 90 degrees
- moved D302 24.2 mm to (106.2, 91.7)
- moved C312 20.1 mm to (55.1, 92.2)
- moved R303 19.9 mm to (73.2, 72.6)
- moved P302 16.3 mm to (92.5, 95.2), turned to 90 degrees
- moved C304 16.0 mm to (88.9, 85.1)
- moved D301 14.2 mm to (106.2, 94.5)
- moved R304 10.0 mm to (113.8, 92.2)
- moved C311 9.66 mm to (83.3, 77.2), turned to 180 degrees
- moved C301 6.72 mm to (50.0, 66.8), turned to 270 degrees
- moved C314 6.59 mm to (85.1, 72.9), turned to 180 degrees
- moved C306 5.21 mm to (102.1, 85.1)
- moved U304 4.72 mm to (97.3, 85.1)
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Routing:
- net TRIGGER: track 0.00 -> 109.2 mm, vias 0 -> 2
- net Net-(C311-Pad1): track 0.00 -> 86.0 mm, vias 0 -> 5
- net Net-(R302-Pad1): track 0.00 -> 51.3 mm
- net Net-(C311-Pad2): track 0.00 -> 49.5 mm, vias 0 -> 3
- net Net-(D301-Pad2): track 0.00 -> 40.2 mm, vias 0 -> 2
- net Net-(P302-Pad2): track 0.00 -> 34.8 mm
- net +VE: track 33.4 -> 67.1 mm, vias 6 -> 11
- net REF: track 153.0 -> 184.9 mm, vias 1 -> 2
- net 0V: track 39.1 -> 66.0 mm, vias 10 -> 19
- net Net-(D301-Pad1): track 0.00 -> 25.9 mm
- net -VE: track 25.3 -> 47.9 mm, vias 4 -> 8
- net Net-(R303-Pad2): track 13.5 -> 30.2 mm
- net REF_PLUS_CTL: track 19.0 -> 17.7 mm
- net Net-(R301-Pad1): track 12.4 -> 13.3 mm
- net RESET: vias 0 -> 2
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
Commit message: tidy
Parts:
- moved C301 0.25 mm to (50.0, 66.5)
Routing:
- net REF: track 184.9 -> 192.0 mm, vias 2 -> 0
- net 0V: track 66.0 -> 72.1 mm, vias 19 -> 20
- net -VE: track 47.9 -> 50.8 mm, vias 8 -> 9
- net +VE: track 67.1 -> 69.9 mm, vias 11 -> 12
- net Net-(R303-Pad2): track 30.2 -> 31.4 mm, vias 0 -> 2
Other:
- board text added: "V0.1"
