File: src/main.sch (KiCad schematic (older format))
At the start: 0 parts

Commit message: just the dw232
Changed lines of the file:
@@
 $EndDescr
-$Sheet
-S 1100 2500 1300 1000
-U 585BBA35
-F0 "ADC" 60
-F1 "adc.sch" 60
-$EndSheet
-$Sheet
-S 1100 1200 1200 750
-U 5861F05C
-F0 "clamps" 60
-F1 "clamps.sch" 60
-$EndSheet
-$Sheet
-S 3800 1300 1350 900
-U 58642788
-F0 "ref" 60
-F1 "ref.sch" 60
-$EndSheet
 $Sheet
 S 5200 2850 1500 800

Commit message: update
Changed lines of the file:
@@
 $Descr A4 11693 8268
 encoding utf-8
-Sheet 1 2
+Sheet 1 3
 Title ""
 Date ""
@@
 F1 "2dw232-ref.sch" 60
 $EndSheet
+$Sheet
+S 1550 2850 1600 750
+U 58843A43
+F0 "adc" 60
+F1 "adc.sch" 60
+$EndSheet
 $EndSCHEMATC

Commit message: update
Changed lines of the file:
@@
 EESchema Schematic File Version 2
+LIBS:main-rescue
 LIBS:my
 LIBS:Carlolib-disc
@@
 $Descr A4 11693 8268
 encoding utf-8
-Sheet 1 3
+Sheet 1 4
 Title ""
 Date ""
@@
 F1 "adc.sch" 60
 $EndSheet
+$Sheet
+S 3700 4350 2000 1000
+U 5889A78C
+F0 "clamps" 60
+F1 "clamps.sch" 60
+$EndSheet
 $EndSCHEMATC
