File: projects/smu/ref-10V.sch (KiCad schematic (older format))
At the start: 4 parts, among them U501 LT1021

Commit message: add power
Parts:
- U901: renamed from U501; footprint (none) -> Housings_SOIC:SOIC-8_3.9x4.9mm_Pitch1.27mm
- renumbered C501 to C901, L501 to L901, R501 to R901
Changed lines of the file:
@@
 $Descr A4 11693 8268
 encoding utf-8
-Sheet 4 4
+Sheet 4 5
 Title ""
 Date ""
@@
 $EndDescr
 $Comp
-L LT1021 U501
+L LT1021 U901
 U 1 1 58AD056A
 P 5450 3050
-F 0 "U501" H 5600 3400 50  0000 L CNN
+F 0 "U901" H 5600 3400 50  0000 L CNN
 F 1 "LT1021" H 5300 2700 50  0000 L CNN
-F 2 "" H 5450 2700 50  0001 C CNN
+F 2 "Housings_SOIC:SOIC-8_3.9x4.9mm_Pitch1.27mm" H 5450 2700 50  0001 C CNN
 F 3 "" H 5450 2700 50  0000 C CNN
 	1    5450 3050
@@
 $EndComp
 Wire Wire Line
-	4600 3000 4700 3000
-Wire Wire Line
-	4700 3000 4850 3000
+	4600 3000 4850 3000
 Text GLabel 4650 3200 0    60   Input ~ 0
 REFGND
@@
 NoConn ~ 6050 3200
 $Comp
-L R R501
+L R R901
 U 1 1 58AD08E8
 P 6400 3100
-F 0 "R501" V 6480 3100 50  0000 C CNN
+F 0 "R901" V 6480 3100 50  0000 C CNN
 F 1 "0R" V 6400 3100 50  0000 C CNN
 F 2 "Resistors_SMD:R_1206" V 6330 3100 50  0001 C CNN
@@
 +VE
 $Comp
-L C C501
+L C C901
 U 1 1 58AD0A77
 P 4700 2650
-F 0 "C501" H 4725 2750 50  0000 L CNN
+F 0 "C901" H 4725 2750 50  0000 L CNN
 F 1 "C" H 4725 2550 50  0000 L CNN
 F 2 "Capacitors_SMD:C_1206" H 4738 2500 50  0001 C CNN
@@
 REFGND
 $Comp
-L INDUCTOR L501
+L INDUCTOR L901
 U 1 1 58AD0B9B
 P 4300 3000
-F 0 "L501" V 4250 3000 50  0000 C CNN
+F 0 "L901" V 4250 3000 50  0000 C CNN
 F 1 "INDUCTOR" V 4400 3000 50  0000 C CNN
 F 2 "Resistors_SMD:R_1206" H 4300 3000 50  0001 C CNN
