File: projects/smu/main.sch (KiCad schematic (older format))
At the start: 3 parts, among them P101 CONN_01X20, P102 CONN_01X28, P103 CONN_01X15

Commit message: update
Parts:
- removed P101: CONN_01X20, symbol CONN_01X20
- removed P103: CONN_01X15, Pin_Headers:Pin_Header_Straight_1x15, symbol CONN_01X15
- added P101: CONN_01X26, symbol CONN_01X26
Connections:
- net +VE: now also P101.5 (P5)
- net -VE: now also P101.7 (P7)
- net 3.3V: now also P102.1 (P1), P102.10 (P10); no longer P102.9 (P9)
- net ADC_IN: now also P101.12 (P12)
- net ADC_IN_CTL: now also P102.13 (P13); no longer P102.12 (P12)
- net ADC_MIN_CTL: now also P102.12 (P12); no longer P102.11 (P11)
- net ADC_PLUS_CTL: now also P102.11 (P11); no longer P102.10 (P10)
- net ADC_RESET: now also P102.14 (P14); no longer P102.13 (P13)
- net ADC_TRIGGER: now also P102.15 (P15); no longer P102.14 (P14)
- net AGND: now also P102.16 (P16), P102.8 (P8), P101.10 (P10), P101.13 (P13), P101.2 (P2), P101.25 (P25), P101.6 (P6); no longer P102.15 (P15), P102.7 (P7)
- net CLAMP_OUT: now also P101.22 (P22)
- net DAC_CS: now also P102.2 (P2); no longer P102.1 (P1)
- net DAC_LDAC: now also P102.6 (P6); no longer P102.5 (P5)
- net DAC_RST: now also P102.7 (P7); no longer P102.6 (P6)
- net DAC_SDI: now also P102.4 (P4); no longer P102.3 (P3)
- net DAC_SDO: now also P102.5 (P5); no longer P102.4 (P4)
- net DAC_SLCK: now also P102.3 (P3); no longer P102.2 (P2)
- net I_FB: now also P101.21 (P21)
- net I_SET: now also P101.16 (P16)
- net PWR_+VE: now also P101.1 (P1)
- net PWR_+VE_CTL: now also P102.18 (P18); no longer P102.17 (P17)
- net PWR_-VE: now also P101.3 (P3)
- net PWR_-VE_CTL: now also P102.19 (P19); no longer P102.18 (P18)
- net REF: now also P101.9 (P9)
- net SLEW_SET: now also P101.17 (P17)
- net V_FB: now also P101.20 (P20)
- net V_OUT_4: now also P101.18 (P18)
- net V_SET: now also P101.15 (P15)
- net REF_IN_-VE: now reaches P102.22 (P22)
- net REF_IN1: no longer names the net of P102.20 (P20)
- net REF_IN2 renamed REF_IN_+VE
- new net OUT: P101.24 (P24)
- no-connect marks 19 -> 16
Other:
- moved on the sheet: P102
Changed lines of the file:
@@
 $Descr A4 11693 8268
 encoding utf-8
-Sheet 1 6
+Sheet 1 7
 Title ""
 Date ""
@@
 F1 "clamps.sch" 60
 $EndSheet
-Text GLabel 2600 950  0    60   Input ~ 0
+Text GLabel 2600 1300 0    60   Input ~ 0
 +VE
-Text GLabel 2600 1050 0    60   Input ~ 0
-AGND
-Text GLabel 2600 1150 0    60   Input ~ 0
+Text GLabel 2600 1400 0    60   Input ~ 0
+AGND
+Text GLabel 2600 1500 0    60   Input ~ 0
 -VE
-Text GLabel 2600 1450 0    60   Input ~ 0
+Text GLabel 2600 1700 0    60   Input ~ 0
 REF
-Text GLabel 2600 1750 0    60   Input ~ 0
+Text GLabel 2600 2000 0    60   Input ~ 0
 ADC_IN
 Text GLabel 4750 1750 0    60   Input ~ 0
@@
 Text GLabel 4750 2150 0    60   Input ~ 0
 ADC_RESET
-Text GLabel 2600 1250 0    60   Input ~ 0
-AGND
-Text GLabel 2600 1850 0    60   Input ~ 0
+Text GLabel 2600 2100 0    60   Input ~ 0
 AGND
 Text GLabel 4750 2350 0    60   Input ~ 0
@@
 Text GLabel 4750 2250 0    60   Input ~ 0
 ADC_TRIGGER
-Text GLabel 7050 1500 3    60   Input ~ 0
+Text GLabel 6250 1500 3    60   Input ~ 0
 +VE
 $Comp
 L PWR_FLAG #FLG01
 U 1 1 58A9E478
-P 7050 1300
-F 0 "#FLG01" H 7050 1395 50  0001 C CNN
-F 1 "PWR_FLAG" H 7050 1480 50  0000 C CNN
-F 2 "" H 7050 1300 50  0000 C CNN
-F 3 "" H 7050 1300 50  0000 C CNN
-	1    7050 1300
+P 6250 1300
+F 0 "#FLG01" H 6250 1395 50  0001 C CNN
+F 1 "PWR_FLAG" H 6250 1480 50  0000 C CNN
+F 2 "" H 6250 1300 50  0000 C CNN
+F 3 "" H 6250 1300 50  0000 C CNN
+	1    6250 1300
 	1    0    0    -1
 $EndComp
@@
 L PWR_FLAG #FLG02
 U 1 1 58A9E47F
-P 7650 1300
-F 0 "#FLG02" H 7650 1395 50  0001 C CNN
-F 1 "PWR_FLAG" H 7650 1480 50  0000 C CNN
-F 2 "" H 7650 1300 50  0000 C CNN
-F 3 "" H 7650 1300 50  0000 C CNN
-	1    7650 1300
-	1    0    0    -1
-$EndComp
-Text GLabel 7650 1500 3    60   Input ~ 0
+P 6850 1300
+F 0 "#FLG02" H 6850 1395 50  0001 C CNN
+F 1 "PWR_FLAG" H 6850 1480 50  0000 C CNN
+F 2 "" H 6850 1300 50  0000 C CNN
+F 3 "" H 6850 1300 50  0000 C CNN
+	1    6850 1300
+	1    0    0    -1
+$EndComp
+Text GLabel 6850 1500 3    60   Input ~ 0
 -VE
-Text GLabel 9200 1400 0    60   Input ~ 0
-AGND
-Text GLabel 9200 1500 0    60   Input ~ 0
-DGND
-Text GLabel 9200 1600 0    60   Input ~ 0
+Text GLabel 7850 1300 0    60   Input ~ 0
+AGND
+Text GLabel 7850 1500 0    60   Input ~ 0
+DGND
+Text GLabel 7850 1700 0    60   Input ~ 0
 REFGND
-Text GLabel 2550 2650 0    60   Input ~ 0
+Text GLabel 2550 2900 0    60   Input ~ 0
 I_FB
-Text GLabel 2550 2750 0    60   Input ~ 0
+Text GLabel 2550 3000 0    60   Input ~ 0
 CLAMP_OUT
-Text GLabel 2550 2550 0    60   Input ~ 0
+Text GLabel 2550 2800 0    60   Input ~ 0
 V_FB
-Text GLabel 2550 2250 0    60   Input ~ 0
+Text GLabel 2550 2500 0    60   Input ~ 0
 SLEW_SET
-Text GLabel 2550 2350 0    60   Input ~ 0
+Text GLabel 2550 2600 0    60   Input ~ 0
 V_OUT_4
 Text GLabel 4800 950  0    60   Input ~ 0
@@
 Text GLabel 4800 1450 0    60   Input ~ 0
 DAC_RST
-Text GLabel 9200 1400 0    60   Input ~ 0
-AGND
-Text GLabel 9200 1500 0    60   Input ~ 0
-DGND
-Text GLabel 9200 1600 0    60   Input ~ 0
+Text GLabel 7850 1300 0    60   Input ~ 0
+AGND
+Text GLabel 7850 1500 0    60   Input ~ 0
+DGND
+Text GLabel 7850 1700 0    60   Input ~ 0
 REFGND
-Text GLabel 2550 2050 0    60   Input ~ 0
+Text GLabel 2550 2300 0    60   Input ~ 0
 V_SET
-Text GLabel 2550 2150 0    60   Input ~ 0
+Text GLabel 2550 2400 0    60   Input ~ 0
 I_SET
-Text GLabel 2600 1550 0    60   Input ~ 0
+Text GLabel 2600 1800 0    60   Input ~ 0
 REFGND
 $Comp
 L CONN_01X28 P102
 U 1 1 58A96BF2
-P 5300 2300
-F 0 "P102" H 5300 3750 50  0000 C CNN
-F 1 "CONN_01X28" V 5400 2300 50  0000 C CNN
-F 2 "Pin_Headers:Pin_Header_Straight_1x28" H 5300 2300 50  0001 C CNN
-F 3 "" H 5300 2300 50  0000 C CNN
-	1    5300 2300
+P 5300 2200
+F 0 "P102" H 5300 3650 50  0000 C CNN
+F 1 "CONN_01X28" V 5400 2200 50  0000 C CNN
+F 2 "Pin_Headers:Pin_Header_Straight_1x28" H 5300 2200 50  0001 C CNN
+F 3 "" H 5300 2200 50  0000 C CNN
+	1    5300 2200
 	1    0    0    -1
 $EndComp
 Text GLabel 4750 2950 0    60   Input ~ 0
-REF_IN2
+REF_IN_-VE
 Text GLabel 4750 2850 0    60   Input ~ 0
-REF_IN1
+REF_IN_+VE
 NoConn ~ 5100 2750
 $Sheet
@@
 F1 "power.sch" 60
 $EndSheet
-$Comp
-L CONN_01X15 P103
-U 1 1 58AE3540
-P 1300 1650
-F 0 "P103" H 1300 2450 50  0000 C CNN
-F 1 "CONN_01X15" V 1400 1650 50  0000 C CNN
-F 2 "Pin_Headers:Pin_Header_Straight_1x15" H 1300 1650 50  0001 C CNN
-F 3 "" H 1300 1650 50  0000 C CNN
-	1    1300 1650
-	1    0    0    -1
-$EndComp
-Text GLabel 1100 950  0    60   Input ~ 0
+Text GLabel 2600 900  0    60   Input ~ 0
 PWR_+VE
-Text GLabel 1100 1150 0    60   Input ~ 0
+Text GLabel 2600 1100 0    60   Input ~ 0
 PWR_-VE
-NoConn ~ 1100 1250
-NoConn ~ 1100 1350
-NoConn ~ 1100 1450
-NoConn ~ 1100 1550
-NoConn ~ 1100 1650
-NoConn ~ 1100 1750
-NoConn ~ 1100 1850
-NoConn ~ 1100 1950
-NoConn ~ 1100 2050
-NoConn ~ 1100 2150
-NoConn ~ 1100 2250
-NoConn ~ 1100 2350
-Text GLabel 1100 1050 0    60   Input ~ 0
+Text GLabel 2600 1000 0    60   Input ~ 0
 AGND
 Text GLabel 4750 2550 0    60   Input ~ 0
@@
 $EndSheet
 Wire Wire Line
-	2850 950  2600 950
-Wire Wire Line
-	2850 1050 2600 1050
-Wire Wire Line
-	2850 1150 2600 1150
-Wire Wire Line
-	2850 1250 2600 1250
-Wire Wire Line
-	7050 1300 7050 1500
-Wire Wire Line
-	7650 1300 7650 1500
-Wire Wire Line
-	9200 1400 9200 1600
+	2850 1300 2600 1300
+Wire Wire Line
+	2850 1400 2600 1400
+Wire Wire Line
+	2850 1500 2600 1500
+Wire Wire Line
+	6250 1300 6250 1500
+Wire Wire Line
+	6850 1300 6850 1500
+Wire Wire Line
+	7850 1300 7850 1900
 Wire Wire Line
 	4800 950  5100 950
@@
 	4800 1550 5100 1550
 Wire Wire Line
-	2550 2050 2850 2050
-Wire Wire Line
-	2550 2150 2850 2150
-Wire Wire Line
-	2550 2250 2850 2250
-Wire Wire Line
-	2550 2350 2850 2350
+	2550 2300 2850 2300
+Wire Wire Line
+	2550 2400 2850 2400
+Wire Wire Line
+	2550 2500 2850 2500
+Wire Wire Line
+	2550 2600 2850 2600
 NoConn ~ 5100 1650
 Wire Wire Line
-	2550 2550 2850 2550
-Wire Wire Line
-	2550 2650 2850 2650
-Wire Wire Line
-	2550 2750 2850 2750
+	2550 2800 2850 2800
+Wire Wire Line
+	2550 2900 2850 2900
+Wire Wire Line
+	2550 3000 2850 3000
 Wire Wire Line
 	4750 2850 5100 2850
@@
 NoConn ~ 5100 2450
 Wire Wire Line
-	2850 1450 2600 1450
-Wire Wire Line
-	2850 1550 2600 1550
-Wire Wire Line
-	2850 1750 2600 1750
-Wire Wire Line
-	2850 1850 2600 1850
-$Comp
-L CONN_01X20 P101
-U 1 1 58C50B86
-P 3050 1900
-F 0 "P101" H 3050 2950 50  0000 C CNN
-F 1 "CONN_01X20" V 3150 1900 50  0000 C CNN
-F 2 "" H 3050 1900 50  0000 C CNN
-F 3 "" H 3050 1900 50  0000 C CNN
-	1    3050 1900
-	1    0    0    -1
-$EndComp
-NoConn ~ 2850 1650
-NoConn ~ 2850 1950
-NoConn ~ 2850 1350
-NoConn ~ 2850 2450
+	2850 1700 2600 1700
+Wire Wire Line
+	2850 1800 2600 1800
+Wire Wire Line
+	2850 2000 2600 2000
+Wire Wire Line
+	2850 2100 2600 2100
+NoConn ~ 2850 1900
+NoConn ~ 2850 2200
+NoConn ~ 2850 1600
+NoConn ~ 2850 2700
+Text GLabel 4800 850  0    60   Input ~ 0
+3.3V
+Wire Wire Line
+	4800 850  5100 850
+NoConn ~ 5100 3050
+NoConn ~ 5100 3150
+NoConn ~ 5100 3250
+NoConn ~ 5100 3350
+NoConn ~ 5100 3450
+NoConn ~ 5100 3550
+$Comp
+L CONN_01X26 P101
+U 1 1 58C4A995
+P 3050 2150
+F 0 "P101" H 3050 3500 50  0000 C CNN
+F 1 "CONN_01X26" V 3150 2150 50  0000 C CNN
+F 2 "" H 3050 2150 50  0000 C CNN
+F 3 "" H 3050 2150 50  0000 C CNN
+	1    3050 2150
+	1    0    0    -1
+$EndComp
+Wire Wire Line
+	2600 900  2850 900
+Wire Wire Line
+	2600 1000 2850 1000
+Wire Wire Line
+	2600 1100 2850 1100
+NoConn ~ 2850 1200
+Text GLabel 2550 3200 0    60   Input ~ 0
+OUT
+Wire Wire Line
+	2550 3200 2850 3200
+NoConn ~ 2850 3100
+Text GLabel 2550 3300 0    60   Input ~ 0
+OUTGND
+Wire Wire Line
+	2550 3300 2850 3300
+NoConn ~ 2850 3400
+Text GLabel 7850 1900 0    60   Input ~ 0
+OUTGND
+$Sheet
+S 3700 5650 1850 850
+U 58C4BEDB
+F0 "feedback" 60
+F1 "feedback.sch" 60
+$EndSheet
 $EndSCHEMATC

Commit message: update
Parts:
- added RL?: Omron_G6S, symbol Omron_G6S
Changed lines of the file:
@@
 LIBS:contrib
 LIBS:valves
+LIBS:relays
 LIBS:main-cache
 EELAYER 25 0
@@
 F1 "feedback.sch" 60
 $EndSheet
+$Comp
+L Omron_G6S RL?
+U 1 1 58C5ED1C
+P 8500 5500
+F 0 "RL?" H 9350 5650 50  0000 L CNN
+F 1 "Omron_G6S" H 9350 5550 50  0000 L CNN
+F 2 "" H 8500 5500 60  0000 C CNN
+F 3 "" H 8500 5500 60  0000 C CNN
+	1    8500 5500
+	1    0    0    -1
+$EndComp
 $EndSCHEMATC
