File: projects/dw232/main.kicad_pcb (KiCad board)
At the start: 4 copper layers, 27 parts, among them P101 CONN_01X07, Q501 MMBT3904, Q502 MMBT3904, U501 LM741, U502 LM741, U503 2DW232

Commit message: add edge cuts
Other:
- board outline added: 99 x 25 mm
- board text added: "Ver. 0.1 (C) JA, 2017 GNU GPL"
- board text removed: "Ver. 0.1 (C) JA, 2017 GNU"
Changed lines of the file:
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@@
     (links 52)
     (no_connects 0)
-    (area 40 29 139.000001 54.000001)
+    (area 39.949999 28.949999 139.050001 54.050001)
     (thickness 1.6)
-    (drawings 8)
+    (drawings 12)
     (tracks 164)
     (zones 0)
@@
     (33 F.Adhes user hide)
     (36 B.SilkS user hide)
-    (37 F.SilkS user)
-    (38 B.Mask user hide)
-    (39 F.Mask user hide)
+    (37 F.SilkS user hide)
+    (38 B.Mask user)
+    (39 F.Mask user)
     (40 Dwgs.User user hide)
     (41 Cmts.User user hide)
     (42 Eco1.User user hide)
     (43 Eco2.User user hide)
-    (44 Edge.Cuts user hide)
+    (44 Edge.Cuts user)
     (45 Margin user hide)
     (47 F.CrtYd user hide)
@@
     (visible_elements FFFFFF7F)
     (pcbplotparams
-      (layerselection 0x012a0_80000007)
+      (layerselection 0x010f0_80000007)
       (usegerberextensions false)
       (excludeedgelayer true)
       (linewidth 0.100000)
-      (plotframeref false)
+      (plotframeref true)
       (viasonmask false)
       (mode 1)
@@
       (net 11 "Net-(R508-Pad1)"))
   )
-  (gr_text "Ver. 0.1 (C) JA, 2017\nGNU" (at 109 51) (layer F.SilkS)
+  (gr_line (start 40 54) (end 40 29) (angle 90) (layer Edge.Cuts) (width 0.1))
+  (gr_line (start 139 54) (end 40 54) (angle 90) (layer Edge.Cuts) (width 0.1))
+  (gr_line (start 139 29) (end 139 54) (angle 90) (layer Edge.Cuts) (width 0.1))
+  (gr_line (start 40 29) (end 139 29) (angle 90) (layer Edge.Cuts) (width 0.1))
+  (gr_text "Ver. 0.1 (C) JA, 2017\nGNU GPL" (at 109 51) (layer F.SilkS)
     (effects (font (size 1.5 1) (thickness 0.25)))
   )
@@
   (segment (start 63.2433 46) (end 60.27 48.9733) (width 0.75) (layer B.Cu) (net 18))
   (segment (start 79.46 46) (end 63.2433 46) (width 0.75) (layer B.Cu) (net 18) (status 10))
-  (zone (net 0) (net_name "") (layer F.Mask) (hatch edge 0.508)
-    (connect_pads (clearance 0.508))
-    (min_thickness 0.254)
-    (fill yes (arc_segments 16) (thermal_gap 0.508) (thermal_bridge_width 0.508))
-    (polygon
-      (pts
-        (xy 139 54) (xy 40 54) (xy 40 29) (xy 139 29)
-      )
-    )
-  )
   (zone (net 15) (net_name AGND) (layer In1.Cu) (hatch edge 0.508)
     (connect_pads (clearance 0.508))
@@
     (connect_pads (clearance 0.508))
     (min_thickness 0.254)
-    (fill yes (arc_segments 16) (thermal_gap 0.508) (thermal_bridge_width 0.508))
-    (polygon
-      (pts
-        (xy 139 54) (xy 40 54) (xy 40 29) (xy 139 29)
-      )
-    )
-  )
-  (zone (net 0) (net_name "") (layer B.Mask) (hatch edge 0.508)
-    (connect_pads (clearance 0.508))
-    (min_thickness 0.254)

Commit message: adjust positions
Parts:
- added L501: INDUCTOR, Resistors_SMD:R_1206, F.Cu at (56.0, 31.0)
- added L502: INDUCTOR, Resistors_SMD:R_1206, F.Cu at (51.0, 31.0)
- added R102: 0R, Resistors_SMD:R_1206, F.Cu at (52.5, 55.5)
- added R103: 0R, Resistors_SMD:R_1206, F.Cu at (55.2, 55.5)
- added R513: 0R, Resistors_SMD:R_1206, F.Cu at (75.0, 48.0)
- added R514: 0R, Resistors_SMD:R_1206, F.Cu at (101.0, 45.0)
- added RV1: 1k, Potentiometers:Potentiometer_Bourns_3296W_3-8Zoll_Inline_ScrewUp, F.Cu at (91.0, 44.0)
- added RV2: 1k, Potentiometers:Potentiometer_Bourns_3296W_3-8Zoll_Inline_ScrewUp, F.Cu at (79.0, 44.0)
- P101: value CONN_01X07 -> CONN_01X11; footprint Pin_Headers:Pin_Header_Straight_1x07 -> Pin_Headers:Pin_Header_Straight_1x11
- R101: value R -> 0R
- R508: value 10k -> 15k
- moved R101 14.5 mm to (49.8, 55.5), turned to 270 degrees
- moved R505 4.00 mm to (82.0, 54.0)
- moved R508 4.00 mm to (94.0, 54.0)
- moved R510 4.00 mm to (82.0, 50.0)
- moved R512 4.00 mm to (94.0, 50.0)
- moved P101 3.16 mm to (42.0, 31.0)
- moved C503 1.00 mm to (51.0, 35.0)
- moved R504 1.00 mm to (82.0, 34.0)
- moved R507 1.00 mm to (94.0, 34.0)
- moved R509 1.00 mm to (82.0, 38.0)
- moved R511 1.00 mm to (94.0, 38.0)
Connections:
- C503 pad 1: -VE -> Net-(C503-Pad1)
- C504 pad 1: -VE -> Net-(C503-Pad1)
- C505 pad 1: -VE -> Net-(C503-Pad1)
- C506 pad 1: +VE -> Net-(C506-Pad1)
- C507 pad 1: +VE -> Net-(C506-Pad1)
- C508 pad 1: +VE -> Net-(C506-Pad1)
- P101 pad 5: REF -> V-OUT
- P101 pad 6: AGND -> Z-SENSE
- P101 pad 7: AGND -> Z-SENSE-GND
- Q502 pad 2: Net-(Q502-Pad2) -> V-OUT
- R502 pad 1: Net-(R502-Pad1) -> T-SENSE
- R503 pad 1: Net-(R502-Pad1) -> T-SENSE
- R504 pad 1: Net-(Q502-Pad2) -> Z-SENSE
- R506 pad 1: Net-(Q502-Pad2) -> V-OUT
- R506 pad 2: REF -> Z-SENSE
- R507 pad 1: Net-(Q502-Pad2) -> V-OUT
- R510 pad 1: Net-(R509-Pad2) -> Net-(R510-Pad1)
- R511 pad 2: Net-(C502-Pad1) -> Net-(R511-Pad2)
- R512 pad 1: Net-(C502-Pad1) -> Net-(R512-Pad1)
- U501 pad 2: Net-(R502-Pad1) -> T-SENSE
- U501 pad 3: Net-(R509-Pad2) -> T-SET
- U502 pad 3: REF -> Z-SENSE
- U503 pad 1: REF -> Z-SENSE
- U503 pad 2: AGND -> Z-SENSE-GND
Routing:
- net REF: track 96.9 -> 0.00 mm, vias 1 -> 0
- net V-OUT: track 0.00 -> 90.1 mm, vias 0 -> 1
- net Z-SENSE: track 0.00 -> 46.3 mm
- net Net-(Q502-Pad2): track 36.7 -> 0.00 mm
- net Net-(R510-Pad1): track 0.00 -> 21.2 mm
- net T-SENSE: track 0.00 -> 18.5 mm, vias 0 -> 2
- net Net-(R502-Pad1): track 18.5 -> 0.00 mm, vias 2 -> 0
- net Net-(R509-Pad2): track 29.7 -> 12.0 mm, vias 1 -> 0
- net Net-(R511-Pad2): track 0.00 -> 12.0 mm
- net Z-SENSE-GND: track 0.00 -> 10.6 mm
- net +VE: track 28.7 -> 19.7 mm, vias 3 -> 1
- net AGND: track 38.7 -> 29.7 mm
- net Net-(C502-Pad1): track 34.1 -> 25.6 mm
- net Net-(C503-Pad1): track 0.00 -> 7.57 mm, vias 0 -> 3
- net -VE: track 12.1 -> 4.91 mm, vias 5 -> 2
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Other:
- board size 99 x 25 mm -> 100 x 30 mm
- board text added: "H-GND"
- board text added: "T-SENSE"
- board text added: "T-SET"
- board text added: "V-OUT"
- board text added: "Ver. 0.2 (C) JA, 2017 GNU GPL"
- board text added: "Z-GND"
- board text added: "Z-SENSE"
- board text removed: "HGND"
- board text removed: "REF"
- board text removed: "Ver. 0.1 (C) JA, 2017 GNU GPL"

Commit message: update
Parts:
- removed L501, L502: INDUCTOR, Resistors_SMD:R_1206
- moved R514 5.10 mm to (102.0, 50.0)
- moved R503 5.00 mm to (61.0, 41.0), turned to 270 degrees
- moved R513 2.24 mm to (74.0, 50.0)
- moved Q501 2.00 mm to (61.0, 34.0)
- moved C503 1.60 mm to (52.0, 33.8)
- moved U503 1.50 mm to (124.0, 43.5)
- moved R502 1.41 mm to (58.0, 41.0), turned to 270 degrees
- moved C506 1.35 mm to (55.5, 33.8)
- moved C502 1.00 mm to (69.0, 50.0)
- moved R506 1.00 mm to (102.0, 36.0)
- moved RV1 1.00 mm to (92.0, 44.0)
- moved R103 0.90 mm to (56.0, 55.0)
- moved R102 0.71 mm to (53.0, 55.0)
- moved R101 0.56 mm to (50.0, 55.0)
Connections:
- C503 pad 1: Net-(C503-Pad1) -> -VE
- C504 pad 1: Net-(C503-Pad1) -> -VE
- C505 pad 1: Net-(C503-Pad1) -> -VE
- C506 pad 1: Net-(C506-Pad1) -> +VE
- C507 pad 1: Net-(C506-Pad1) -> +VE
- C508 pad 1: Net-(C506-Pad1) -> +VE
Routing:
- net (no net): track 0.00 -> 143.1 mm
- net Z-SENSE: track 46.3 -> 158.7 mm
- net Net-(Q501-Pad2): track 70.9 -> 0.00 mm
- net Z-SENSE-GND: track 10.6 -> 80.5 mm
- net H-GND: track 83.6 -> 18.2 mm, vias 1 -> 0
- net V-OUT: track 90.1 -> 26.1 mm, vias 1 -> 0
- net T-SET: track 2.24 -> 51.4 mm, vias 1 -> 0
- net AGND: track 29.7 -> 0.00 mm, vias 2 -> 0
- net Net-(C501-Pad2): track 21.4 -> 0.00 mm
- net +VE: track 19.7 -> 0.00 mm, vias 1 -> 0
- net Net-(R510-Pad1): track 21.2 -> 6.19 mm
- net Net-(R511-Pad2): track 12.0 -> 0.00 mm
- net Net-(R509-Pad2): track 12.0 -> 0.00 mm
- net Net-(C503-Pad1): track 7.57 -> 0.00 mm, vias 3 -> 0
- net Net-(C506-Pad1): track 6.56 -> 0.00 mm, vias 1 -> 0
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Other:
- outline, holes or cut-outs redrawn
- net class Default: clearance 0.25 -> 0.5
- rule trace_clearance: 0.25 -> 0.5

Commit message: ok, routed and reasonable
Parts:
- moved R101 15.0 mm to (51.0, 40.0), turned to 90 degrees
- moved R103 7.00 mm to (49.0, 55.0)
- moved C508 6.40 mm to (68.0, 48.0)
- moved R513 6.19 mm to (78.2, 54.5)
- moved U502 6.10 mm to (72.5, 48.0)
- moved R503 6.08 mm to (67.0, 40.0), turned to 90 degrees
- moved C505 5.83 mm to (77.0, 48.0)
- moved R502 5.10 mm to (63.0, 40.0), turned to 90 degrees
- moved C502 4.27 mm to (70.5, 54.0)
- moved R506 4.12 mm to (106.0, 37.0)
- moved R504 4.00 mm to (86.0, 34.0)
- moved R505 4.00 mm to (86.0, 54.0)
- moved R507 4.00 mm to (98.0, 34.0)
- moved R508 4.00 mm to (98.0, 54.0)
- moved R509 4.00 mm to (86.0, 38.0)
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Routing:
- net (no net): track 143.1 -> 0.00 mm
- net H-GND: track 18.2 -> 97.8 mm, vias 0 -> 2
- net Net-(Q501-Pad2): track 0.00 -> 70.8 mm
- net Z-SENSE: track 158.7 -> 105.3 mm, vias 0 -> 1
- net V-OUT: track 26.1 -> 72.0 mm, vias 0 -> 1
- net Z-SENSE-GND: track 80.5 -> 107.5 mm, vias 0 -> 1
- net T-SENSE: track 12.3 -> 35.7 mm, vias 0 -> 3
- net Net-(C501-Pad2): track 0.00 -> 23.0 mm
- net Net-(Q502-Pad1): track 0.00 -> 21.8 mm
- net AGND: track 0.00 -> 19.4 mm, vias 0 -> 8
- net Net-(C502-Pad1): track 25.4 -> 44.7 mm, vias 0 -> 1
- net +VE: track 0.00 -> 16.5 mm, vias 0 -> 5
- net -VE: track 0.00 -> 12.9 mm, vias 0 -> 4
- net Net-(R509-Pad2): track 0.00 -> 8.87 mm
- net Net-(R510-Pad1): track 6.19 -> 14.9 mm
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
Commit message: reset
Parts:
- moved R506 32.0 mm to (74.0, 36.0)
- moved R102 5.10 mm to (58.0, 56.0), turned to 180 degrees
- moved Q502 4.53 mm to (67.5, 33.5)
- moved R513 3.29 mm to (75.0, 55.0)
- moved R103 3.16 mm to (52.0, 56.0), turned to 0 degrees
- moved R504 3.00 mm to (83.0, 34.0)
- moved R505 3.00 mm to (83.0, 54.0)
- moved R507 3.00 mm to (95.0, 34.0)
- moved R508 3.00 mm to (95.0, 54.0)
- moved R509 3.00 mm to (83.0, 38.0)
- moved R510 3.00 mm to (83.0, 50.0)
- moved R511 3.00 mm to (95.0, 38.0)
- moved R512 3.00 mm to (95.0, 50.0)
- moved R514 3.00 mm to (103.0, 50.0)
- moved RV1 3.00 mm to (92.0, 44.0)
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Routing:
- net Z-SENSE-GND: track 107.5 -> 9.23 mm, vias 1 -> 0
- net H-GND: track 97.8 -> 0.00 mm, vias 2 -> 0
- net Net-(Q501-Pad2): track 70.8 -> 0.00 mm
- net (no net): track 0.00 -> 69.4 mm
- net Net-(R503-Pad2): track 58.2 -> 0.00 mm
- net T-SET: track 57.1 -> 0.00 mm
- net V-OUT: track 72.0 -> 23.7 mm, vias 1 -> 0
- net Net-(C502-Pad1): track 44.7 -> 6.19 mm, vias 1 -> 0
- net T-SENSE: track 35.7 -> 4.00 mm, vias 3 -> 0
- net Net-(C501-Pad2): track 23.0 -> 0.00 mm
- net Net-(Q502-Pad1): track 21.8 -> 0.00 mm
- net AGND: track 19.4 -> 3.10 mm, vias 8 -> 0
- net Net-(R510-Pad1): track 14.9 -> 0.00 mm
- net Z-SENSE: track 105.3 -> 91.9 mm, vias 1 -> 0
- net Net-(R507-Pad2): track 4.00 -> 13.5 mm
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
Commit message: fix
Routing:
- net Z-SENSE: track 91.9 -> 0.00 mm
- net (no net): track 69.4 -> 0.00 mm
- net Net-(R512-Pad1): track 26.2 -> 0.00 mm
- net V-OUT: track 23.7 -> 0.00 mm
- net Net-(R507-Pad2): track 13.5 -> 0.00 mm
- net Z-SENSE-GND: track 9.23 -> 0.00 mm
- net Net-(R508-Pad1): track 8.87 -> 0.00 mm
Changed lines of the file:
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@@
   (general
     (links 65)
-    (no_connects 54)
+    (no_connects 59)
     (area 38.949999 28.949999 139.050001 59.050001)
     (thickness 1.6)
     (drawings 21)
-    (tracks 54)
+    (tracks 20)
     (zones 0)
     (modules 33)
@@
     (1 In1.Cu signal hide)
     (2 In2.Cu signal hide)
-    (31 B.Cu signal hide)
+    (31 B.Cu signal)
     (33 F.Adhes user hide)
     (36 B.SilkS user hide)
@@
     (effects (font (size 1.5 1) (thickness 0.25)) (justify left))
   )
-  (segment (start 101.2519 56.1395) (end 102.3206 55.0708) (width 0.75) (layer B.Cu) (net 0))
-  (segment (start 60.7505 56.1395) (end 101.2519 56.1395) (width 0.75) (layer B.Cu) (net 0))
-  (segment (start 49.9701 45.3591) (end 60.7505 56.1395) (width 0.75) (layer B.Cu) (net 0))
-  (segment (start 52.0476 45.1778) (end 55.424 48.5542) (width 0.75) (layer B.Cu) (net 0))
-  (segment (start 57.6553 48.5542) (end 55.424 48.5542) (width 0.75) (layer B.Cu) (net 0))
-  (segment (start 61.2588 44.9507) (end 57.6553 48.5542) (width 0.75) (layer B.Cu) (net 0))
   (segment (start 57.365 45.3) (end 57.365 46.635) (width 0.75) (layer F.Cu) (net 1))
   (segment (start 57 47) (end 54 47) (width 0.75) (layer F.Cu) (net 1))
@@
   (segment (start 88.08 44) (end 88.08 40.9941) (width 0.75) (layer In1.Cu) (net 6))
   (segment (start 83.46 38) (end 85.0859 38) (width 0.75) (layer In1.Cu) (net 6))
-  (segment (start 97.0859 46.9941) (end 100.08 44) (width 0.75) (layer B.Cu) (net 9))
-  (segment (start 97.0859 50) (end 97.0859 46.9941) (width 0.75) (layer B.Cu) (net 9))
-  (segment (start 95.46 50) (end 97.0859 50) (width 0.75) (layer B.Cu) (net 9))
   (segment (start 53.45 56) (end 56.55 56) (width 0.75) (layer F.Cu) (net 12))
-  (segment (start 104.9952 31.8293) (end 106 32.8341) (width 0.75) (layer B.Cu) (net 14))
-  (segment (start 99.2566 31.8293) (end 104.9952 31.8293) (width 0.75) (layer B.Cu) (net 14))
-  (segment (start 97.0859 34) (end 99.2566 31.8293) (width 0.75) (layer B.Cu) (net 14))
-  (segment (start 106 34.46) (end 106 32.8341) (width 0.75) (layer B.Cu) (net 14))
-  (segment (start 95.46 34) (end 97.0859 34) (width 0.75) (layer B.Cu) (net 14))
-  (segment (start 58.5877 41.16) (end 63.6136 36.1341) (width 0.75) (layer B.Cu) (net 16))
-  (segment (start 42 41.16) (end 58.5877 41.16) (width 0.75) (layer B.Cu) (net 16))
-  (segment (start 83.46 34) (end 81.8341 34) (width 0.75) (layer B.Cu) (net 17))
-  (segment (start 42 43.7) (end 43.8913 43.7) (width 0.75) (layer B.Cu) (net 17))
-  (segment (start 44.0648 43.5265) (end 43.8913 43.7) (width 0.75) (layer B.Cu) (net 17))
-  (segment (start 71.2233 43.5265) (end 44.0648 43.5265) (width 0.75) (layer B.Cu) (net 17))
-  (segment (start 74.8111 47.1143) (end 71.2233 43.5265) (width 0.75) (layer B.Cu) (net 17))
-  (segment (start 81.8341 40.0913) (end 74.8111 47.1143) (width 0.75) (layer B.Cu) (net 17))
-  (segment (start 81.8341 34) (end 81.8341 40.0913) (width 0.75) (layer B.Cu) (net 17))
-  (segment (start 106 39.54) (end 74.8749 38.54) (width 0.75) (layer B.Cu) (net 17) (status 20))
-  (segment (start 81.9204 40.1776) (end 81.8341 40.0913) (width 0.75) (layer B.Cu) (net 17))
-  (segment (start 74.2373 39.1776) (end 81.9204 40.1776) (width 0.75) (layer B.Cu) (net 17) (status 10))
-  (segment (start 74.8749 38.54) (end 74.2373 39.1776) (width 0.75) (layer B.Cu) (net 17) (status 30))
-  (segment (start 43.8913 50.7183) (end 45.9108 52.7378) (width 0.75) (layer B.Cu) (net 18))
-  (segment (start 43.8913 46.24) (end 43.8913 50.7183) (width 0.75) (layer B.Cu) (net 18))
-  (segment (start 42 46.24) (end 43.8913 46.24) (width 0.75) (layer B.Cu) (net 18))
   (segment (start 63 40.95) (end 67 40.95) (width 0.75) (layer F.Cu) (net 19) (status 20))
-  (segment (start 94.0431 47.4969) (end 97.54 44) (width 0.75) (layer B.Cu) (net 23))
-  (segment (start 83.0793 47.4969) (end 94.0431 47.4969) (width 0.75) (layer B.Cu) (net 23))
-  (segment (start 78.0788 52.4974) (end 83.0793 47.4969) (width 0.75) (layer B.Cu) (net 23))
-  (segment (start 74.9072 52.4974) (end 78.0788 52.4974) (width 0.75) (layer B.Cu) (net 23))
   (zone (net 12) (net_name AGND) (layer In1.Cu) (hatch edge 0.508)
     (connect_pads (clearance 0.508))

Commit message: before ses import
Parts:
- moved R102 0.50 mm to (58.0, 55.5)
- moved R103 0.50 mm to (52.0, 55.5)
Routing:
- net Net-(R504-Pad2): track 8.87 -> 0.00 mm
- net Net-(C502-Pad1): track 6.19 -> 0.00 mm
Other:
- board size 100 x 30 mm -> 100 x 31 mm
Changed lines of the file:
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@@
   (general
     (links 65)
-    (no_connects 59)
-    (area 38.949999 28.949999 139.050001 59.050001)
+    (no_connects 55)
+    (area 38.949999 28.949999 139.050001 60.050001)
     (thickness 1.6)
-    (drawings 21)
-    (tracks 20)
+    (drawings 25)
+    (tracks 14)
     (zones 0)
     (modules 33)
@@
     (43 Eco2.User user hide)
     (44 Edge.Cuts user)
-    (45 Margin user)
+    (45 Margin user hide)
     (47 F.CrtYd user hide)
     (49 F.Fab user hide)
@@
   )
   (module Resistors_SMD:R_1206 (layer F.Cu)
-    (at 58 56 180)
+    (at 58 55.5 180)
     (descr "Resistor SMD 1206, reflow soldering, Vishay (see dcrcw.pdf)")
     (tags "resistor 1206")
@@
   )
   (module Resistors_SMD:R_1206 (layer F.Cu)
-    (at 52 56)
+    (at 52 55.5)
     (descr "Resistor SMD 1206, reflow soldering, Vishay (see dcrcw.pdf)")
     (tags "resistor 1206")
@@
     )
   )
+  (gr_line (start 39 59) (end 39 60) (angle 90) (layer Edge.Cuts) (width 0.1))
+  (gr_line (start 139 59) (end 139 60) (angle 90) (layer Edge.Cuts) (width 0.1))
+  (gr_line (start 139 60) (end 139 59) (angle 90) (layer Margin) (width 0.2))
+  (gr_line (start 39 60) (end 139 60) (angle 90) (layer Margin) (width 0.2))
+  (gr_line (start 39 59) (end 39 60) (angle 90) (layer Margin) (width 0.2))
   (gr_line (start 39 30) (end 39 29) (angle 90) (layer Margin) (width 0.2))
   (gr_line (start 39 59) (end 39 30) (angle 90) (layer Margin) (width 0.2))
-  (gr_line (start 137 59) (end 37 59) (angle 90) (layer Margin) (width 0.2))
   (gr_line (start 139 29) (end 139 59) (angle 90) (layer Margin) (width 0.2))
   (gr_line (start 39 29) (end 139 29) (angle 90) (layer Margin) (width 0.2))
   (gr_line (start 39 59) (end 39 29) (angle 90) (layer Edge.Cuts) (width 0.1))
-  (gr_line (start 139 59) (end 39 59) (angle 90) (layer Edge.Cuts) (width 0.1))
+  (gr_line (start 139 60) (end 39 60) (angle 90) (layer Edge.Cuts) (width 0.1))
   (gr_line (start 139 29) (end 139 59) (angle 90) (layer Edge.Cuts) (width 0.1))
   (gr_line (start 39 29) (end 139 29) (angle 90) (layer Edge.Cuts) (width 0.1))
@@
   (segment (start 75 49.5) (end 73.605 49.5) (width 0.75) (layer F.Cu) (net 2))
   (segment (start 73.605 49.5) (end 72.405 50.7) (width 0.75) (layer F.Cu) (net 2))
-  (segment (start 95 40.5851) (end 95.46 40.1251) (width 0.75) (layer In1.Cu) (net 5))
-  (segment (start 95 44) (end 95 40.5851) (width 0.75) (layer In1.Cu) (net 5))
-  (segment (start 95.46 38) (end 95.46 40.1251) (width 0.75) (layer In1.Cu) (net 5))
-  (segment (start 88.08 40.9941) (end 85.0859 38) (width 0.75) (layer In1.Cu) (net 6))
-  (segment (start 88.08 44) (end 88.08 40.9941) (width 0.75) (layer In1.Cu) (net 6))
-  (segment (start 83.46 38) (end 85.0859 38) (width 0.75) (layer In1.Cu) (net 6))
-  (segment (start 53.45 56) (end 56.55 56) (width 0.75) (layer F.Cu) (net 12))
+  (segment (start 53.45 55.5) (end 56.55 55.5) (width 0.75) (layer F.Cu) (net 12) (status 20))
   (segment (start 63 40.95) (end 67 40.95) (width 0.75) (layer F.Cu) (net 19) (status 20))
   (zone (net 12) (net_name AGND) (layer In1.Cu) (hatch edge 0.508)
@@
     (polygon
       (pts
-        (xy 139 59) (xy 39 59) (xy 39 29) (xy 139 29)
+        (xy 139 60) (xy 39 60) (xy 39 29) (xy 139 29)
       )
     )
@@
     (polygon
       (pts
-        (xy 139 59) (xy 39 59) (xy 39 29) (xy 139 29)
+        (xy 139 60) (xy 39 60) (xy 39 29) (xy 139 29)
       )
     )
@@
     (polygon
       (pts
-        (xy 139 59) (xy 39 59) (xy 39 29) (xy 139 29)
+        (xy 139 60) (xy 39 60) (xy 39 29) (xy 139 29)
       )
     )
