File: projects/dw232/main.kicad_pcb (KiCad board)
At the start: 4 copper layers, 100 x 31 mm, 33 parts, among them P101 CONN_01X11, Q501 MMBT3904, Q502 MMBT3904, U501 LM741, U502 LM741, U503 2DW232

Commit message: update
Parts:
- moved R513 28.0 mm to (103.0, 55.0)
- moved R503 1.50 mm to (68.5, 39.5)
- moved P101 0.71 mm to (41.5, 31.5)
- moved R502 0.50 mm to (63.5, 39.5)
- moved R506 0.50 mm to (73.5, 36.0)
- moved R514 0.50 mm to (103.0, 49.5)
Routing:
- net T-SENSE: track 4.00 -> 0.00 mm
- net AGND: track 3.10 -> 0.00 mm
Changed lines of the file:
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@@
   (general
     (links 65)
-    (no_connects 55)
+    (no_connects 60)
     (area 38.949999 28.949999 139.050001 60.050001)
     (thickness 1.6)
@@
     (1 In1.Cu signal hide)
     (2 In2.Cu signal hide)
-    (31 B.Cu signal)
+    (31 B.Cu signal hide)
     (33 F.Adhes user hide)
     (36 B.SilkS user hide)
@@
     (pad_to_mask_clearance 0)
     (aux_axis_origin 0 0)
+    (grid_origin 103 55)
     (visible_elements FFFEFF7F)
     (pcbplotparams
@@
   )
   (module Resistors_SMD:R_1206 (layer F.Cu)
-    (at 63 39.5 90)
+    (at 63.5 39.5 90)
     (descr "Resistor SMD 1206, reflow soldering, Vishay (see dcrcw.pdf)")
     (tags "resistor 1206")
@@
   )
   (module Resistors_SMD:R_1206 (layer F.Cu)
-    (at 67 39.5 90)
+    (at 68.5 39.5 90)
     (descr "Resistor SMD 1206, reflow soldering, Vishay (see dcrcw.pdf)")
     (tags "resistor 1206")
@@
   )
   (module Resistors_ThroughHole:Resistor_TO-220_Vertical (layer F.Cu)
-    (at 74 36 270)
+    (at 73.5 36 270)
     (descr "Resistor, TO-220, Vertical,")
     (tags "Resistor, TO-220, Vertical,")
@@
   )
   (module Pin_Headers:Pin_Header_Straight_1x11 (layer F.Cu)
-    (at 42 31)
+    (at 41.5 31.5)
     (descr "Through hole pin header")
     (tags "pin header")
@@
   )
   (module Resistors_SMD:R_1206 (layer F.Cu)
-    (at 75 55 90)
+    (at 103 55 90)
     (descr "Resistor SMD 1206, reflow soldering, Vishay (see dcrcw.pdf)")
     (tags "resistor 1206")
@@
   )
   (module Resistors_SMD:R_1206 (layer F.Cu)
-    (at 103 50 90)
+    (at 103 49.5 90)
     (descr "Resistor SMD 1206, reflow soldering, Vishay (see dcrcw.pdf)")
     (tags "resistor 1206")
@@
   (gr_line (start 139 29) (end 139 59) (angle 90) (layer Edge.Cuts) (width 0.1))
   (gr_line (start 39 29) (end 139 29) (angle 90) (layer Edge.Cuts) (width 0.1))
-  (gr_text AGND (at 44 56.4) (layer F.SilkS)
+  (gr_text AGND (at 44 56.9) (layer F.SilkS)
     (effects (font (size 1.5 1) (thickness 0.25)) (justify left))
   )
-  (gr_text AGND (at 44 54) (layer F.SilkS)
+  (gr_text AGND (at 44 54.5) (layer F.SilkS)
     (effects (font (size 1.5 1) (thickness 0.25)) (justify left))
   )
-  (gr_text T-SET (at 44 51.4) (layer F.SilkS)
+  (gr_text T-SET (at 44 51.9) (layer F.SilkS)
     (effects (font (size 1.5 1) (thickness 0.25)) (justify left))
   )
-  (gr_text Z-SENSE (at 44 43.8) (layer F.SilkS)
+  (gr_text Z-SENSE (at 44 44.3) (layer F.SilkS)
     (effects (font (size 1.5 1) (thickness 0.25)) (justify left))
   )
@@
     (effects (font (size 1.5 1) (thickness 0.25)))
   )
-  (gr_text T-SENSE (at 44 48.8) (layer F.SilkS)
+  (gr_text T-SENSE (at 44 49.3) (layer F.SilkS)
     (effects (font (size 1.5 1) (thickness 0.25)) (justify left))
   )
-  (gr_text Z-GND (at 44 46.2) (layer F.SilkS)
+  (gr_text Z-GND (at 44 46.7) (layer F.SilkS)
     (effects (font (size 1.5 1) (thickness 0.25)) (justify left))
   )
-  (gr_text V-OUT (at 44 41.25) (layer F.SilkS)
+  (gr_text V-OUT (at 44 41.75) (layer F.SilkS)
     (effects (font (size 1.5 1) (thickness 0.25)) (justify left))
   )
-  (gr_text "H-GND\n" (at 44 38.6) (layer F.SilkS)
+  (gr_text "H-GND\n" (at 44 39.1) (layer F.SilkS)
     (effects (font (size 1.5 1) (thickness 0.25)) (justify left))
   )
-  (gr_text "-VE\n" (at 44 36) (layer F.SilkS)
+  (gr_text "-VE\n" (at 44 36.5) (layer F.SilkS)
     (effects (font (size 1.5 1) (thickness 0.25)) (justify left))
   )
-  (gr_text AGND (at 44 33.5) (layer F.SilkS)
+  (gr_text AGND (at 44 34) (layer F.SilkS)
     (effects (font (size 1.5 1) (thickness 0.25)) (justify left))
   )
-  (gr_text +VE (at 44 31) (layer F.SilkS)
+  (gr_text +VE (at 44 31.5) (layer F.SilkS)
     (effects (font (size 1.5 1) (thickness 0.25)) (justify left))
   )
   (segment (start 57.365 45.3) (end 57.365 46.635) (width 0.75) (layer F.Cu) (net 1))
-  (segment (start 57 47) (end 54 47) (width 0.75) (layer F.Cu) (net 1))
+  (segment (start 54.5 47) (end 53.75 47) (width 0.75) (layer F.Cu) (net 1))
+  (segment (start 57 47) (end 54.5 47) (width 0.75) (layer F.Cu) (net 1))
   (segment (start 57.365 46.635) (end 57 47) (width 0.75) (layer F.Cu) (net 1))
-  (segment (start 54 47) (end 53.5 46.5) (width 0.75) (layer F.Cu) (net 1))
+  (segment (start 53.75 47) (end 53.5 46.75) (width 0.75) (layer F.Cu) (net 1))
+  (segment (start 53.5 46.75) (end 53.5 46.5) (width 0.75) (layer F.Cu) (net 1))
   (segment (start 69.865 45.3) (end 69.865 46.635) (width 0.75) (layer F.Cu) (net 1))
-  (segment (start 69.5 47) (end 66 47) (width 0.75) (layer F.Cu) (net 1))
+  (segment (start 69.5 47) (end 66.5 47) (width 0.75) (layer F.Cu) (net 1))
   (segment (start 69.865 46.635) (end 69.5 47) (width 0.75) (layer F.Cu) (net 1))
-  (segment (start 66 47) (end 66 46.5) (width 0.75) (layer F.Cu) (net 1))
+  (segment (start 66.5 47) (end 66 46.5) (width 0.75) (layer F.Cu) (net 1))
   (segment (start 62.5 49.5) (end 61.105 49.5) (width 0.75) (layer F.Cu) (net 2))
   (segment (start 61.105 49.5) (end 59.905 50.7) (width 0.75) (layer F.Cu) (net 2))
   (segment (start 75 49.5) (end 73.605 49.5) (width 0.75) (layer F.Cu) (net 2))
   (segment (start 73.605 49.5) (end 72.405 50.7) (width 0.75) (layer F.Cu) (net 2))
-  (segment (start 53.45 55.5) (end 56.55 55.5) (width 0.75) (layer F.Cu) (net 12) (status 20))
-  (segment (start 63 40.95) (end 67 40.95) (width 0.75) (layer F.Cu) (net 19) (status 20))
   (zone (net 12) (net_name AGND) (layer In1.Cu) (hatch edge 0.508)
     (connect_pads (clearance 0.508))
