File: projects/dw232/main.kicad_pcb (KiCad board)
At the start: 4 copper layers, 100 x 31 mm, 33 parts, among them P101 CONN_01X11, Q501 MMBT3904, Q502 MMBT3904, U501 LM741, U502 LM741, U503 2DW232

Commit message: better
Parts:
- moved R513 28.0 mm to (75.0, 54.0)
- moved RV1 1.00 mm to (93.0, 44.0)
- moved U503 0.50 mm to (124.0, 44.0)
Routing:
- net Net-(R510-Pad1): track 40.0 -> 15.5 mm, vias 2 -> 0
- net H-GND: track 106.8 -> 96.2 mm, vias 3 -> 2
- net T-SET: track 71.7 -> 64.1 mm
- net Z-SENSE: track 117.3 -> 112.4 mm, vias 2 -> 1
- net T-SENSE: track 41.3 -> 46.0 mm, vias 2 -> 1
- net V-OUT: track 62.4 -> 58.2 mm, vias 1 -> 0
- net Net-(R503-Pad2): track 57.7 -> 61.4 mm, vias 2 -> 0
- net AGND: track 21.5 -> 18.8 mm, vias 9 -> 10
- net Net-(C501-Pad2): track 21.9 -> 19.4 mm
- net Z-SENSE-GND: track 110.3 -> 107.8 mm, vias 1 -> 0
- net -VE: track 16.4 -> 14.1 mm
- net Net-(Q502-Pad1): track 12.7 -> 14.7 mm, vias 2 -> 0
- net +VE: track 21.4 -> 19.6 mm
- net Net-(Q501-Pad2): track 69.7 -> 70.9 mm, vias 2 -> 0
- net Net-(R512-Pad1): track 17.2 -> 16.4 mm
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Other:
- board text removed: "+VE"
- board text removed: "-VE"
- board text removed: "AGND"
- board text removed: "H-GND"
- board text removed: "T-SENSE"
- board text removed: "T-SET"
- board text removed: "V-OUT"
- board text removed: "Ver. 0.2 (C) JA, 2017 GNU GPL"
- board text removed: "Z-GND"
- board text removed: "Z-SENSE"

Commit message: fill in gnd
Routing:
- net H-GND: track 96.2 -> 94.2 mm, vias 2 -> 3
Other:
- board text added: "+VE"
- board text added: "-VE"
- board text added: "AGND"
- board text added: "H-GND"
- board text added: "T-SENSE"
- board text added: "T-SET"
- board text added: "V-OUT"
- board text added: "Z-GND"
- board text added: "Z-SENSE"
Changed lines of the file:
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@@
     (area 38.949999 28.949999 139.050001 60.050001)
     (thickness 1.6)
-    (drawings 13)
-    (tracks 253)
+    (drawings 24)
+    (tracks 256)
     (zones 0)
     (modules 33)
@@
     (1 In1.Cu signal hide)
     (2 In2.Cu signal hide)
-    (31 B.Cu signal hide)
+    (31 B.Cu signal)
     (33 F.Adhes user hide)
     (36 B.SilkS user hide)
@@
     (descr "Through hole pin header")
     (tags "pin header")
-    (fp_text reference P101 (at 5 27 180) (layer F.SilkS)
+    (fp_text reference P101 (at 5 27.25 180) (layer F.SilkS)
       (effects (font (size 1 1) (thickness 0.15)))
     )
@@
       (rotate (xyz 0 0 0))
     )
+  )
+  (gr_text AGND (at 44 57) (layer F.SilkS)
+    (effects (font (size 1.5 1) (thickness 0.25)) (justify left))
+  )
+  (gr_text AGND (at 44 54.5) (layer F.SilkS)
+    (effects (font (size 1.5 1) (thickness 0.25)) (justify left))
+  )
+  (gr_text T-SET (at 44 52) (layer F.SilkS)
+    (effects (font (size 1.5 1) (thickness 0.25)) (justify left))
+  )
+  (gr_text T-SENSE (at 44 49.5) (layer F.SilkS)
+    (effects (font (size 1.5 1) (thickness 0.25)) (justify left))
+  )
+  (gr_text Z-GND (at 49.25 46.75) (layer F.SilkS)
+    (effects (font (size 1.5 1) (thickness 0.25)) (justify right))
+  )
+  (gr_text Z-SENSE (at 47.5 44.25) (layer F.SilkS)
+    (effects (font (size 1.5 1) (thickness 0.25)))
+  )
+  (gr_text V-OUT (at 46.5 41.75) (layer F.SilkS)
+    (effects (font (size 1.5 1) (thickness 0.25)))
+  )
+  (gr_text "H-GND\n" (at 46.5 39) (layer F.SilkS)
+    (effects (font (size 1.5 1) (thickness 0.25)))
+  )
+  (gr_text "-VE\n" (at 45.5 36.5) (layer F.SilkS)
+    (effects (font (size 1.5 1) (thickness 0.25)))
+  )
+  (gr_text AGND (at 46 34) (layer F.SilkS)
+    (effects (font (size 1.5 1) (thickness 0.25)))
+  )
+  (gr_text +VE (at 45.5 31.5) (layer F.SilkS)
+    (effects (font (size 1.5 1) (thickness 0.25)))
   )
   (gr_line (start 39 59) (end 39 60) (angle 90) (layer Edge.Cuts) (width 0.1))
@@
   (segment (start 56.893 34.9479) (end 56.6753 34.7302) (width 0.75) (layer F.Cu) (net 12))
   (segment (start 55 34.5) (end 56.6753 34.5) (width 0.75) (layer F.Cu) (net 12))
-  (via (at 46.9255 42.4361) (size 1) (layers F.Cu B.Cu) (net 13))
+  (segment (start 48 41.5) (end 45.75 39.25) (width 0.75) (layer B.Cu) (net 13))
+  (segment (start 45.62 39.12) (end 41.5 39.12) (width 0.75) (layer F.Cu) (net 13))
+  (segment (start 45.75 39.25) (end 45.62 39.12) (width 0.75) (layer F.Cu) (net 13))
+  (via (at 45.75 39.25) (size 1) (drill 0.5) (layers F.Cu B.Cu) (net 13))
+  (via (at 48 41.5) (size 1) (layers F.Cu B.Cu) (net 13))
   (via (at 83.6252 38.5925) (size 1) (layers F.Cu B.Cu) (net 13))
   (segment (start 51 41.45) (end 49.2747 41.45) (width 0.75) (layer F.Cu) (net 13))
-  (segment (start 41.5 39.12) (end 43.3913 39.12) (width 0.75) (layer B.Cu) (net 13))
   (segment (start 118.7513 46.794) (end 124 46.794) (width 0.75) (layer F.Cu) (net 13))
   (segment (start 112.0824 40.1251) (end 118.7513 46.794) (width 0.75) (layer F.Cu) (net 13))
@@
   (segment (start 83.6252 38.5925) (end 83.6252 38.8886) (width 0.75) (layer F.Cu) (net 13))
   (segment (start 47.9116 41.45) (end 49.2747 41.45) (width 0.75) (layer F.Cu) (net 13))
-  (segment (start 46.9255 42.4361) (end 47.9116 41.45) (width 0.75) (layer F.Cu) (net 13))
-  (segment (start 46.7074 42.4361) (end 46.9255 42.4361) (width 0.75) (layer B.Cu) (net 13))
-  (segment (start 43.3913 39.12) (end 46.7074 42.4361) (width 0.75) (layer B.Cu) (net 13))
+  (segment (start 48 41.5) (end 47.9116 41.45) (width 0.75) (layer F.Cu) (net 13))
   (segment (start 82.0502 40.1675) (end 83.6252 38.5925) (width 0.75) (layer B.Cu) (net 13))
   (segment (start 79.4072 40.1675) (end 82.0502 40.1675) (width 0.75) (layer B.Cu) (net 13))
   (segment (start 76.1537 36.914) (end 79.4072 40.1675) (width 0.75) (layer B.Cu) (net 13))
   (segment (start 52.4476 36.914) (end 76.1537 36.914) (width 0.75) (layer B.Cu) (net 13))
-  (segment (start 46.9255 42.4361) (end 52.4476 36.914) (width 0.75) (layer B.Cu) (net 13))
+  (segment (start 48 41.5) (end 52.4476 36.914) (width 0.75) (layer B.Cu) (net 13))
   (segment (start 97.54 38) (end 97.54 34) (width 0.75) (layer F.Cu) (net 14))
   (segment (start 81.2051 40.1251) (end 80.46 40.1251) (width 0.75) (layer F.Cu) (net 15))
   (segment (start 85.08 44) (end 81.2051 40.1251) (width 0.75) (layer F.Cu) (net 15))
   (segment (start 80.46 38) (end 80.46 40.1251) (width 0.75) (layer F.Cu) (net 15))
+  (segment (start 50 37.1108) (end 49.8892 37.1108) (width 0.75) (layer F.Cu) (net 16))
+  (segment (start 45.34 41.66) (end 43.734 41.66) (width 0.75) (layer F.Cu) (net 16))
+  (segment (start 49.8892 37.1108) (end 45.34 41.66) (width 0.75) (layer F.Cu) (net 16))
   (segment (start 70.4649 32.55) (end 68.5008 32.55) (width 0.75) (layer F.Cu) (net 16))
   (segment (start 71.3749 33.46) (end 70.4649 32.55) (width 0.75) (layer F.Cu) (net 16))
@@
   (segment (start 64.0756 34.4239) (end 64.0756 33.8739) (width 0.75) (layer F.Cu) (net 16))
   (segment (start 61.3887 37.1108) (end 64.0756 34.4239) (width 0.75) (layer F.Cu) (net 16))
-  (segment (start 48.2832 37.1108) (end 61.3887 37.1108) (width 0.75) (layer F.Cu) (net 16))
-  (segment (start 43.734 41.66) (end 48.2832 37.1108) (width 0.75) (layer F.Cu) (net 16))
+  (segment (start 50 37.1108) (end 61.3887 37.1108) (width 0.75) (layer F.Cu) (net 16))
   (segment (start 41.5 41.66) (end 43.734 41.66) (width 0.75) (layer F.Cu) (net 16))
-  (via (at 71.1879 47.3228) (size 1) (layers F.Cu B.Cu) (net 17))
+  (via (at 71.25 47.25) (size 1) (layers F.Cu B.Cu) (net 17))
   (segment (start 73.5 38.54) (end 71.3749 38.54) (width 0.75) (layer B.Cu) (net 17))
   (segment (start 80.46 34) (end 82.0859 34) (width 0.75) (layer F.Cu) (net 17))
@@
   (segment (start 82.0859 39.1176) (end 84.963 41.9947) (width 0.75) (layer F.Cu) (net 17))
   (segment (start 82.0859 34) (end 82.0859 39.1176) (width 0.75) (layer F.Cu) (net 17))
-  (segment (start 71.135 47.3757) (end 71.1879 47.3228) (width 0.75) (layer F.Cu) (net 17))
-  (segment (start 71.135 50.7) (end 71.135 47.3757) (width 0.75) (layer F.Cu) (net 17))
-  (segment (start 71.1879 43.4704) (end 71.1879 47.3228) (width 0.75) (layer B.Cu) (net 17))
+  (segment (start 71.1971 47.3029) (end 71.25 47.25) (width 0.75) (layer F.Cu) (net 17))
+  (segment (start 71.135 50.7) (end 71.1971 47.3029) (width 0.75) (layer F.Cu) (net 17))
+  (segment (start 71.1879 43.4704) (end 71.25 47.25) (width 0.75) (layer B.Cu) (net 17))
   (segment (start 71.3749 43.2834) (end 71.1879 43.4704) (width 0.75) (layer B.Cu) (net 17))
   (segment (start 71.3749 38.54) (end 71.3749 43.2834) (width 0.75) (layer B.Cu) (net 17))
