File: projects/dw232/2dw232-ref.sch (KiCad schematic (older format))
At the start: 25 parts, among them Q501 MMBT3904, Q502 MMBT3904, U501 LM741, U502 LM741, U503 2DW232

Commit message: annotate component values
Parts:
- gave numbers to parts that had none: 5
Other:
- moved on the sheet: C501, R508, R512
Changed lines of the file:
@@
 L R R508
 U 1 1 5881849D
-P 6300 3300
-F 0 "R508" V 6380 3300 50  0000 C CNN
-F 1 "10k" V 6300 3300 50  0000 C CNN
-F 2 "Resistors_ThroughHole:Resistor_TO-220_Vertical" V 6230 3300 50  0001 C CNN
-F 3 "" H 6300 3300 50  0000 C CNN
-	1    6300 3300
+P 6300 3350
+F 0 "R508" V 6380 3350 50  0000 C CNN
+F 1 "10k" V 6300 3350 50  0000 C CNN
+F 2 "Resistors_ThroughHole:Resistor_TO-220_Vertical" V 6230 3350 50  0001 C CNN
+F 3 "" H 6300 3350 50  0000 C CNN
+	1    6300 3350
 	1    0    0    -1
 $EndComp
@@
 $EndComp
 Wire Wire Line
-	3850 1650 8750 1650
+	3850 1650 4450 1650
+Wire Wire Line
+	4450 1650 6300 1650
+Wire Wire Line
+	6300 1650 8750 1650
 Wire Wire Line
 	6300 1650 6300 1750
 Wire Wire Line
-	6300 2400 6300 2750
+	6300 2400 6300 2650
+Wire Wire Line
+	6300 2650 6300 2800
 Text GLabel 7300 2200 1    60   Input ~ 0
 +VE
@@
 AGND
 Wire Wire Line
-	6300 2650 7100 2650
+	6300 2650 6700 2650
+Wire Wire Line
+	6700 2650 7100 2650
 Connection ~ 6300 2650
 Wire Wire Line
-	4150 2450 7100 2450
-Wire Wire Line
-	3850 4150 6700 4150
+	4150 2450 4450 2450
+Wire Wire Line
+	4450 2450 7100 2450
+Wire Wire Line
+	3850 4150 4450 4150
+Wire Wire Line
+	4450 4150 6300 4150
+Wire Wire Line
+	6300 4150 6700 4150
 Connection ~ 6300 4150
 $Comp
@@
 $EndComp
 Wire Wire Line
-	2500 3000 3150 3000
+	2500 3000 3000 3000
+Wire Wire Line
+	3000 3000 3150 3000
 Wire Wire Line
 	3000 3000 3000 3600
@@
 L C C501
 U 1 1 5881B5FE
-P 1900 3250
-F 0 "C501" H 1925 3350 50  0000 L CNN
-F 1 "10uF" H 1925 3150 50  0000 L CNN
-F 2 "Capacitors_SMD:C_1206" H 1938 3100 50  0001 C CNN
-F 3 "" H 1900 3250 50  0000 C CNN
-	1    1900 3250
-	1    0    0    -1
-$EndComp
-Wire Wire Line
-	1700 3000 2200 3000
-Wire Wire Line
-	1900 3000 1900 3100
-Wire Wire Line
-	1900 3400 1900 3500
-Wire Wire Line
-	1650 3500 2200 3500
+P 1950 3250
+F 0 "C501" H 1975 3350 50  0000 L CNN
+F 1 "10uF" H 1975 3150 50  0000 L CNN
+F 2 "Capacitors_SMD:C_1206" H 1988 3100 50  0001 C CNN
+F 3 "" H 1950 3250 50  0000 C CNN
+	1    1950 3250
+	1    0    0    -1
+$EndComp
+Wire Wire Line
+	1700 3000 1950 3000
+Wire Wire Line
+	1950 3000 2200 3000
+Wire Wire Line
+	1950 3000 1950 3100
+Wire Wire Line
+	1950 3400 1950 3500
+Wire Wire Line
+	1650 3500 1700 3500
+Wire Wire Line
+	1700 3500 1950 3500
+Wire Wire Line
+	1950 3500 2200 3500
 Text GLabel 2600 2700 1    60   Input ~ 0
 +VE
 Wire Wire Line
 	2600 2700 2600 3200
-Connection ~ 1900 3500
+Connection ~ 1950 3500
 Text GLabel 1350 2700 1    60   Input ~ 0
 +VE
@@
 NoConn ~ 2500 3800
 Wire Wire Line
-	6300 3450 6300 4150
+	6300 3500 6300 4150
 Wire Wire Line
 	3850 4100 3850 4150
 Wire Wire Line
-	6700 3550 6700 4400
+	6700 3550 6700 4150
+Wire Wire Line
+	6700 4150 6700 4400
 Connection ~ 6700 4150
 Wire Wire Line
-	6300 3050 6300 3150
+	6300 3100 6300 3200
 $Comp
 L C C503
@@
 	1850 950  1850 1100
 Wire Wire Line
-	1850 1100 2450 1100
-Wire Wire Line
-	1850 1400 2450 1400
+	1850 1100 2150 1100
+Wire Wire Line
+	2150 1100 2450 1100
+Wire Wire Line
+	1850 1400 2150 1400
+Wire Wire Line
+	2150 1400 2450 1400
 Connection ~ 2150 1100
 Connection ~ 2150 1400
@@
 	4450 2600 4600 2600
 Wire Wire Line
-	4450 2300 4450 2600
+	4450 2300 4450 2450
+Wire Wire Line
+	4450 2450 4450 2600
 Wire Wire Line
 	4450 1650 4450 2000
@@
 	850  950  850  1100
 Wire Wire Line
-	850  1100 1450 1100
-Wire Wire Line
-	850  1400 1450 1400
+	850  1100 1150 1100
+Wire Wire Line
+	1150 1100 1450 1100
+Wire Wire Line
+	850  1400 1150 1400
+Wire Wire Line
+	1150 1400 1450 1400
 Connection ~ 1150 1100
 Connection ~ 1150 1400
@@
 	4150 1550 4150 2450
 $Comp
-L R R?
+L R R510
 U 1 1 58A3A42F
 P 3850 3600
-F 0 "R?" V 3930 3600 50  0000 C CNN
+F 0 "R510" V 3930 3600 50  0000 C CNN
 F 1 "0" V 3850 3600 50  0000 C CNN
 F 2 "Resistors_ThroughHole:Resistor_TO-220_Vertical" V 3780 3600 50  0001 C CNN
@@
 	3850 3750 3850 3800
 Wire Wire Line
-	3850 3350 3850 3450
+	3850 3350 3850 3400
+Wire Wire Line
+	3850 3400 3850 3450
 Wire Wire Line
 	3850 3400 2800 3400
 $Comp
-L R R?
+L R R509
 U 1 1 58A3A676
 P 3850 3200
-F 0 "R?" V 3930 3200 50  0000 C CNN
+F 0 "R509" V 3930 3200 50  0000 C CNN
 F 1 "0" V 3850 3200 50  0000 C CNN
 F 2 "Resistors_ThroughHole:Resistor_TO-220_Vertical" V 3780 3200 50  0001 C CNN
@@
 $EndComp
 $Comp
-L R R?
+L R R512
 U 1 1 58A3AFA3
-P 6300 2900
-F 0 "R?" V 6380 2900 50  0000 C CNN
-F 1 "0" V 6300 2900 50  0000 C CNN
-F 2 "Resistors_ThroughHole:Resistor_TO-220_Vertical" V 6230 2900 50  0001 C CNN
-F 3 "" H 6300 2900 50  0000 C CNN
-	1    6300 2900
-	1    0    0    -1
-$EndComp
-$Comp
-L R R?
+P 6300 2950
+F 0 "R512" V 6380 2950 50  0000 C CNN
+F 1 "0" V 6300 2950 50  0000 C CNN
+F 2 "Resistors_ThroughHole:Resistor_TO-220_Vertical" V 6230 2950 50  0001 C CNN
+F 3 "" H 6300 2950 50  0000 C CNN
+	1    6300 2950
+	1    0    0    -1
+$EndComp
+$Comp
+L R R511
 U 1 1 58A3B1B3
 P 6300 2250
-F 0 "R?" V 6380 2250 50  0000 C CNN
+F 0 "R511" V 6380 2250 50  0000 C CNN
 F 1 "0" V 6300 2250 50  0000 C CNN
 F 2 "Resistors_ThroughHole:Resistor_TO-220_Vertical" V 6230 2250 50  0001 C CNN
@@
 	6300 2050 6300 2100
 $Comp
-L C C?
+L C C509
 U 1 1 58A3D583
 P 1700 3250
-F 0 "C?" H 1725 3350 50  0000 L CNN
+F 0 "C509" H 1725 3350 50  0000 L CNN
 F 1 "10uF" H 1725 3150 50  0000 L CNN
 F 2 "Capacitors_SMD:C_1206" H 1738 3100 50  0001 C CNN
@@
 Wire Wire Line
 	1700 3000 1700 3100
-Connection ~ 1900 3000
+Connection ~ 1950 3000
 Wire Wire Line
 	1700 3400 1700 3500

Commit message: update
Other:
- moved on the sheet: R506
Changed lines of the file:
@@
 $EndComp
 Wire Wire Line
-	3850 1650 4450 1650
-Wire Wire Line
-	4450 1650 6300 1650
-Wire Wire Line
-	6300 1650 8750 1650
+	3850 1650 8750 1650
 Wire Wire Line
 	6300 1650 6300 1750
 Wire Wire Line
-	6300 2400 6300 2650
-Wire Wire Line
-	6300 2650 6300 2800
+	6300 2400 6300 2800
 Text GLabel 7300 2200 1    60   Input ~ 0
 +VE
@@
 AGND
 Wire Wire Line
-	6300 2650 6700 2650
-Wire Wire Line
-	6700 2650 7100 2650
+	6300 2650 7100 2650
 Connection ~ 6300 2650
 Wire Wire Line
-	4150 2450 4450 2450
-Wire Wire Line
-	4450 2450 7100 2450
-Wire Wire Line
-	3850 4150 4450 4150
-Wire Wire Line
-	4450 4150 6300 4150
-Wire Wire Line
-	6300 4150 6700 4150
+	4150 2450 7100 2450
+Wire Wire Line
+	3850 4150 6700 4150
 Connection ~ 6300 4150
 $Comp
 L R R506
 U 1 1 5881872C
-P 4450 2150
-F 0 "R506" V 4530 2150 50  0000 C CNN
-F 1 "100" V 4450 2150 50  0000 C CNN
-F 2 "Resistors_ThroughHole:Resistor_TO-220_Vertical" V 4380 2150 50  0001 C CNN
-F 3 "" H 4450 2150 50  0000 C CNN
-	1    4450 2150
+P 4450 2050
+F 0 "R506" V 4530 2050 50  0000 C CNN
+F 1 "100" V 4450 2050 50  0000 C CNN
+F 2 "Resistors_ThroughHole:Resistor_TO-220_Vertical" V 4380 2050 50  0001 C CNN
+F 3 "" H 4450 2050 50  0000 C CNN
+	1    4450 2050
 	1    0    0    -1
 $EndComp
@@
 $EndComp
 Wire Wire Line
-	2500 3000 3000 3000
-Wire Wire Line
-	3000 3000 3150 3000
+	2500 3000 3150 3000
 Wire Wire Line
 	3000 3000 3000 3600
@@
 $EndComp
 Wire Wire Line
-	1700 3000 1950 3000
-Wire Wire Line
-	1950 3000 2200 3000
+	1700 3000 2200 3000
 Wire Wire Line
 	1950 3000 1950 3100
 Wire Wire Line
-	1950 3400 1950 3500
-Wire Wire Line
-	1650 3500 1700 3500
-Wire Wire Line
-	1700 3500 1950 3500
-Wire Wire Line
-	1950 3500 2200 3500
+	1950 3500 1950 3400
+Wire Wire Line
+	1650 3500 2200 3500
 Text GLabel 2600 2700 1    60   Input ~ 0
 +VE
@@
 	3850 4100 3850 4150
 Wire Wire Line
-	6700 3550 6700 4150
-Wire Wire Line
-	6700 4150 6700 4400
+	6700 3550 6700 4400
 Connection ~ 6700 4150
 Wire Wire Line
@@
 	1850 950  1850 1100
 Wire Wire Line
-	1850 1100 2150 1100
-Wire Wire Line
-	2150 1100 2450 1100
-Wire Wire Line
-	1850 1400 2150 1400
-Wire Wire Line
-	2150 1400 2450 1400
+	1850 1100 2450 1100
+Wire Wire Line
+	1850 1400 2450 1400
 Connection ~ 2150 1100
 Connection ~ 2150 1400
@@
 	4450 2600 4600 2600
 Wire Wire Line
-	4450 2300 4450 2450
-Wire Wire Line
-	4450 2450 4450 2600
-Wire Wire Line
-	4450 1650 4450 2000
+	4450 2200 4450 2600
+Wire Wire Line
+	4450 1650 4450 1900
 Connection ~ 4450 1650
 Connection ~ 4450 2450
@@
 	850  950  850  1100
 Wire Wire Line
-	850  1100 1150 1100
-Wire Wire Line
-	1150 1100 1450 1100
-Wire Wire Line
-	850  1400 1150 1400
-Wire Wire Line
-	1150 1400 1450 1400
+	850  1100 1450 1100
+Wire Wire Line
+	850  1400 1450 1400
 Connection ~ 1150 1100
 Connection ~ 1150 1400
@@
 	3850 3750 3850 3800
 Wire Wire Line
-	3850 3350 3850 3400
-Wire Wire Line
-	3850 3400 3850 3450
+	3850 3350 3850 3450
 Wire Wire Line
 	3850 3400 2800 3400

Commit message: v0.2 2dw232
Parts:
- added L501, L502: INDUCTOR, symbol INDUCTOR
- added R513: R, symbol R
- added R514: 0, Resistors_ThroughHole:Resistor_TO-220_Vertical, symbol R
- added RV1, RV2: 1k, symbol POT
- R508: value 10k -> 15k
Connections:
- net +VE: now also L501.1; no longer C506.1, C507.1, C508.1
- net -VE: now also L502.1; no longer C503.1, C504.1, C505.1
- net AGND: no longer U503.2 (A2)
- net at C502.1, U502.2 (-): now also R514.1, RV1.2; no longer R511.2, R512.1
- net V-OUT: now reaches Q502.2 (E), R506.1, R507.1
- net V-OUT: no longer R504.1
- net T-SENSE: now reaches R502.1, R503.1, U501.2 (-)
- net REF renamed Z-SENSE
- net Z-SENSE: now also R504.1
- new net: C503.1, C504.1, C505.1, L502.2
- new net: C506.1, C507.1, C508.1, L501.2
- new net: R510.1, R513.1, RV2.1
- new net: R509.2, RV2.3
- new net: R512.1, R514.2, RV1.3
- new net: R511.2, RV1.1
- new net T-SET: R513.2, RV2.2, U501.3 (+)
- new net Z-SENSE-GND: U503.2 (A2)
Other:
- moved on the sheet: C501, C502, C503, C504, C505, C506, C507, C508, C509, Q501, Q502, R502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

Commit message: update components
Parts:
- L501, L502: footprint (none) -> Resistors_SMD:R_1206
- R513: value R -> 0R; footprint (none) -> Resistors_SMD:R_1206
- R514: value 0 -> 0R; footprint Resistors_ThroughHole:Resistor_TO-220_Vertical -> Resistors_SMD:R_1206
- RV1, RV2: footprint (none) -> Potentiometers:Potentiometer_Bourns_3296W_3-8Zoll_Inline_ScrewUp
Changed lines of the file:
@@
 F 0 "L502" V 2650 5450 50  0000 C CNN
 F 1 "INDUCTOR" V 2800 5450 50  0000 C CNN
-F 2 "" H 2700 5450 50  0000 C CNN
+F 2 "Resistors_SMD:R_1206" H 2700 5450 50  0001 C CNN
 F 3 "" H 2700 5450 50  0000 C CNN
 	1    2700 5450
@@
 F 0 "L501" V 1650 5450 50  0000 C CNN
 F 1 "INDUCTOR" V 1800 5450 50  0000 C CNN
-F 2 "" H 1700 5450 50  0000 C CNN
+F 2 "Resistors_SMD:R_1206" H 1700 5450 50  0001 C CNN
 F 3 "" H 1700 5450 50  0000 C CNN
 	1    1700 5450
@@
 F 0 "RV1" H 7050 2270 50  0000 C CNN
 F 1 "1k" H 7050 2350 50  0000 C CNN
-F 2 "" H 7050 2350 50  0000 C CNN
+F 2 "Potentiometers:Potentiometer_Bourns_3296W_3-8Zoll_Inline_ScrewUp" H 7050 2350 50  0001 C CNN
 F 3 "" H 7050 2350 50  0000 C CNN
 	1    7050 2350
@@
 P 7250 2550
 F 0 "R514" V 7330 2550 50  0000 C CNN
-F 1 "0" V 7250 2550 50  0000 C CNN
-F 2 "Resistors_ThroughHole:Resistor_TO-220_Vertical" V 7180 2550 50  0001 C CNN
+F 1 "0R" V 7250 2550 50  0000 C CNN
+F 2 "Resistors_SMD:R_1206" V 7180 2550 50  0001 C CNN
 F 3 "" H 7250 2550 50  0000 C CNN
 	1    7250 2550
@@
 F 0 "RV2" H 4150 3020 50  0000 C CNN
 F 1 "1k" H 4150 3100 50  0000 C CNN
-F 2 "" H 4150 3100 50  0000 C CNN
+F 2 "Potentiometers:Potentiometer_Bourns_3296W_3-8Zoll_Inline_ScrewUp" H 4150 3100 50  0001 C CNN
 F 3 "" H 4150 3100 50  0000 C CNN
 	1    4150 3100
@@
 P 3900 3300
 F 0 "R513" V 3980 3300 50  0000 C CNN
-F 1 "R" V 3900 3300 50  0000 C CNN
-F 2 "" V 3830 3300 50  0000 C CNN
+F 1 "0R" V 3900 3300 50  0000 C CNN
+F 2 "Resistors_SMD:R_1206" V 3830 3300 50  0001 C CNN
 F 3 "" H 3900 3300 50  0000 C CNN
 	1    3900 3300
@@
 	7050 1700 7050 1750
 Wire Wire Line
-	3100 3100 3700 3100
-Wire Wire Line
-	3700 3100 4000 3100
+	3100 3100 4000 3100
 Wire Wire Line
 	4150 3650 4150 3650
@@
 Connection ~ 2000 5850
 Wire Wire Line
-	1700 6150 2000 6150
-Wire Wire Line
-	2000 6150 2300 6150
-Wire Wire Line
-	1700 5850 2000 5850
-Wire Wire Line
-	2000 5850 2300 5850
+	1700 6150 2300 6150
+Wire Wire Line
+	1700 5850 2300 5850
 Wire Wire Line
 	1700 5750 1700 5850
@@
 	6500 1350 6500 1600
 Wire Wire Line
-	4750 1100 4750 1750
-Wire Wire Line
-	4750 1750 4750 2150
-Wire Wire Line
-	4750 2150 4750 2300
+	4750 1100 4750 2300
 Wire Wire Line
 	4750 2300 4900 2300
@@
 Connection ~ 3000 5850
 Wire Wire Line
-	2700 6150 3000 6150
-Wire Wire Line
-	3000 6150 3300 6150
-Wire Wire Line
-	2700 5850 3000 5850
-Wire Wire Line
-	3000 5850 3300 5850
+	2700 6150 3300 6150
+Wire Wire Line
+	2700 5850 3300 5850
 Wire Wire Line
 	7050 3150 7050 3250
 Connection ~ 7500 4100
 Wire Wire Line
-	7500 3250 7500 4100
-Wire Wire Line
-	7500 4100 7500 4500
-Wire Wire Line
-	4150 4100 7050 4100
-Wire Wire Line
-	7050 4100 7500 4100
+	7500 3250 7500 4500
+Wire Wire Line
+	4150 4100 7500 4100
 Wire Wire Line
 	7050 4100 7050 3550
@@
 	9500 2700 9000 2700
 Wire Wire Line
-	9500 1100 9500 1350
-Wire Wire Line
-	9500 1350 9500 2700
+	9500 1100 9500 2700
 Wire Wire Line
 	1400 2250 1400 3000
@@
 	2900 2250 2900 2900
 Wire Wire Line
-	1700 3200 1900 3200
-Wire Wire Line
-	1900 3200 2250 3200
-Wire Wire Line
-	2250 3200 2500 3200
+	1700 3200 2500 3200
 Wire Wire Line
 	2250 3200 2250 3100
@@
 	2250 2700 2250 2800
 Wire Wire Line
-	1900 2700 2250 2700
-Wire Wire Line
-	2250 2700 2500 2700
+	1900 2700 2500 2700
 Connection ~ 3300 2700
 Wire Wire Line
 	3300 3300 3100 3300
 Wire Wire Line
-	3300 2250 3300 2700
-Wire Wire Line
-	3300 2700 3300 3300
-Wire Wire Line
-	2800 2700 3300 2700
-Wire Wire Line
-	3300 2700 3450 2700
+	3300 2250 3300 3300
+Wire Wire Line
+	2800 2700 3450 2700
 Wire Wire Line
 	4150 2200 4150 2300
@@
 	2700 5750 2700 5850
 Wire Wire Line
-	7050 2500 7050 2700
-Wire Wire Line
-	7050 2700 7050 2850
+	7050 2500 7050 2850
 Wire Wire Line
 	7050 2050 7050 2200
@@
 Connection ~ 7250 2350
 Wire Wire Line
-	4150 3250 4150 3300
-Wire Wire Line
-	4150 3300 4150 3350
+	4150 3250 4150 3350
 Wire Wire Line
 	4150 2600 4150 2950
@@
 	3750 3300 3700 3300
 Wire Wire Line
-	3700 3100 3700 3300
-Wire Wire Line
-	3700 3300 3700 3800
+	3700 3100 3700 3800
 Connection ~ 3700 3100
 Connection ~ 3700 3300
@@
 Connection ~ 6500 2150
 Wire Wire Line
-	4750 2150 6500 2150
-Wire Wire Line
-	6500 2150 7850 2150
+	4750 2150 7850 2150
 Wire Wire Line
 	4150 4000 4150 4100
 Wire Wire Line
-	7200 2350 7250 2350
-Wire Wire Line
-	7250 2350 7500 2350
-Wire Wire Line
-	7500 2350 7850 2350
+	7200 2350 7850 2350
 Wire Wire Line
 	1400 3700 900  3700
@@
 Connection ~ 9500 1350
 Wire Wire Line
-	6500 1350 7050 1350
-Wire Wire Line
-	7050 1350 9500 1350
+	6500 1350 9500 1350
 $EndSCHEMATC

Commit message: update
Parts:
- removed L501, L502: INDUCTOR, Resistors_SMD:R_1206, symbol INDUCTOR
Connections:
- net +VE: now also C506.1, C507.1, C508.1
- net -VE: now also C503.1, C504.1, C505.1
Changed lines of the file:
@@
 	1    0    0    -1
 $EndComp
-Text GLabel 2700 5150 1    60   Input ~ 0
+Text GLabel 2700 5300 1    60   Input ~ 0
 -VE
 Text GLabel 2700 6350 3    60   Input ~ 0
@@
 	1    0    0    -1
 $EndComp
-Text GLabel 1700 5150 1    60   Input ~ 0
+Text GLabel 1700 5300 1    60   Input ~ 0
 +VE
 Text GLabel 1700 6350 3    60   Input ~ 0
@@
 Text GLabel 9500 1100 1    60   Input ~ 0
 V-OUT
-$Comp
-L INDUCTOR L502
-U 1 1 58B22D8C
-P 2700 5450
-F 0 "L502" V 2650 5450 50  0000 C CNN
-F 1 "INDUCTOR" V 2800 5450 50  0000 C CNN
-F 2 "Resistors_SMD:R_1206" H 2700 5450 50  0001 C CNN
-F 3 "" H 2700 5450 50  0000 C CNN
-	1    2700 5450
-	1    0    0    -1
-$EndComp
-$Comp
-L INDUCTOR L501
-U 1 1 58B25362
-P 1700 5450
-F 0 "L501" V 1650 5450 50  0000 C CNN
-F 1 "INDUCTOR" V 1800 5450 50  0000 C CNN
-F 2 "Resistors_SMD:R_1206" H 1700 5450 50  0001 C CNN
-F 3 "" H 1700 5450 50  0000 C CNN
-	1    1700 5450
-	1    0    0    -1
-$EndComp
 $Comp
 L POT RV1
@@
 	1700 5850 2300 5850
 Wire Wire Line
-	1700 5750 1700 5850
+	1700 5300 1700 5850
 Wire Wire Line
 	5900 2600 6000 2600
@@
 	7050 1350 7050 1400
 Wire Wire Line
-	2700 5750 2700 5850
+	2700 5300 2700 5850
 Wire Wire Line
 	7050 2500 7050 2850

Commit message: fix schematic v0.3
Connections:
- net T-SENSE: now also R503.2, U503.3 (K); no longer R502.1, R503.1, U501.2 (-)
- net V-OUT: now also R504.1
- net Z-SENSE: no longer R504.1
- new net: R502.1, R503.1, U501.2 (-)
Other:
- moved on the sheet: R503
Changed lines of the file:
@@
 L R R503
 U 1 1 5881B3DC
-P 3600 2700
-F 0 "R503" V 3680 2700 50  0000 C CNN
-F 1 "10k" V 3600 2700 50  0000 C CNN
-F 2 "Resistors_SMD:R_1206" V 3530 2700 50  0001 C CNN
-F 3 "" H 3600 2700 50  0000 C CNN
-	1    3600 2700
+P 3450 2700
+F 0 "R503" V 3530 2700 50  0000 C CNN
+F 1 "10k" V 3450 2700 50  0000 C CNN
+F 2 "Resistors_SMD:R_1206" V 3380 2700 50  0001 C CNN
+F 3 "" H 3450 2700 50  0000 C CNN
+	1    3450 2700
 	0    -1   -1   0
 $EndComp
@@
 	1    0    0    -1
 $EndComp
-Text GLabel 3300 2250 1    60   Input ~ 0
+Text GLabel 3700 1100 1    60   Input ~ 0
 T-SENSE
-Text GLabel 3700 3800 3    60   Input ~ 0
+Text GLabel 3700 4500 3    60   Input ~ 0
 T-SET
 Text GLabel 9500 1100 1    60   Input ~ 0
@@
 	7050 1700 7050 1750
 Wire Wire Line
-	3100 3100 4000 3100
+	3100 3100 3700 3100
+Wire Wire Line
+	3700 3100 4000 3100
 Wire Wire Line
 	4150 3650 4150 3650
@@
 Connection ~ 2000 5850
 Wire Wire Line
-	1700 6150 2300 6150
-Wire Wire Line
-	1700 5850 2300 5850
+	1700 6150 2000 6150
+Wire Wire Line
+	2000 6150 2300 6150
+Wire Wire Line
+	1700 5850 2000 5850
+Wire Wire Line
+	2000 5850 2300 5850
 Wire Wire Line
 	1700 5300 1700 5850
@@
 Connection ~ 4750 2150
 Wire Wire Line
-	6500 1350 6500 1600
-Wire Wire Line
-	4750 1100 4750 2300
+	6500 1250 6500 1600
+Wire Wire Line
+	4750 1100 4750 2150
+Wire Wire Line
+	4750 2150 4750 2300
 Wire Wire Line
 	4750 2300 4900 2300
 Wire Wire Line
-	3750 2700 4900 2700
+	3600 2700 3700 2700
+Wire Wire Line
+	3700 2700 4900 2700
 Wire Wire Line
 	4750 2500 4750 4500
@@
 Connection ~ 3000 5850
 Wire Wire Line
-	2700 6150 3300 6150
-Wire Wire Line
-	2700 5850 3300 5850
+	2700 6150 3000 6150
+Wire Wire Line
+	3000 6150 3300 6150
+Wire Wire Line
+	2700 5850 3000 5850
+Wire Wire Line
+	3000 5850 3300 5850
 Wire Wire Line
 	7050 3150 7050 3250
 Connection ~ 7500 4100
 Wire Wire Line
-	7500 3250 7500 4500
-Wire Wire Line
-	4150 4100 7500 4100
+	7500 3250 7500 4100
+Wire Wire Line
+	7500 4100 7500 4500
+Wire Wire Line
+	4150 4100 7050 4100
+Wire Wire Line
+	7050 4100 7500 4100
 Wire Wire Line
 	7050 4100 7050 3550
@@
 	9500 2700 9000 2700
 Wire Wire Line
-	9500 1100 9500 2700
+	9500 1100 9500 1250
+Wire Wire Line
+	9500 1250 9500 2700
 Wire Wire Line
 	1400 2250 1400 3000
@@
 	2900 2250 2900 2900
 Wire Wire Line
-	1700 3200 2500 3200
+	1700 3200 1900 3200
+Wire Wire Line
+	1900 3200 2250 3200
+Wire Wire Line
+	2250 3200 2500 3200
 Wire Wire Line
 	2250 3200 2250 3100
@@
 	2250 2700 2250 2800
 Wire Wire Line
-	1900 2700 2500 2700
-Connection ~ 3300 2700
-Wire Wire Line
-	3300 3300 3100 3300
-Wire Wire Line
-	3300 2250 3300 3300
-Wire Wire Line
-	2800 2700 3450 2700
+	1900 2700 2250 2700
+Wire Wire Line
+	2250 2700 2500 2700
+Connection ~ 3200 2700
+Wire Wire Line
+	3200 3300 3100 3300
+Wire Wire Line
+	3200 2700 3200 3300
+Wire Wire Line
+	2800 2700 3200 2700
+Wire Wire Line
+	3200 2700 3300 2700
 Wire Wire Line
 	4150 2200 4150 2300
@@
 Wire Wire Line
 	7500 2350 7500 2950
-Connection ~ 7050 1350
+Connection ~ 7050 1250
 Connection ~ 7050 4100
 Wire Wire Line
 	8050 1850 8050 1950
 Wire Wire Line
-	7050 1350 7050 1400
+	7050 1250 7050 1400
 Wire Wire Line
 	2700 5300 2700 5850
 Wire Wire Line
-	7050 2500 7050 2850
+	7050 2500 7050 2700
+Wire Wire Line
+	7050 2700 7050 2850
 Wire Wire Line
 	7050 2050 7050 2200
@@
 Connection ~ 7250 2350
 Wire Wire Line
-	4150 3250 4150 3350
+	4150 3250 4150 3300
+Wire Wire Line
+	4150 3300 4150 3350
 Wire Wire Line
 	4150 2600 4150 2950
@@
 	3750 3300 3700 3300
 Wire Wire Line
-	3700 3100 3700 3800
+	3700 3100 3700 3300
+Wire Wire Line
+	3700 3300 3700 4500
 Connection ~ 3700 3100
 Connection ~ 3700 3300
@@
 Connection ~ 6500 2150
 Wire Wire Line
-	4750 2150 7850 2150
+	4750 2150 6500 2150
+Wire Wire Line
+	6500 2150 7850 2150
 Wire Wire Line
 	4150 4000 4150 4100
 Wire Wire Line
-	7200 2350 7850 2350
+	7200 2350 7250 2350
+Wire Wire Line
+	7250 2350 7500 2350
+Wire Wire Line
+	7500 2350 7850 2350
 Wire Wire Line
 	1400 3700 900  3700
 Wire Wire Line
-	900  3700 900  1350
-Wire Wire Line
-	900  1350 6000 1350
+	900  3700 900  1650
+Wire Wire Line
+	900  1650 6000 1650
 Wire Wire Line
 	1400 3700 1400 3400
 Wire Wire Line
-	6000 1350 6000 2400
-Wire Wire Line
-	4150 1750 4750 1750
-Connection ~ 4750 1750
-Wire Wire Line
-	4150 1750 4150 1900
-Connection ~ 9500 1350
-Wire Wire Line
-	6500 1350 9500 1350
+	4150 1250 4150 1900
+Connection ~ 9500 1250
+Wire Wire Line
+	4150 1250 6500 1250
+Wire Wire Line
+	6500 1250 7050 1250
+Wire Wire Line
+	7050 1250 9500 1250
+Wire Wire Line
+	6000 1650 6000 2400
+Connection ~ 6500 1250
+Wire Wire Line
+	3700 1100 3700 2700
+Connection ~ 3700 2700
 $EndSCHEMATC
